Commit message: disable odom_x and odom_y

File: catkin_home/src/robot_description/urdf/tiago.urdf.xacro (robot description, xacro)
@@ -99,5 +99,5 @@
     <parent link="odom_yx_link"/>
     <child link="odom_xr_link"/>
-    <limit lower="-10" upper="10" velocity="0.4" effort="1"/>
+    <limit lower="0" upper="0" velocity="0.4" effort="1"/>
     <dynamics damping="0.7" friction="2"/>
   </joint>

File: docker/noetic/tiago_files/tiago.urdf.xacro (robot description, xacro)
@@ -99,5 +99,5 @@
     <parent link="odom_yx_link"/>
     <child link="odom_xr_link"/>
-    <limit lower="-10" upper="10" velocity="0.5" effort="1"/>
+    <limit lower="0" upper="0" velocity="0.5" effort="1"/>
     <dynamics damping="0.7" friction="2"/>
   </joint>
