Commit message: WIP new urdf - first iteration

File: catkin_home/src/robot_description/urdf/robot.gazebo.xacro (robot description, xacro)
@@ -1,15 +1,16 @@
 <?xml version="1.0" encoding="utf-8"?>
 <robot name="robot_sim" xmlns:xacro="http://ros.org/wiki/xacro">
-  <!-- <gazebo>
+  <!-- Differential Plugin -->
+  <gazebo>
     <plugin name="skid_steer_drive_controller" filename="libgazebo_ros_skid_steer_drive.so">
       <updateRate>10.0</updateRate>
-      <robotBaseFrame>/base_footprint</robotBaseFrame>
-      <wheelSeparation>0.20</wheelSeparation>
-      <wheelDiameter>0.08</wheelDiameter>
+      <robotBaseFrame>base_footprint</robotBaseFrame>
+      <!-- <wheelSeparation>0.20</wheelSeparation> -->
+      <wheelDiameter>0.1</wheelDiameter>
       <torque>5</torque>
-      <leftFrontJoint>front_left_wheel_hinge</leftFrontJoint>
-      <rightFrontJoint>front_right_wheel_hinge</rightFrontJoint>
-      <leftRearJoint>rear_left_wheel_hinge</leftRearJoint>
-      <rightRearJoint>rear_right_wheel_hinge</rightRearJoint>
+      <leftFrontJoint>R2</leftFrontJoint>
+      <rightFrontJoint>R1</rightFrontJoint>
+      <leftRearJoint>R3</leftRearJoint>
+      <rightRearJoint>R4</rightRearJoint>
       <topicName>cmd_vel</topicName>
       <commandTopic>cmd_vel</commandTopic>
@@ -21,5 +22,5 @@
       <covariance_yaw>0.010000</covariance_yaw>
     </plugin>
-  </gazebo> -->
+  </gazebo>
   <gazebo>
     <plugin name="gazebo_ros_control" filename="libgazebo_ros_control.so">
@@ -27,27 +28,47 @@
     </plugin>
   </gazebo>
+  <!-- Mechanum Plugin -->
+  <!-- <gazebo>
+    <plugin name="nexus_ros_force_based_move" filename="libnexus_ros_force_based_move.so">
+      <commandTopic>cmd_vel</commandTopic>
+      <odometryTopic>odom</odometryTopic>
+      <odometryFrame>odom</odometryFrame>
+      <odometryRate>25.0</odometryRate>
+      <robotBaseFrame>base_footprint</robotBaseFrame>
+      <cmdVelTimeOut>0.25</cmdVelTimeOut>
+      <publishOdometryTf>1</publishOdometryTf>
+      <yaw_velocity_p_gain>1.0</yaw_velocity_p_gain>
+      <x_velocity_p_gain>15.0</x_velocity_p_gain>
+      <y_velocity_p_gain>15.0</y_velocity_p_gain>
+      <max_x_velocity>0.6</max_x_velocity>
+      <max_y_velocity>0.6</max_y_velocity>
+      <max_yaw_velocity>0.5</max_yaw_velocity>
+    </plugin>
+  </gazebo> -->
   <gazebo reference="base_footprint">
     <material>Gazebo/White</material>
+    <gravity>true</gravity>
+  </gazebo>
+  <gazebo reference="base_link">
+    <material>Gazebo/White</material>
   </gazebo>
   <gazebo reference="base_scan">
     <material>Gazebo/Black</material>
   </gazebo>
-  <gazebo reference="camera_link">
-    <material>Gazebo/Black</material>
-  </gazebo>
-  <!-- <gazebo reference="front_left_wheel">
-    <material>Gazebo/Black</material>
-  </gazebo>
-  <gazebo reference="front_right_wheel">
-    <material>Gazebo/Black</material>
-  </gazebo>
-  <gazebo reference="rear_left_wheel">
-    <material>Gazebo/Black</material>
-  </gazebo>
-  <gazebo reference="rear_right_wheel">
-    <material>Gazebo/Black</material>
-  </gazebo> -->
-  <!-- astra -->
-  <gazebo reference="camera_link">
+  <gazebo reference="R1">
+    <material>Gazebo/Black</material>
+  </gazebo>
+  <gazebo reference="R2">
+    <material>Gazebo/Black</material>
+  </gazebo>
+  <gazebo reference="R3">
+    <material>Gazebo/Black</material>
+  </gazebo>
+  <gazebo reference="R4">
+    <material>Gazebo/Black</material>
+  </gazebo>
+  <!-- astra camera -->
+  <gazebo reference="neck_link">
+    <material>Gazebo/Black</material>
     <sensor type="depth" name="openni_camera_camera">
       <always_on>1</always_on>
@@ -225,3 +246,21 @@
     </sensor>
   </gazebo> -->
+  <gazebo reference="arm_elevator">
+    <material>Gazebo/White</material>
+  </gazebo>
+  <gazebo reference="arm1">
+    <material>Gazebo/White</material>
+  </gazebo>
+  <gazebo reference="arm2">
+    <material>Gazebo/White</material>
+  </gazebo>
+  <gazebo reference="arm3">
+    <material>Gazebo/White</material>
+  </gazebo>
+  <gazebo reference="gripper_left">
+    <material>Gazebo/Black</material>
+  </gazebo>
+  <gazebo reference="gripper_right">
+    <material>Gazebo/Black</material>
+  </gazebo>
 </robot>

File: catkin_home/src/robot_description/urdf/robot.urdf.xacro (robot description, xacro)
@@ -6,4 +6,44 @@
   <virtual_joint name="world_joint" type="planar" parent_frame="odom" child_link="base_footprint"/>
   <link name="base_footprint"></link>
+  <!-- Base -->
+  <link name="base_link">
+    <inertial>
+      <origin
+        xyz="0.148335999572134 -0.00210936158006633 0.352199605023976"
+        rpy="0 0 0" />
+      <mass
+        value="18.1215133555874" />
+      <inertia
+        ixx="0.749373660807315"
+        ixy="-2.04114489679135E-05"
+        ixz="-0.0287031101977872"
+        iyy="0.757729413836528"
+        iyz="2.12902753512543E-05"
+        izz="0.727122404257029" />
+    </inertial>
+    <visual>
+      <origin
+        xyz="0 0 0"
+        rpy="0 0 0" />
+      <geometry>
+        <mesh
+          filename="package://robot_description/meshes/BASE.STL" />
+      </geometry>
+      <material
+        name="">
+        <color
+          rgba="0.792156862745098 0.819607843137255 0.933333333333333 1" />
+      </material>
+    </visual>
+    <collision>
+      <origin
+        xyz="0 0 0"
+        rpy="0 0 0" />
+      <geometry>
+        <mesh
+          filename="package://robot_description/meshes/BASE.STL" />
+      </geometry>
+    </collision>
+  </link>
   <joint name="base_joint" type="fixed">
     <origin xyz="0 0 0" rpy="0 0 0"/>
@@ -11,105 +51,679 @@
     <child link="base_link"/>
   </joint>
-  <!--
-    TODO: SPLIT base_link -> base, lidar, camara, arm.
-    - Check Model Coordinate System
-  -->
-  <link name="base_link">
-    <pose>0 0 0.5 0 0 0</pose>
-    <inertial>
-      <mass
-        value="10" />
-      <origin xyz="0 0 0.04" rpy=" 0 0 0"/>
-      <inertia
-      ixx="0.01" ixy="0.01" ixz="0"
-      iyy="0.01" iyz="0.01"
-      izz="0.01"
-      />
-    </inertial>
-    <visual>
-      <origin
-        xyz="0.2 0.15 0.09"
-        rpy="1.5708 1.5708 3.14159" />
-      <geometry>
-        <mesh
-          filename="package://robot_description/meshes/base_all.STL" />
-      </geometry>
-      <material name="White"/>
-    </visual>
-    <collision>
-      <origin xyz="0 0 0.02" rpy="0 0 0"/>
-      <geometry>
-        <mesh
-          filename="package://robot_description/meshes/base_link.STL" />
-      </geometry>
-    </collision>
-  </link>
-  <!-- Orbbec Astra RGBD Camera -->
-  <joint name="astra_joint" type="fixed">
-    <axis xyz="0 0 0" />
-    <origin xyz="0.19 0.01 0.40" rpy="0 0 0"/>
-    <parent link="base_link"/>
-    <child link="camera_link"/>
-  </joint>
-  <link name="camera_link">
-    <collision>
-      <origin xyz="0.02 0 0" rpy="0 0 0"/>
-      <geometry>0
-        <box size="0.001 0.001 0.001"/>
-      </geometry>
-    </collision>
-    <visual>
-      <origin xyz="-0.01 0 -0.03" rpy="1.5707 0 1.5707"/>
-      <geometry>
-        <mesh filename="package://robot_description/meshes/astra.stl" scale="0.001 0.001 0.001" />
-      </geometry>
-      <material name="Black"/>
-    </visual>
-    <inertial>
-      <mass value="1e-5" />
-      <origin xyz="0 0 0" rpy="0 0 0"/>
-      <inertia ixx="0" ixy="0" ixz="0" iyy="0" iyz="0" izz="0" />
-    </inertial>
+  <!-- Wheel 1 -->
+  <link name="R1">
+    <inertial>
+      <origin
+        xyz="0.275519820527114 0.309814791308341 0.221501694981234"
+        rpy="0 0 0" />
+      <mass
+        value="18.3972196623177" />
+      <inertia
+        ixx="0.749442552183365"
+        ixy="-0.0287031104298118"
+        ixz="2.04115489386414E-05"
+        iyy="0.727191295174375"
+        iyz="-2.12900371583151E-05"
+        izz="0.757827089539184" />
+    </inertial>
+    <visual>
+      <origin
+        xyz="0 0 0"
+        rpy="0 0 0" />
+      <geometry>
+        <mesh
+          filename="package://robot_description/meshes/R1.STL" />
+      </geometry>
+      <material
+        name="">
+        <color
+          rgba="1 1 1 1" />
+      </material>
+    </visual>
+    <collision>
+      <origin
+        xyz="0 0 0"
+        rpy="0 0 0" />
+      <geometry>
+        <mesh
+          filename="package://robot_description/meshes/R1.STL" />
+      </geometry>
+    </collision>
+  </link>
+  <joint name="R1_joint" type="continuous">
+    <origin
+      xyz="-0.13138 0.22304 0.037671"
+      rpy="1.5708 0 0" />
+    <parent
+      link="base_link" />
+    <child
+      link="R1" />
+    <axis
+      xyz="0 0 -1" />
+    <limit
+      effort="1"
+      velocity="5" />
+  </joint>
+  <!-- Wheel 2 -->
+  <link name="R2">
+    <inertial>
+      <origin
+        xyz="0.275519820395461 0.309814790937721 -0.219246732323442"
+        rpy="0 0 0" />
+      <mass
+        value="18.3972196619009" />
+      <inertia
+        ixx="0.749442552215334"
+        ixy="-0.0287031103929444"
+        ixz="2.04115310934196E-05"
+        iyy="0.727191295142013"
+        iyz="-2.12900304772101E-05"
+        izz="0.757827089538814" />
+    </inertial>
+    <visual>
+      <origin
+        xyz="0 0 0"
+        rpy="0 0 0" />
+      <geometry>
+        <mesh
+          filename="package://robot_description/meshes/R2.STL" />
+      </geometry>
+      <material
+        name="">
+        <color
+          rgba="1 1 1 1" />
+      </material>
+    </visual>
+    <collision>
+      <origin
+        xyz="0 0 0"
+        rpy="0 0 0" />
+      <geometry>
+        <mesh
+          filename="package://robot_description/meshes/R2.STL" />
+      </geometry>
+    </collision>
+  </link>
+  <joint name="R2_joint" type="continuous">
+    <origin
+      xyz="-0.13138 -0.22496 0.037671"
+      rpy="1.5708 0 0" />
+    <parent
+      link="base_link" />
+    <child
+      link="R2" />
+    <axis
+      xyz="0 0 -1" />
+    <limit
+      effort="1"
+      velocity="5" />
+  </joint>
+  <!-- Wheel 3 -->
+  <link name="R3">
+    <inertial>
+      <origin
+        xyz="-0.150991110454201 0.309322284097167 0.221501694992569"
+        rpy="0 0 0" />
+      <mass
+        value="18.3972196614284" />
+      <inertia
+        ixx="0.749442552215324"
+        ixy="-0.028703110392855"
+        ixz="2.04115310493071E-05"
+        iyy="0.727191295141718"
+        iyz="-2.12900304537731E-05"
+        izz="0.757827089538575" />
+    </inertial>
+    <visual>
+      <origin
+        xyz="0 0 0"
+        rpy="0 0 0" />
+      <geometry>
+        <mesh
+          filename="package://robot_description/meshes/R3.STL" />
+      </geometry>
+      <material
+        name="">
+        <color
+          rgba="1 1 1 1" />
+      </material>
+    </visual>
+    <collision>
+      <origin
+        xyz="0 0 0"
+        rpy="0 0 0" />
+      <geometry>
+        <mesh
+          filename="package://robot_description/meshes/R3.STL" />
+      </geometry>
+    </collision>
+  </link>
+  <joint name="R3_joint" type="continuous">
+    <origin
+      xyz="0.30162 0.22304 0.038171"
+      rpy="1.5708 0 0" />
+    <parent
+      link="base_link" />
+    <child
+      link="R3" />
+    <axis
+      xyz="0 0 -1" />
+    <limit
+      effort="1"
+      velocity="5" />
+  </joint>
+  <!-- Wheel 4 -->
+  <link name="R4">
+    <inertial>
+      <origin
+        xyz="-0.150991110454394 0.309814790946295 -0.219246732330144"
+        rpy="0 0 0" />
+      <mass
+        value="18.3972196613813" />
+      <inertia
+        ixx="0.749442552215129"
+        ixy="-0.0287031103929106"
+        ixz="2.04115311086233E-05"
+        iyy="0.727191295141816"
+        iyz="-2.12900304940143E-05"
+        izz="0.757827089538487" />
+    </inertial>
+    <visual>
+      <origin
+        xyz="0 0 0"
+        rpy="0 0 0" />
+      <geometry>
+        <mesh
+          filename="package://robot_description/meshes/R4.STL" />
+      </geometry>
+      <material
+        name="">
+        <color
+          rgba="1 1 1 1" />
+      </material>
+    </visual>
+    <collision>
+      <origin
+        xyz="0 0 0"
+        rpy="0 0 0" />
+      <geometry>
+        <mesh
+          filename="package://robot_description/meshes/R4.STL" />
+      </geometry>
+    </collision>
+  </link>
+  <joint name="R4_joint" type="continuous">
+    <origin
+      xyz="0.30162 -0.22496 0.037671"
+      rpy="1.5708 0 0" />
+    <parent
+      link="base_link" />
+    <child
+      link="R4" />
+    <axis
+      xyz="0 0 -1" />
+    <limit
+      effort="1"
+      velocity="5" />
+  </joint>
+  <!-- LIDAR -->
+  <link name="base_scan">
+    <inertial>
+      <origin
+        xyz="0.298611792953018 0.166778725375199 0.00235894981226928"
+        rpy="0 0 0" />
+      <mass
+        value="18.1945955083061" />
+      <inertia
+        ixx="0.749393288148743"
+        ixy="-0.0287035550731546"
+        ixz="2.08817863862389E-05"
+        iyy="0.727163821762413"
+        iyz="-2.12378707755408E-05"
+        izz="0.757753493041592" />
+    </inertial>
+    <visual>
+      <origin
+        xyz="0 0 0"
+        rpy="0 0 0" />
+      <geometry>
+        <mesh
+          filename="package://robot_description/meshes/LIDAR.STL" />
+      </geometry>
+      <material
+        name="">
+        <color
+          rgba="0.792156862745098 0.819607843137255 0.933333333333333 1" />
+      </material>
+    </visual>
+    <collision>
+      <origin
+        xyz="0 0 0"
+        rpy="0 0 0" />
+      <geometry>
+        <mesh
+          filename="package://robot_description/meshes/LIDAR.STL" />
+      </geometry>
+    </collision>
+  </link>
+  <joint name="lidar_joint" type="fixed">
+    <origin
+      xyz="-0.15144 0.00025604 0.18467"
+      rpy="1.5708 0 0" />
+    <parent
+      link="base_link" />
+    <child
+      link="base_scan" />
+    <axis
+      xyz="0 0 0" />
+  </joint>
+  <!-- Neck -->
+  <link name="neck_link">
+    <inertial>
+      <origin
+        xyz="0.222197387044784 -1.38426413702887 0.0179928237545597"
+        rpy="0 0 0" />
+      <mass
+        value="18.1786261624806" />
+      <inertia
+        ixx="0.749404759543456"
+        ixy="-0.0287034119161846"
+        ixz="2.25265620986072E-05"
+        iyy="0.727158689359743"
+        iyz="-2.13534274070571E-05"
+        izz="0.75773953813485" />
+    </inertial>
+    <visual>
+      <origin
+        xyz="0 0 0"
+        rpy="0 0 0" />
+      <geometry>
+        <mesh
+          filename="package://robot_description/meshes/CUELLO_CAMARA.STL" />
+      </geometry>
+      <material
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