Commit message: Add gazebo sensors to urdf

File: catkin_home/src/robot_description/urdf/robot.gazebo.xacro (robot description, xacro)
@@ -1,33 +1,6 @@
 <?xml version="1.0" encoding="utf-8"?>
-<robot name="robot_sim" xmlns:xacro="http://ros.org/wiki/xacro">
-  <!-- Differential Plugin -->
+<robot name="robot_description" xmlns:xacro="http://ros.org/wiki/xacro">
+  <!-- Mechanum Plugin -->
   <gazebo>
-    <plugin name="skid_steer_drive_controller" filename="libgazebo_ros_skid_steer_drive.so">
-      <updateRate>10.0</updateRate>
-      <robotBaseFrame>base_footprint</robotBaseFrame>
-      <!-- <wheelSeparation>0.20</wheelSeparation> -->
-      <wheelDiameter>0.1</wheelDiameter>
-      <torque>5</torque>
-      <leftFrontJoint>R2</leftFrontJoint>
-      <rightFrontJoint>R1</rightFrontJoint>
-      <leftRearJoint>R3</leftRearJoint>
-      <rightRearJoint>R4</rightRearJoint>
-      <topicName>cmd_vel</topicName>
-      <commandTopic>cmd_vel</commandTopic>
-      <broadcastTF>true</broadcastTF>
-      <odometryTopic>odom</odometryTopic>
-      <odometryFrame>/odom</odometryFrame>
-      <covariance_x>0.000100</covariance_x>
-      <covariance_y>0.000100</covariance_y>
-      <covariance_yaw>0.010000</covariance_yaw>
-    </plugin>
-  </gazebo>
-  <gazebo>
-    <plugin name="gazebo_ros_control" filename="libgazebo_ros_control.so">
-      <legacyModeNS>true</legacyModeNS>
-    </plugin>
-  </gazebo>
-  <!-- Mechanum Plugin -->
-  <!-- <gazebo>
     <plugin name="nexus_ros_force_based_move" filename="libnexus_ros_force_based_move.so">
       <commandTopic>cmd_vel</commandTopic>
@@ -45,5 +18,5 @@
       <max_yaw_velocity>0.5</max_yaw_velocity>
     </plugin>
-  </gazebo> -->
+  </gazebo>
   <gazebo reference="base_footprint">
     <material>Gazebo/White</material>
@@ -246,20 +219,20 @@
     </sensor>
   </gazebo> -->
-  <gazebo reference="arm_elevator">
-    <material>Gazebo/White</material>
-  </gazebo>
-  <gazebo reference="arm1">
-    <material>Gazebo/White</material>
-  </gazebo>
-  <gazebo reference="arm2">
-    <material>Gazebo/White</material>
-  </gazebo>
-  <gazebo reference="arm3">
-    <material>Gazebo/White</material>
-  </gazebo>
-  <gazebo reference="gripper_left">
-    <material>Gazebo/Black</material>
-  </gazebo>
-  <gazebo reference="gripper_right">
+  <gazebo reference="Elevador">
+    <material>Gazebo/White</material>
+  </gazebo>
+  <gazebo reference="Brazo_1">
+    <material>Gazebo/White</material>
+  </gazebo>
+  <gazebo reference="Brazo_2">
+    <material>Gazebo/White</material>
+  </gazebo>
+  <gazebo reference="Pinza">
+    <material>Gazebo/White</material>
+  </gazebo>
+  <gazebo reference="Garra_D">
+    <material>Gazebo/Black</material>
+  </gazebo>
+  <gazebo reference="Garra_I">
     <material>Gazebo/Black</material>
   </gazebo>

File: catkin_home/src/robot_description/urdf/robot.urdf.xacro (robot description, xacro)
@@ -10,37 +10,37 @@
     <inertial>
       <origin
-        xyz="0.148335999572134 -0.00210936158006633 0.352199605023976"
+        xyz="-0.140101678990613 0.00114478625174914 0.287628607282214"
         rpy="0 0 0" />
       <mass
         value="18.1215133555874" />
       <inertia
-        ixx="0.749373660807315"
-        ixy="-2.04114489679135E-05"
-        ixz="-0.0287031101977872"
-        iyy="0.757729413836528"
-        iyz="2.12902753512543E-05"
-        izz="0.727122404257029" />
-    </inertial>
-    <visual>
-      <origin
-        xyz="0 0 0"
-        rpy="0 0 0" />
-      <geometry>
-        <mesh
-          filename="package://robot_description/meshes/BASE.STL" />
-      </geometry>
-      <material
-        name="">
-        <color
-          rgba="0.792156862745098 0.819607843137255 0.933333333333333 1" />
-      </material>
-    </visual>
-    <collision>
-      <origin
-        xyz="0 0 0"
-        rpy="0 0 0" />
-      <geometry>
-        <mesh
-          filename="package://robot_description/meshes/BASE.STL" />
+        ixx="0.749373660807314"
+        ixy="-2.04114489679086E-05"
+        ixz="0.0287031101977871"
+        iyy="0.757729413836533"
+        iyz="-2.12902753512747E-05"
+        izz="0.727122404257033" />
+    </inertial>
+    <visual>
+      <origin
+        xyz="0 0 0"
+        rpy="0 0 0" />
+      <geometry>
+        <mesh
+          filename="package://robot_description/meshes/base_link.STL" />
+      </geometry>
+      <material
+        name="">
+        <color
+          rgba="0.792156862745098 0.819607843137255 0.933333333333333 1" />
+      </material>
+    </visual>
+    <collision>
+      <origin
+        xyz="0 0 0"
+        rpy="0 0 0" />
+      <geometry>
+        <mesh
+          filename="package://robot_description/meshes/base_link.STL" />
       </geometry>
     </collision>
@@ -55,15 +55,15 @@
     <inertial>
       <origin
-        xyz="0.275519820527114 0.309814791308341 0.221501694981234"
-        rpy="0 0 0" />
-      <mass
-        value="18.3972196623177" />
-      <inertia
-        ixx="0.749442552183365"
-        ixy="-0.0287031104298118"
-        ixz="2.04115489386414E-05"
-        iyy="0.727191295174375"
-        iyz="-2.12900371583151E-05"
-        izz="0.757827089539184" />
+        xyz="3.23195320450775E-07 -0.0179507439124115 1.34412548334628E-07"
+        rpy="0 0 0" />
+      <mass
+        value="0.27570630673027" />
+      <inertia
+        ixx="6.88913760503531E-05"
+        ixy="-9.99707194725952E-11"
+        ixz="2.32024543753798E-10"
+        iyy="9.7675702655705E-05"
+        iyz="2.38192945242156E-10"
+        izz="6.88909173459932E-05" />
     </inertial>
     <visual>
@@ -91,179 +91,500 @@
     </collision>
   </link>
-  <joint name="R1_joint" type="continuous">
-    <origin
-      xyz="-0.13138 0.22304 0.037671"
-      rpy="1.5708 0 0" />
+  <joint name="Chasis-R1" type="continuous">
+    <origin
+      xyz="0.13960999018429 -0.224000012165135 -0.0268998000000014"
+      rpy="0 0 0" />
     <parent
       link="base_link" />
     <child
       link="R1" />
+    <axis
+      xyz="0 1 0" />
+  </joint>
+  <!-- Wheel 2 -->
+  <link name="R2">
+    <inertial>
+      <origin
+        xyz="3.32396812519065E-07 0.0179292857255078 1.09213569882138E-07"
+        rpy="0 0 0" />
+      <mass
+        value="0.275706306313456" />
+      <inertia
+        ixx="6.88914080188531E-05"
+        ixy="-8.21254945713304E-11"
+        ixz="1.95157168736736E-10"
+        iyy="9.76757022851765E-05"
+        iyz="2.44874061876534E-10"
+        izz="6.88908849846178E-05" />
+    </inertial>
+    <visual>
+      <origin
+        xyz="0 0 0"
+        rpy="0 0 0" />
+      <geometry>
+        <mesh
+          filename="package://robot_description/meshes/R2.STL" />
+      </geometry>
+      <material
+        name="">
+        <color
+          rgba="1 1 1 1" />
+      </material>
+    </visual>
+    <collision>
+      <origin
+        xyz="0 0 0"
+        rpy="0 0 0" />
+      <geometry>
+        <mesh
+          filename="package://robot_description/meshes/R2.STL" />
+      </geometry>
+    </collision>
+  </link>
+  <joint name="Chasis-R2" type="continuous">
+    <origin
+      xyz="0.13960999018429 0.223999987834865 -0.0268998000000016"
+      rpy="0 0 0" />
+    <parent
+      link="base_link" />
+    <child
+      link="R2" />
+    <axis
+      xyz="0 1 0" />
+  </joint>
+  <!-- Wheel 3 -->
+  <link name="R3">
+    <inertial>
+      <origin
+        xyz="3.3240531571721E-07 -0.0179507439283899 1.09240773635277E-07"
+        rpy="0 0 0" />
+      <mass
+        value="0.275706305841014" />
+      <inertia
+        ixx="6.88914080095044E-05"
+        ixy="-8.20813841371881E-11"
+        ixz="1.95067792411591E-10"
+        iyy="9.76757020468613E-05"
+        iyz="2.44897502150705E-10"
+        izz="6.88908846889313E-05" />
+    </inertial>
+    <visual>
+      <origin
+        xyz="0 0 0"
+        rpy="0 0 0" />
+      <geometry>
+        <mesh
+          filename="package://robot_description/meshes/R3.STL" />
+      </geometry>
+      <material
+        name="">
+        <color
+          rgba="1 1 1 1" />
+      </material>
+    </visual>
+    <collision>
+      <origin
+        xyz="0 0 0"
+        rpy="0 0 0" />
+      <geometry>
+        <mesh
+          filename="package://robot_description/meshes/R3.STL" />
+      </geometry>
+    </collision>
+  </link>
+  <joint name="Chasis-R3" type="continuous">
+    <origin
+      xyz="-0.29339000981571 -0.224000012165135 -0.0263997999996424"
+      rpy="0 0 0" />
+    <parent
+      link="base_link" />
+    <child
+      link="R3" />
+    <axis
+      xyz="0 1 0" />
+  </joint>
+  <!-- Wheel 4 -->
+  <link name="R4">
+    <inertial>
+      <origin
+        xyz="3.32392385726799E-07 0.017929285725242 1.09201910493406E-07"
+        rpy="0 0 0" />
+      <mass
+        value="0.275706305793894" />
+      <inertia
+        ixx="6.88914078143537E-05"
+        ixy="-8.21406947723185E-11"
+        ixz="1.95123343999065E-10"
+        iyy="9.76757019588434E-05"
+        iyz="2.44857261652816E-10"
+        izz="6.88908847877444E-05" />
+    </inertial>
+    <visual>
+      <origin
+        xyz="0 0 0"
+        rpy="0 0 0" />
+      <geometry>
+        <mesh
+          filename="package://robot_description/meshes/R4.STL" />
+      </geometry>
+      <material
+        name="">
+        <color
+          rgba="1 1 1 1" />
+      </material>
+    </visual>
+    <collision>
+      <origin
+        xyz="0 0 0"
+        rpy="0 0 0" />
+      <geometry>
+        <mesh
+          filename="package://robot_description/meshes/R4.STL" />
+      </geometry>
+    </collision>
+  </link>
+  <joint name="Chasis-R4" type="continuous">
+    <origin
+      xyz="-0.29339000981571 0.223999987834865 -0.0268998000000015"
+      rpy="0 0 0" />
+    <parent
+      link="base_link" />
+    <child
+      link="R4" />
+    <axis
+      xyz="0 1 0" />
+  </joint>
+  <!-- Elevator -->
+  <link name="Elevador">
+    <inertial>
+      <origin
+        xyz="0.0256407575110341 0.00951016603506605 0.836794245964807"
+        rpy="0 0 0" />
+      <mass
+        value="2.29765936695568" />
+      <inertia
+        ixx="0.125843979664499"
+        ixy="-0.00024645090309376"
+        ixz="7.99558557981761E-06"
+        iyy="0.126438488389742"
+        iyz="2.81429202947702E-06"
+        izz="0.00295411777217587" />
+    </inertial>
+    <visual>
+      <origin
+        xyz="0 0 0"
+        rpy="0 0 0" />
+      <geometry>
+        <mesh
+          filename="package://robot_description/meshes/Elevador.STL" />
+      </geometry>
+      <material
+        name="">
+        <color
+          rgba="0.792156862745098 0.819607843137255 0.933333333333333 1" />
+      </material>
+    </visual>
+    <collision>
+      <origin
+        xyz="0 0 0"
+        rpy="0 0 0" />
+      <geometry>
+        <mesh
+          filename="package://robot_description/meshes/Elevador.STL" />
+      </geometry>
+    </collision>
+  </link>
+  <joint name="Chasis-Elevador" type="revolute">
+    <origin
+      xyz="0 0 -0.0462248000000028"
+      rpy="0 0 0" />
+    <parent
+      link="base_link" />
+    <child
+      link="Elevador" />
+    <axis
+      xyz="0 0 1" />
+    <limit
+      lower="0"
+      upper="0"
+      effort="0"
+      velocity="0" />
+  </joint>
+  <!-- Arm -->
+  <link name="Brazo_1">
+    <inertial>
+      <origin
+        xyz="0.0759877131609833 0.027953575150604 0.0262647126343514"
+        rpy="0 0 0" />
+      <mass
+        value="0.773990320286721" />
+      <inertia
+        ixx="0.000777921915114249"
+        ixy="-0.000249211880454501"
+        ixz="7.9321129777271E-06"
+        iyy="0.00136773587721977"
+        iyz="2.67772483004737E-06"
+        izz="0.00197079000077455" />
+    </inertial>
+    <visual>
+      <origin
+        xyz="0 0 0"
+        rpy="0 0 0" />
+      <geometry>
+        <mesh
+          filename="package://robot_description/meshes/Brazo_1.STL" />
+      </geometry>
+      <material
+        name="">
+        <color
+          rgba="0.792156862745098 0.819607843137255 0.933333333333333 1" />
+      </material>
+    </visual>
+    <collision>
+      <origin
+        xyz="0 0 0"
+        rpy="0 0 0" />
+      <geometry>
+        <mesh
+          filename="package://robot_description/meshes/Brazo_1.STL" />
+      </geometry>
+    </collision>
+  </link>
+  <joint name="Elevador-Brazo_1" type="prismatic">
+    <origin
+      xyz="0 0 0.614229577737656"
+      rpy="0 0 0" />
+    <parent
+      link="Elevador" />
+    <child
+      link="Brazo_1" />
     <axis
       xyz="0 0 -1" />
     <limit
-      effort="1"
-      velocity="5" />
-  </joint>
-  <!-- Wheel 2 -->
-  <link name="R2">
-    <inertial>
-      <origin
-        xyz="0.275519820395461 0.309814790937721 -0.219246732323442"
-        rpy="0 0 0" />
-      <mass
-        value="18.3972196619009" />
-      <inertia
-        ixx="0.749442552215334"
-        ixy="-0.0287031103929444"
-        ixz="2.04115310934196E-05"
-        iyy="0.727191295142013"
-        iyz="-2.12900304772101E-05"
-        izz="0.757827089538814" />
-    </inertial>
-    <visual>
-      <origin
-        xyz="0 0 0"
-        rpy="0 0 0" />
-      <geometry>
-        <mesh
-          filename="package://robot_description/meshes/R2.STL" />
-      </geometry>
-      <material
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
Commit message: fix simulation & gazebo

File: catkin_home/src/robot_description/urdf/robot.gazebo.xacro (robot description, xacro)
@@ -41,6 +41,9 @@
     <material>Gazebo/Black</material>
   </gazebo>
+  <gazebo reference="neck_link">
+    <material>Gazebo/Black</material>
+  </gazebo>
   <!-- astra camera -->
-  <gazebo reference="neck_link">
+  <gazebo reference="camera">
     <material>Gazebo/Black</material>
     <sensor type="depth" name="openni_camera_camera">

File: catkin_home/src/robot_description/urdf/robot.urdf.xacro (robot description, xacro)
@@ -643,15 +643,15 @@
     <inertial>
       <origin
-        xyz="0.0647261774483371 0.0186554769619905 -0.000995943661880272"
-        rpy="0 0 0" />
-      <mass
-        value="0.057112807286796" />
-      <inertia
-        ixx="3.10982316541205E-05"
-        ixy="-2.11505936581601E-06"
-        ixz="2.9733163075116E-07"
-        iyy="1.01242984131521E-05"
-        iyz="-6.49412945412217E-08"
-        izz="3.6285611573039E-05" />
+        xyz="0.0470517349686886 0.0123919567767552 -0.00720656108065509"
+        rpy="0 0 0" />
+      <mass
+        value="0.0123607422626627" />
+      <inertia
+        ixx="3.82073961685766E-06"
+        ixy="-2.35941568160262E-06"
+        ixz="2.98718036301739E-07"
+        iyy="6.17958376424488E-06"
+        iyz="-6.2747610746023E-08"
+        izz="8.92356852920518E-06" />
     </inertial>
     <visual>
@@ -695,18 +695,69 @@
       velocity="0" />
   </joint>
-  <!-- Camera Rgb -->
+  <!-- Camera -->
+  <link name="camera">
+    <inertial>
+      <origin
+        xyz="0.069607946372356 0.0203854936510277 0.000719459986366688"
+        rpy="0 0 0" />
+      <mass
+        value="0.0447520630064878" />
+      <inertia
+        ixx="2.72774898672935E-05"
+        ixy="2.4435672012364E-07"
+        ixz="-1.38631264252966E-09"
+        iyy="3.94471446072863E-06"
+        iyz="-2.1932086349915E-09"
+        izz="2.73620409048763E-05" />
+    </inertial>
+    <visual>
+      <origin
+        xyz="0 0 0"
+        rpy="0 0 0" />
+      <geometry>
+        <mesh
+          filename="package://robot_description/meshes/Camara.STL" />
+      </geometry>
+      <material
+        name="">
+        <color
+          rgba="0.792156862745098 0.819607843137255 0.933333333333333 1" />
+      </material>
+    </visual>
+    <collision>
+      <origin
+        xyz="0 0 0"
+        rpy="0 0 0" />
+      <geometry>
+        <mesh
+          filename="package://robot_description/meshes/Camara.STL" />
+      </geometry>
+    </collision>
+  </link>
+  <joint name="camera_joint" type="fixed">
+    <origin
+      xyz="0 0 0"
+      rpy="0 0.8 0" />
+    <parent
+      link="neck_link" />
+    <child
+      link="camera" />
+    <axis
+      xyz="0 0 0" />
+  </joint>
+  <!-- Camera Rgb Frame -->
   <link name="camera_rgb_frame">
   </link>
   <joint name="camera_optical_joint" type="fixed">
     <origin xyz="0 0 0" rpy="-1.5707 0 -1.5707"/>
-    <parent link="neck_link"/>
+    <parent link="camera"/>
     <child link="camera_rgb_frame"/>
   </joint>
-  <!-- Camera Depth -->
+  <!-- Camera Depth Frame -->
   <link name="camera_depth_frame">
   </link>
   <joint name="camera_depth_joint" type="fixed">
     <origin xyz="0 0 0" rpy="-1.5707 0 -1.5707"/>
-    <parent link="neck_link"/>
+    <parent link="camera"/>
     <child link="camera_depth_frame"/>
   </joint>

Commit message: temp gazebo map

File: catkin_home/src/robot_description/urdf/robot.gazebo.xacro (robot description, xacro)
@@ -44,5 +44,6 @@
     <material>Gazebo/Black</material>
   </gazebo>
-  <!-- astra camera -->
+  <!-- TODO: @josecisneros001, Fix Frames. -->
+  <!-- camera -->
   <gazebo reference="camera">
     <material>Gazebo/Black</material>

File: catkin_home/src/robot_description/urdf/robot.urdf.xacro (robot description, xacro)
@@ -746,9 +746,10 @@
       xyz="0 0 0" />
   </joint>
+  <!-- TODO: @josecisneros001, Fix URDF Camara Joint, No need of x transition. -->
   <!-- Camera Rgb Frame -->
   <link name="camera_rgb_frame">
   </link>
   <joint name="camera_optical_joint" type="fixed">
-    <origin xyz="0 0 0" rpy="-1.5707 0 -1.5707"/>
+    <origin xyz="0.1 0 0" rpy="-1.5707 0 -1.5707"/>
     <parent link="camera"/>
     <child link="camera_rgb_frame"/>
@@ -758,5 +759,5 @@
   </link>
   <joint name="camera_depth_joint" type="fixed">
-    <origin xyz="0 0 0" rpy="-1.5707 0 -1.5707"/>
+    <origin xyz="0.1 0 0" rpy="-1.5707 0 -1.5707"/>
     <parent link="camera"/>
     <child link="camera_depth_frame"/>
