Commit message: fix house simulation

File: catkin_home/src/robot_description/urdf/robot.gazebo.xacro (robot description, xacro)
@@ -44,11 +44,9 @@
     <material>Gazebo/Black</material>
   </gazebo>
-  <!-- TODO: @josecisneros001, Fix Frames. -->
   <!-- camera -->
   <gazebo reference="camera">
     <material>Gazebo/Black</material>
     <sensor type="depth" name="openni_camera_camera">
-      <always_on>1</always_on>
-      <visualize>true</visualize>
+      <update_rate>20</update_rate>
       <camera>
         <horizontal_fov>1.047</horizontal_fov>
@@ -56,16 +54,14 @@
           <width>640</width>
           <height>480</height>
-          <format>R8G8B8</format>
+          <format>B8G8R8</format>
         </image>
-        <depth_camera>
-        </depth_camera>
         <clip>
-          <near>0.1</near>
-          <far>100</far>
+          <near>0.05</near>
+          <far>5</far>
         </clip>
       </camera>
-      <plugin name="kinect_controller" filename="libgazebo_ros_openni_kinect.so">
+      <plugin name="camera_controller" filename="libgazebo_ros_openni_kinect.so">
         <alwaysOn>true</alwaysOn>
-        <updateRate>10.0</updateRate>
+        <updateRate>5.0</updateRate>
         <cameraName>camera</cameraName>
         <frameName>camera_depth_frame</frameName>
@@ -75,15 +71,16 @@
         <cameraInfoTopicName>rgb/camera_info</cameraInfoTopicName>
         <depthImageCameraInfoTopicName>depth/camera_info</depthImageCameraInfoTopicName>
-        <pointCloudCutoff>0.4</pointCloudCutoff>
+        <pointCloudCutoff>0.5</pointCloudCutoff>
         <hackBaseline>0.07</hackBaseline>
-        <distortionK1>0.0</distortionK1>
-        <distortionK2>0.0</distortionK2>
-        <distortionK3>0.0</distortionK3>
-        <distortionT1>0.0</distortionT1>
-        <distortionT2>0.0</distortionT2>
-        <CxPrime>0.0</CxPrime>
-        <Cx>0.0</Cx>
-        <Cy>0.0</Cy>
-        <focalLength>0.0</focalLength>
+        <pointCloudCutoffMax>5.0</pointCloudCutoffMax>
+        <distortionK1>0.00000001</distortionK1>
+        <distortionK2>0.00000001</distortionK2>
+        <distortionK3>0.00000001</distortionK3>
+        <distortionT1>0.00000001</distortionT1>
+        <distortionT2>0.00000001</distortionT2>
+        <CxPrime>0</CxPrime>
+        <Cx>0</Cx>
+        <Cy>0</Cy>
+        <focalLength>0</focalLength>
       </plugin>
     </sensor>

File: catkin_home/src/robot_description/urdf/robot.urdf.xacro (robot description, xacro)
@@ -10,5 +10,5 @@
     <inertial>
       <origin
-        xyz="-0.140101678990613 0.00114478625174914 0.287628607282214"
+        xyz="-0.140101678990613 0.00114478625174916 0.287628607282214"
         rpy="0 0 0" />
       <mass
@@ -259,15 +259,15 @@
     <inertial>
       <origin
-        xyz="0.0256407575110341 0.00951016603506605 0.836794245964807"
-        rpy="0 0 0" />
-      <mass
-        value="2.29765936695568" />
-      <inertia
-        ixx="0.125843979664499"
-        ixy="-0.00024645090309376"
-        ixz="7.99558557981761E-06"
-        iyy="0.126438488389742"
-        iyz="2.81429202947702E-06"
-        izz="0.00295411777217587" />
+        xyz="8.74099458403436E-05 0.000128980381426474 0.936510293479917"
+        rpy="0 0 0" />
+      <mass
+        value="1.52366903082899" />
+      <inertia
+        ixx="0.125067051697286"
+        ixy="3.36175729833583E-06"
+        ixz="8.45368215712956E-08"
+        iyy="0.125069758562973"
+        iyz="1.24631936090211E-07"
+        izz="0.000983327770578956" />
     </inertial>
     <visual>
@@ -315,15 +315,15 @@
     <inertial>
       <origin
-        xyz="0.0759877131609833 0.027953575150604 0.0262647126343514"
-        rpy="0 0 0" />
-      <mass
-        value="0.773990320286721" />
-      <inertia
-        ixx="0.000777921915114249"
-        ixy="-0.000249211880454501"
-        ixz="7.9321129777271E-06"
-        iyy="0.00136773587721977"
-        iyz="2.67772483004737E-06"
-        izz="0.00197079000077455" />
+        xyz="0.079485082754661 0.0154161125335201 0.0357647125153742"
+        rpy="0 0 0" />
+      <mass
+        value="0.77399031960245" />
+      <inertia
+        ixx="0.000714231181888783"
+        ixy="-0.000143123610723033"
+        ixz="8.25869170762567E-06"
+        iyy="0.00143142661510733"
+        iyz="1.37208246328159E-06"
+        izz="0.00197079000658016" />
     </inertial>
     <visual>
@@ -353,5 +353,5 @@
   <joint name="Elevador-Brazo_1" type="prismatic">
     <origin
-      xyz="0 0 0.614229577737656"
+      xyz="0 0 1.09559517536383"
       rpy="0 0 0" />
     <parent
@@ -370,14 +370,14 @@
     <inertial>
       <origin
-        xyz="0.0649979523199693 -0.0804644889479631 -0.0374323913726272"
+        xyz="0.0603177504461659 0.0112878907909101 -0.0279323913726812"
         rpy="0 0 0" />
       <mass
         value="0.437735318876537" />
       <inertia
-        ixx="0.000607820226495373"
-        ixy="0.000430163763985843"
-        ixz="-1.81605266791317E-06"
-        iyy="0.000700121702994888"
-        iyz="1.62843527970453E-06"
+        ixx="0.00025073637578851"
+        ixy="-0.000156756565273837"
+        ixz="-2.39699601792785E-06"
+        iyy="0.00105720555370175"
+        iyz="-4.51950044643041E-07"
         izz="0.00127483380576478" />
     </inertial>
@@ -408,5 +408,5 @@
   <joint name="Elevador-Brazo_2" type="revolute">
     <origin
-      xyz="0.199881404444355 0.12095830267619 0.00474999999999426"
+      xyz="0.229569270853049 0.0439197092955038 0.00475000000002312"
       rpy="0 0 0" />
     <parent
@@ -426,15 +426,15 @@
     <inertial>
       <origin
-        xyz="0.00822789096267251 -0.160174627601703 -0.0523447920814668"
-        rpy="0 0 0" />
-      <mass
-        value="0.378776731215642" />
-      <inertia
-        ixx="0.000195731499797995"
-        ixy="-5.30850733973627E-06"
-        ixz="8.11309040685371E-06"
-        iyy="0.000174638445386028"
-        iyz="3.53105582147945E-06"
-        izz="0.000280838631677078" />
+        xyz="0.0208773657549359 0.000373663977065494 -0.0428447957769276"
+        rpy="0 0 0" />
+      <mass
+        value="0.378776835881696" />
+      <inertia
+        ixx="0.000188658302137669"
+        ixy="-1.12847877871589E-05"
+        ixz="8.84794994829402E-06"
+        iyy="0.000181711737296685"
+        iyz="6.68363237323879E-08"
+        izz="0.000280838719177474" />
     </inertial>
     <visual>
@@ -464,5 +464,5 @@
   <joint name="Brazo_2-Pinza" type="revolute">
     <origin
-      xyz="0.132103898911925 0.0368532399958369 -0.0561933909573693"
+      xyz="0.134775790545599 0.0253548131501961 -0.0561933909574026"
       rpy="0 0 0" />
     <parent
@@ -481,15 +481,15 @@
     <inertial>
       <origin
-        xyz="0.0460540376842404 -0.141548931512324 -0.0433793457424966"
-        rpy="0 0 0" />
-      <mass
-        value="0.0862122663862086" />
-      <inertia
-        ixx="5.18920653975593E-05"
-        ixy="-4.52035584941934E-05"
-        ixz="-1.64203668115444E-06"
-        iyy="0.00011331665564641"
-        iyz="-7.60067376670158E-07"
-        izz="0.000130229108633702" />
+        xyz="0.0531225495268128 -0.0339315603548094 -0.0338793472285259"
+        rpy="0 0 0" />
+      <mass
+        value="0.0862123514148233" />
+      <inertia
+        ixx="5.55837007753562E-05"
+        ixy="4.75027774203442E-05"
+        ixz="-1.51320049118783E-06"
+        iyy="0.000109625335346762"
+        iyz="9.92062324277158E-07"
+        izz="0.000130229416831597" />
     </inertial>
     <visual>
@@ -519,5 +519,5 @@
   <joint name="Pinza-Garra_D" type="revolute">
     <origin
-      xyz="0.0775308919720135 0 -0.0115566090426307"
+      xyz="0.071320629609374 -0.0304040623161534 -0.0115566090426307"
       rpy="0 0 0" />
     <parent
@@ -536,15 +536,15 @@
     <inertial>
       <origin
-        xyz="0.0442330222941579 -0.138024523633636 -0.0433792120867414"
-        rpy="0 0 0" />
-      <mass
-        value="0.0862121352254107" />
-      <inertia
-        ixx="5.00841677058406E-05"
-        ixy="-4.39207489780319E-05"
-        ixz="-1.57017913968264E-06"
-        iyy="0.000115123380941554"
-        iyz="-8.99780118632641E-07"
-        izz="0.000130227952992073" />
+        xyz="0.0482430439842013 0.0405700502182957 -0.0338792120173566"
+        rpy="0 0 0" />
+      <mass
+        value="0.0862120959250573" />
+      <inertia
+        ixx="6.87877660993918E-05"
+        ixy="-5.28740526602163E-05"
+        ixz="-1.37095235100696E-06"
+        iyy="9.64196061499374E-05"
+        iyz="-1.18133299687127E-06"
+        izz="0.000130227781147899" />
     </inertial>
     <visual>
@@ -574,5 +574,5 @@
   <joint name="Pinza-Garra_I" type="revolute">
     <origin
-      xyz="0.045932 0.06246 -0.011557"
+      xyz="0.0667460022512851 0.0394462976294805 -0.0115566090426305"
       rpy="0 0 0" />
     <parent
@@ -682,5 +682,5 @@
     <origin
       xyz="0.083 -0.018139 1.6763"
-      rpy="0 0 0" />
+      rpy="0 0.8 0" />
     <parent
       link="base_link" />
@@ -699,5 +699,5 @@
     <inertial>
       <origin
-        xyz="0.069607946372356 0.0203854936510277 0.000719459986366688"
+        xyz="0.011952 -0.0017536 -3.078E-05"
         rpy="0 0 0" />
       <mass
@@ -737,6 +737,6 @@
   <joint name="camera_joint" type="fixed">
     <origin
-      xyz="0 0 0"
-      rpy="0 0.8 0" />
+      xyz="0.0576563175333489 0.0221390644809871 0.000750239601432945"
+      rpy="0 0 0" />
     <parent
       link="neck_link" />
@@ -746,10 +746,9 @@
       xyz="0 0 0" />
   </joint>
-  <!-- TODO: @josecisneros001, Fix URDF Camara Joint, No need of x transition. -->
   <!-- Camera Rgb Frame -->
   <link name="camera_rgb_frame">
   </link>
   <joint name="camera_optical_joint" type="fixed">
-    <origin xyz="0.1 0 0" rpy="-1.5707 0 -1.5707"/>
+    <origin xyz="0 0 0" rpy="-1.5707 0 -1.5707"/>
     <parent link="camera"/>
     <child link="camera_rgb_frame"/>
@@ -759,5 +758,5 @@
   </link>
   <joint name="camera_depth_joint" type="fixed">
-    <origin xyz="0.1 0 0" rpy="-1.5707 0 -1.5707"/>
+    <origin xyz="0 0 0" rpy="-1.5707 0 -1.5707"/>
     <parent link="camera"/>
     <child link="camera_depth_frame"/>

Commit message: setup octomap & gazebo move controllers

File: catkin_home/src/robot_description/urdf/robot.gazebo.xacro (robot description, xacro)
@@ -43,4 +43,6 @@
   <gazebo reference="neck_link">
     <material>Gazebo/Black</material>
+    <mu1>0.2</mu1>
+    <mu2>0.2</mu2>
   </gazebo>
   <!-- camera -->
@@ -232,4 +234,7 @@
     <material>Gazebo/White</material>
   </gazebo>
+  <gazebo reference="BASE_PINZA">
+    <material>Gazebo/White</material>
+  </gazebo>
   <gazebo reference="Garra_D">
     <material>Gazebo/Black</material>
@@ -238,3 +243,31 @@
     <material>Gazebo/Black</material>
   </gazebo>
+  <!-- Arm Motors Plugin -->
+  <xacro:macro name="gazebo-joint" params="joint">
+    <transmission name="${joint}_transmission">
+      <type>transmission_interface/SimpleTransmission</type>
+      <joint name="${joint}">
+        <hardwareInterface>hardware_interface/EffortJointInterface</hardwareInterface>
+      </joint>
+      <actuator name="${joint}_motor">
+        <hardwareInterface>hardware_interface/EffortJointInterface</hardwareInterface>
+        <mechanicalReduction>1</mechanicalReduction>
+      </actuator>
+    </transmission>
+  </xacro:macro>
+  <xacro:gazebo-joint joint="Chasis_Elevador" />
+  <xacro:gazebo-joint joint="Elevador_Brazo_1" />
+  <xacro:gazebo-joint joint="Elevador_Brazo_2" />
+  <xacro:gazebo-joint joint="Brazo_2_Pinza" />
+  <xacro:gazebo-joint joint="BASE_PINZA_joint" />
+  <xacro:gazebo-joint joint="Pinza_Garra_D" />
+  <xacro:gazebo-joint joint="Pinza_Garra_I" />
+  <xacro:gazebo-joint joint="neck_joint" />
+  <xacro:gazebo-joint joint="Chasis_R1" />
+  <xacro:gazebo-joint joint="Chasis_R2" />
+  <xacro:gazebo-joint joint="Chasis_R3" />
+  <xacro:gazebo-joint joint="Chasis_R4" />
+  <gazebo>
+    <plugin name="gazebo_ros_control" filename="libgazebo_ros_control.so"/>
+  </gazebo>
 </robot>

File: catkin_home/src/robot_description/urdf/robot.urdf.xacro (robot description, xacro)
@@ -298,9 +298,122 @@
     <origin
       xyz="0 0 -0.0462248000000028"
-      rpy="0 0 0" />
+      rpy="0 0 1.57" />
     <parent
       link="base_link" />
     <child
       link="Elevador" />
+    <axis
+      xyz="0 0 1" />
+    <limit
+      lower="-3.14"
+      upper="0"
+      effort="39.0"
+      velocity="4.0" />
+    <dynamics damping="0.7" friction="100.0"/>
+  </joint>
+  <!-- Arm -->
+  <link name="Brazo_1">
+    <inertial>
+      <origin
+        xyz="0.080562 -0.0080834 0.035765"
+        rpy="0 0 0" />
+      <mass
+        value="0.77399" />
+      <inertia
+        ixx="0.00069468"
+        ixy="7.7994E-05"
+        ixz="8.3045E-06"
+        iyy="0.001451"
+        iyz="-1.0599E-06"
+        izz="0.0019708" />
+    </inertial>
+    <visual>
+      <origin
+        xyz="0 0 0"
+        rpy="0 0 0" />
+      <geometry>
+        <mesh
+          filename="package://robot_description/meshes/Brazo_1.STL" />
+      </geometry>
+      <material
+        name="">
+        <color
+          rgba="0.792156862745098 0.819607843137255 0.933333333333333 1" />
+      </material>
+    </visual>
+    <collision>
+      <origin
+        xyz="0 0 0"
+        rpy="0 0 0" />
+      <geometry>
+        <mesh
+          filename="package://robot_description/meshes/Brazo_1.STL" />
+      </geometry>
+    </collision>
+  </link>
+  <joint name="Elevador_Brazo_1" type="prismatic">
+    <origin
+      xyz="0 0 1.09559517536383"
+      rpy="0 0 0" />
+    <parent
+      link="Elevador" />
+    <child
+      link="Brazo_1" />
+    <axis
+      xyz="0 0 -1" />
+    <limit
+      lower="-0.3"
+      upper="0.8"
+      effort="39.0"
+      velocity="4.0" />
+    <dynamics damping="0.7" friction="100.0"/>
+  </joint>
+  <link name="Brazo_2">
+    <inertial>
+      <origin
+        xyz="0.0613443977261393 -0.00158504415996192 -0.0279323913726532"
+        rpy="0 0 0" />
+      <mass
+        value="0.437735318876537" />
+      <inertia
+        ixx="0.000221898875336565"
+        ixy="2.20105438729185E-05"
+        ixz="-2.43850077800155E-06"
+        iyy="0.0010860430541537"
+        iyz="5.96884283352628E-08"
+        izz="0.00127483380576477" />
+    </inertial>
+    <visual>
+      <origin
+        xyz="0 0 0"
+        rpy="0 0 0" />
+      <geometry>
+        <mesh
+          filename="package://robot_description/meshes/Brazo_2.STL" />
+      </geometry>
+      <material
+        name="">
+        <color
+          rgba="0.792156862745098 0.819607843137255 0.933333333333333 1" />
+      </material>
+    </visual>
+    <collision>
+      <origin
+        xyz="0 0 0"
+        rpy="0 0 0" />
+      <geometry>
+        <mesh
+          filename="package://robot_description/meshes/Brazo_2.STL" />
+      </geometry>
+    </collision>
+  </link>
+  <joint name="Elevador_Brazo_2" type="revolute">
+    <origin
+      xyz="0.23254 -0.024031 0.00475"
+      rpy="0 0 0" />
+    <parent
+      link="Brazo_1" />
+    <child
+      link="Brazo_2" />
     <axis
       xyz="0 0 1" />
@@ -310,110 +423,54 @@
       effort="39.0"
       velocity="4.0" />
-    <!-- <dynamics damping="1.0"/> -->
-  </joint>
-  <!-- Arm -->
-  <link name="Brazo_1">
-    <inertial>
-      <origin
-        xyz="0.080562 -0.0080834 0.035765"
-        rpy="0 0 0" />
-      <mass
-        value="0.77399" />
-      <inertia
-        ixx="0.00069468"
-        ixy="7.7994E-05"
-        ixz="8.3045E-06"
-        iyy="0.001451"
-        iyz="-1.0599E-06"
-        izz="0.0019708" />
-    </inertial>
-    <visual>
-      <origin
-        xyz="0 0 0"
-        rpy="0 0 0" />
-      <geometry>
-        <mesh
-          filename="package://robot_description/meshes/Brazo_1.STL" />
-      </geometry>
-      <material
-        name="">
-        <color
-          rgba="0.792156862745098 0.819607843137255 0.933333333333333 1" />
-      </material>
-    </visual>
-    <collision>
-      <origin
-        xyz="0 0 0"
-        rpy="0 0 0" />
-      <geometry>
-        <mesh
-          filename="package://robot_description/meshes/Brazo_1.STL" />
-      </geometry>
-    </collision>
-  </link>
-  <joint name="Elevador_Brazo_1" type="prismatic">
-    <origin
-      xyz="0 0 1.09559517536383"
-      rpy="0 0 0" />
-    <parent
-      link="Elevador" />
-    <child
-      link="Brazo_1" />
-    <axis
-      xyz="0 0 -1" />
-    <limit
-      lower="-0.3"
-      upper="0.8"
-      effort="39.0"
-      velocity="4.0" />
-    <!-- <dynamics damping="1.0"/> -->
-  </joint>
-  <link name="Brazo_2">
-    <inertial>
-      <origin
-        xyz="0.0613443977261393 -0.00158504415996192 -0.0279323913726532"
-        rpy="0 0 0" />
-      <mass
-        value="0.437735318876537" />
-      <inertia
-        ixx="0.000221898875336565"
-        ixy="2.20105438729185E-05"
-        ixz="-2.43850077800155E-06"
-        iyy="0.0010860430541537"
-        iyz="5.96884283352628E-08"
-        izz="0.00127483380576477" />
-    </inertial>
-    <visual>
-      <origin
-        xyz="0 0 0"
-        rpy="0 0 0" />
-      <geometry>
-        <mesh
-          filename="package://robot_description/meshes/Brazo_2.STL" />
-      </geometry>
-      <material
-        name="">
-        <color
-          rgba="0.792156862745098 0.819607843137255 0.933333333333333 1" />
-      </material>
-    </visual>
-    <collision>
-      <origin
-        xyz="0 0 0"
-        rpy="0 0 0" />
-      <geometry>
-        <mesh
-          filename="package://robot_description/meshes/Brazo_2.STL" />
-      </geometry>
-    </collision>
-  </link>
-  <joint name="Elevador_Brazo_2" type="revolute">
-    <origin
-      xyz="0.23254 -0.024031 0.00475"
-      rpy="0 0 0" />
-    <parent
-      link="Brazo_1" />
-    <child
+    <dynamics damping="0.7" friction="100.0"/>
+  </joint>
+  <!-- Gripper -->
+  <link name="Pinza">
+    <inertial>
+      <origin
+        xyz="-0.00819814655383083 -0.00485061932930608 -0.0427651052453255"
+        rpy="0 0 0" />
+      <mass
+        value="0.197688743751798" />
+      <inertia
+        ixx="7.22039610387706E-05"
+        ixy="-1.22111943994307E-05"
+        ixz="6.4739455800225E-06"
+        iyy="0.000104014076525274"
+        iyz="-3.68010060734193E-07"
+        izz="0.000125770789679146" />
+    </inertial>
+    <visual>
+      <origin
+        xyz="0 0 0"
+        rpy="0 0 0" />
+      <geometry>
+        <mesh
+          filename="package://robot_description/meshes/Pinza.STL" />
+      </geometry>
+      <material
+        name="">
+        <color
+          rgba="0.792156862745098 0.819607843137255 0.933333333333333 1" />
+      </material>
+    </visual>
+    <collision>
+      <origin
+        xyz="0 0 0"
+        rpy="0 0 0" />
+      <geometry>
+        <mesh
+          filename="package://robot_description/meshes/Pinza.STL" />
+      </geometry>
+    </collision>
+  </link>
+  <joint name="Brazo_2_Pinza" type="revolute">
+    <origin
+      xyz="0.13777 -0.0035105 -0.04825"
+      rpy="0 0 0" />
+    <parent
       link="Brazo_2" />
+    <child
+      link="Pinza" />
     <axis
       xyz="0 0 1" />
@@ -423,62 +480,5 @@
       effort="39.0"
       velocity="4.0" />
-    <!-- <dynamics damping="1.0"/> -->
-  </joint>
-  <!-- Gripper -->
-  <link name="Pinza">
-    <inertial>
-      <origin
-        xyz="-0.00819814655383083 -0.00485061932930608 -0.0427651052453255"
-        rpy="0 0 0" />
-      <mass
-        value="0.197688743751798" />
-      <inertia
-        ixx="7.22039610387706E-05"
-        ixy="-1.22111943994307E-05"
-        ixz="6.4739455800225E-06"
-        iyy="0.000104014076525274"
-        iyz="-3.68010060734193E-07"
-        izz="0.000125770789679146" />
-    </inertial>
-    <visual>
-      <origin
-        xyz="0 0 0"
-        rpy="0 0 0" />
-      <geometry>
-        <mesh
-          filename="package://robot_description/meshes/Pinza.STL" />
-      </geometry>
-      <material
-        name="">
-        <color
-          rgba="0.792156862745098 0.819607843137255 0.933333333333333 1" />
-      </material>
-    </visual>
-    <collision>
-      <origin
-        xyz="0 0 0"
-        rpy="0 0 0" />
-      <geometry>
-        <mesh
-          filename="package://robot_description/meshes/Pinza.STL" />
-      </geometry>
-    </collision>
-  </link>
-  <joint name="Brazo_2_Pinza" type="revolute">
-    <origin
-      xyz="0.13777 -0.0035105 -0.04825"
-      rpy="0 0 0" />
-    <parent
-      link="Brazo_2" />
-    <child
-      link="Pinza" />
-    <axis
-      xyz="0 0 1" />
-    <limit
-      lower="-1.57"
-      upper="1.57"
-      effort="39.0"
-      velocity="4.0" />
-    <!-- <dynamics damping="1.0"/> -->
+    <dynamics damping="0.7" friction="100.0"/>
   </joint>
   <link name="BASE_PINZA">
@@ -536,4 +536,5 @@
       effort="39.0"
       velocity="4.0" />
+    <dynamics damping="0.7" friction="100.0"/>
   </joint>
   <link name="Garra_D">
@@ -591,5 +592,5 @@
       effort="39.0"
       velocity="4.0" />
-    <!-- <dynamics damping="1.0"/> -->
+    <dynamics damping="0.7" friction="100.0"/>
   </joint>
   <link name="Garra_I">
@@ -647,5 +648,5 @@
       effort="39.0"
       velocity="4.0" />
-    <!-- <dynamics damping="1.0"/> -->
+    <dynamics damping="0.7" friction="100.0"/>
   </joint>
   <!-- LIDAR -->
@@ -753,7 +754,7 @@
       lower="-0.8"
       upper="0.5"
-      effort="0"
-      velocity="0" />
-    <!-- <dynamics damping="0.1"/> -->
+      effort="80.0"
+      velocity="4.0" />
+    <dynamics damping="0.7" friction="100"/>
   </joint>
   <!-- Camera -->
