Commit message: save tmr 2022 status

File: catkin_home/src/robot_description/urdf/robot.gazebo.xacro (robot description, xacro)
@@ -31,21 +31,21 @@
   <gazebo reference="R1">
     <material>Gazebo/Black</material>
-    <mu1>10</mu1>
-    <mu2>10</mu2>
+    <mu1>0.0</mu1>
+    <mu2>0.0</mu2>
   </gazebo>
   <gazebo reference="R2">
     <material>Gazebo/Black</material>
-    <mu1>10</mu1>
-    <mu2>10</mu2>
+    <mu1>0.0</mu1>
+    <mu2>0.0</mu2>
   </gazebo>
   <gazebo reference="R3">
     <material>Gazebo/Black</material>
-    <mu1>10</mu1>
-    <mu2>10</mu2>
+    <mu1>0.0</mu1>
+    <mu2>0.0</mu2>
   </gazebo>
   <gazebo reference="R4">
     <material>Gazebo/Black</material>
-    <mu1>10</mu1>
-    <mu2>10</mu2>
+    <mu1>0.0</mu1>
+    <mu2>0.0</mu2>
   </gazebo>
   <gazebo reference="neck_link">
@@ -273,8 +273,4 @@
   <xacro:gazebo-joint joint="Pinza_Garra_I" />
   <xacro:gazebo-joint joint="neck_joint" />
-  <xacro:gazebo-joint joint="Chasis_R1" />
-  <xacro:gazebo-joint joint="Chasis_R2" />
-  <xacro:gazebo-joint joint="Chasis_R3" />
-  <xacro:gazebo-joint joint="Chasis_R4" />
   <gazebo>
     <plugin name="gazebo_ros_control" filename="libgazebo_ros_control.so"/>

File: catkin_home/src/robot_description/urdf/robot.urdf.xacro (robot description, xacro)
@@ -91,5 +91,5 @@
     </collision>
   </link>
-  <joint name="Chasis_R1" type="continuous">
+  <joint name="Chasis_R1" type="fixed">
     <origin
       xyz="0.13960999018429 -0.224000012165135 -0.0268998000000014"
@@ -101,4 +101,6 @@
     <axis
       xyz="0 1 0" />
+    <limit effort="1" velocity="10"/>
+    <joint_properties damping="5.0" friction="10.0"/>
   </joint>
   <!-- Wheel 2 -->
@@ -142,5 +144,5 @@
     </collision>
   </link>
-  <joint name="Chasis_R2" type="continuous">
+  <joint name="Chasis_R2" type="fixed">
     <origin
       xyz="0.13960999018429 0.223999987834865 -0.0268998000000016"
@@ -152,4 +154,6 @@
     <axis
       xyz="0 1 0" />
+    <limit effort="1" velocity="10"/>
+    <joint_properties damping="5.0" friction="10.0"/>
   </joint>
   <!-- Wheel 3 -->
@@ -193,5 +197,5 @@
     </collision>
   </link>
-  <joint name="Chasis_R3" type="continuous">
+  <joint name="Chasis_R3" type="fixed">
     <origin
       xyz="-0.29339000981571 -0.224000012165135 -0.0263997999996424"
@@ -203,4 +207,6 @@
     <axis
       xyz="0 1 0" />
+    <limit effort="1" velocity="10"/>
+    <joint_properties damping="5.0" friction="10.0"/>
   </joint>
   <!-- Wheel 4 -->
@@ -244,5 +250,5 @@
     </collision>
   </link>
-  <joint name="Chasis_R4" type="continuous">
+  <joint name="Chasis_R4" type="fixed">
     <origin
       xyz="-0.29339000981571 0.223999987834865 -0.0268998000000015"
@@ -254,4 +260,6 @@
     <axis
       xyz="0 1 0" />
+    <limit effort="1" velocity="10"/>
+    <joint_properties damping="5.0" friction="10.0"/>
   </joint>
   <!-- Elevator -->
@@ -480,5 +488,5 @@
       effort="39.0"
       velocity="4.0" />
-    <dynamics damping="0.7" friction="1"/>/>
+    <dynamics damping="0.7" friction="1"/>
   </joint>
   <link name="BASE_PINZA">
@@ -530,5 +538,5 @@
       link="BASE_PINZA" />
     <axis
-      xyz="-0.31288 0.94979 0" />
+      xyz="0 1 0" />
     <limit
       lower="-0.1"
@@ -744,5 +752,5 @@
     <origin
       xyz="0.083 -0.018139 1.6763"
-      rpy="0 0.8 0" />
+      rpy="0 1.1 0" />
     <parent
       link="base_link" />
@@ -752,6 +760,6 @@
       xyz="0 1 0" />
     <limit
-      lower="-0.8"
-      upper="0.5"
+      lower="-1.1"
+      upper="0.2"
       effort="40.0"
       velocity="2.0" />

Commit message: Small Obstacle Avoidance Costmap Implementation

File: catkin_home/src/robot_description/urdf/robot.gazebo.xacro (robot description, xacro)
@@ -14,6 +14,6 @@
       <x_velocity_p_gain>15.0</x_velocity_p_gain>
       <y_velocity_p_gain>15.0</y_velocity_p_gain>
-      <max_x_velocity>1.0</max_x_velocity>
-      <max_y_velocity>1.0</max_y_velocity>
+      <max_x_velocity>0.6</max_x_velocity>
+      <max_y_velocity>0.6</max_y_velocity>
       <max_yaw_velocity>0.5</max_yaw_velocity>
     </plugin>
@@ -230,24 +230,4 @@
     </sensor>
   </gazebo> -->
-  <gazebo reference="imu_link">
-    <gravity>true</gravity>
-    <sensor name="imu_sensor" type="imu">
-      <always_on>true</always_on>
-      <update_rate>100</update_rate>
-      <visualize>true</visualize>
-      <topic>imu</topic>
-      <plugin filename="libgazebo_ros_imu_sensor.so" name="imu_plugin">
-        <topicName>imu</topicName>
-        <bodyName>imu_link</bodyName>
-        <updateRateHZ>10.0</updateRateHZ>
-        <gaussianNoise>0.0</gaussianNoise>
-        <xyzOffset>0 0 0</xyzOffset>
-        <rpyOffset>0 0 0</rpyOffset>
-        <frameName>imu_link</frameName>
-        <initialOrientationAsReference>false</initialOrientationAsReference>
-      </plugin>
-      <pose>0 0 0 0 0 0</pose>
-    </sensor>
-  </gazebo>
   <xacro:macro name="arm_gazebo" params="link">
       <gazebo reference="${link}">
@@ -293,8 +273,4 @@
   <xacro:gazebo-joint joint="Pinza_Garra_I" />
   <xacro:gazebo-joint joint="neck_joint" />
-  <xacro:gazebo-joint joint="Chasis_R1" />
-  <xacro:gazebo-joint joint="Chasis_R2" />
-  <xacro:gazebo-joint joint="Chasis_R3" />
-  <xacro:gazebo-joint joint="Chasis_R4" />
   <gazebo>
     <plugin name="gazebo_ros_control" filename="libgazebo_ros_control.so"/>

File: catkin_home/src/robot_description/urdf/robot.urdf.xacro (robot description, xacro)
@@ -91,5 +91,5 @@
     </collision>
   </link>
-  <joint name="Chasis_R1" type="continuous">
+  <joint name="Chasis_R1" type="fixed">
     <origin
       xyz="0.13960999018429 -0.224000012165135 -0.0268998000000014"
@@ -101,4 +101,6 @@
     <axis
       xyz="0 1 0" />
+    <limit effort="1" velocity="10"/>
+    <joint_properties damping="5.0" friction="10.0"/>
   </joint>
   <!-- Wheel 2 -->
@@ -111,10 +113,10 @@
         value="0.275706306313456" />
       <inertia
-        ixx="6.88914080188531E-05"
-        ixy="-8.21254945713304E-11"
-        ixz="1.95157168736736E-10"
-        iyy="9.76757022851765E-05"
-        iyz="2.44874061876534E-10"
-        izz="6.88908849846178E-05" />
+        ixx="6.88913760503531E-05"
+        ixy="-9.99707194725952E-11"
+        ixz="2.32024543753798E-10"
+        iyy="9.7675702655705E-05"
+        iyz="2.38192945242156E-10"
+        izz="6.88909173459932E-05" />
     </inertial>
     <visual>
@@ -142,5 +144,5 @@
     </collision>
   </link>
-  <joint name="Chasis_R2" type="continuous">
+  <joint name="Chasis_R2" type="fixed">
     <origin
       xyz="0.13960999018429 0.223999987834865 -0.0268998000000016"
@@ -152,4 +154,6 @@
     <axis
       xyz="0 1 0" />
+    <limit effort="1" velocity="10"/>
+    <joint_properties damping="5.0" friction="10.0"/>
   </joint>
   <!-- Wheel 3 -->
@@ -193,5 +197,5 @@
     </collision>
   </link>
-  <joint name="Chasis_R3" type="continuous">
+  <joint name="Chasis_R3" type="fixed">
     <origin
       xyz="-0.29339000981571 -0.224000012165135 -0.0263997999996424"
@@ -203,4 +207,6 @@
     <axis
       xyz="0 1 0" />
+    <limit effort="1" velocity="10"/>
+    <joint_properties damping="5.0" friction="10.0"/>
   </joint>
   <!-- Wheel 4 -->
@@ -244,5 +250,5 @@
     </collision>
   </link>
-  <joint name="Chasis_R4" type="continuous">
+  <joint name="Chasis_R4" type="fixed">
     <origin
       xyz="-0.29339000981571 0.223999987834865 -0.0268998000000015"
@@ -254,4 +260,6 @@
     <axis
       xyz="0 1 0" />
+    <limit effort="1" velocity="10"/>
+    <joint_properties damping="5.0" friction="10.0"/>
   </joint>
   <!-- Elevator -->
@@ -354,5 +362,5 @@
   <joint name="Elevador_Brazo_1" type="prismatic">
     <origin
-      xyz="0 0 1.09559517536383"
+      xyz="0 0 1"
       rpy="0 0 0" />
     <parent
@@ -480,5 +488,5 @@
       effort="39.0"
       velocity="4.0" />
-    <dynamics damping="0.7" friction="1"/>/>
+    <dynamics damping="0.7" friction="1"/>
   </joint>
   <link name="BASE_PINZA">
@@ -530,5 +538,5 @@
       link="BASE_PINZA" />
     <axis
-      xyz="-0.31288 0.94979 0" />
+      xyz="0 1 0" />
     <limit
       lower="-0.1"
@@ -744,5 +752,5 @@
     <origin
       xyz="0.083 -0.018139 1.6763"
-      rpy="0 0.8 0" />
+      rpy="0 1.1 0" />
     <parent
       link="base_link" />
@@ -752,6 +760,6 @@
       xyz="0 1 0" />
     <limit
-      lower="-0.8"
-      upper="0.5"
+      lower="-1.1"
+      upper="0.2"
       effort="40.0"
       velocity="2.0" />
@@ -825,12 +833,3 @@
     <child link="camera_depth_frame"/>
   </joint>
-  <joint name="imu_joint" type="fixed">
-    <axis xyz="0 1 0" />
-    <origin xyz="0.02 0 0.07" rpy="0 0 3.14"/>
-    <parent link="base_link"/>
-    <child link="imu_link"/>
-  </joint>
-  <!-- imu -->
-  <link name="imu_link">
-  </link>
 </robot>
