Commit message: v2.0 dashgo urdf

File: catkin_home/src/robot_description/urdf/dashgo.urdf.xacro (robot description, xacro)
@@ -3,11 +3,10 @@
      Commit Version: 1.6.0-4-g7f85cfe  Build Version: 1.6.7995.38578
      For more information, please see http://wiki.ros.org/sw_urdf_exporter -->
-<robot
-  name="dashgo">
+<robot xmlns:xacro="http://ros.org/wiki/xacro" name="dashgo">
   <link
     name="Base">
     <inertial>
       <origin
-        xyz="7.28752940389825E-05 0.0569098315439797 0.259207232289335"
+        xyz="7.28752940389763E-05 0.0569098315439798 0.259207232289335"
         rpy="0 0 0" />
       <mass
@@ -15,9 +14,9 @@
       <inertia
         ixx="0.134189556605473"
-        ixy="-2.49642917566475E-05"
-        ixz="7.32459015732295E-10"
+        ixy="-2.49642917566465E-05"
+        ixz="7.32459015245289E-10"
         iyy="0.135866070097009"
-        iyz="0.000122787889238702"
-        izz="0.0791062934791392" />
+        iyz="0.000122787889238699"
+        izz="0.0791062934791391" />
     </inertial>
     <visual>
@@ -49,5 +48,5 @@
     <inertial>
       <origin
-        xyz="4.02455846426619E-16 6.52256026967279E-16 0.0200000000000002"
+        xyz="5.39845945723982E-15 1.04291575375726E-14 0.019999999999994"
         rpy="0 0 0" />
       <mass
@@ -55,8 +54,8 @@
       <inertia
         ixx="0.000631308353030454"
-        ixy="-1.64320882748444E-36"
+        ixy="6.14301607074545E-41"
         ixz="1.72050413075699E-18"
         iyy="0.000631308353030454"
-        iyz="-1.31827511759956E-36"
+        iyz="-1.33885585873066E-36"
         izz="0.00112157176228534" />
     </inertial>
@@ -86,9 +85,9 @@
   </link>
   <joint
-    name="Cont1.1Llanta"
+    name="Cont1_1Llanta"
     type="continuous">
     <origin
-      xyz="0.145999999999999 0.1155 0.0375"
-      rpy="1.5707963267949 0 1.5707963267949" />
+      xyz="0.146 0.1155 0.0375"
+      rpy="1.5708 0 1.5708" />
     <parent
       link="Base" />
@@ -139,9 +138,9 @@
   </link>
   <joint
-    name="Cont1.2Llanta"
+    name="Cont1_2Llanta"
     type="continuous">
     <origin
       xyz="-0.146 0.1155 0.0375"
-      rpy="1.5707963267949 0.0209487637131551 1.5707963267949" />
+      rpy="1.5708 0.020949 1.5708" />
     <parent
       link="Base" />
@@ -155,5 +154,5 @@
     <inertial>
       <origin
-        xyz="-1.38777878078145E-17 0.0345546529721542 1.38777878078145E-17"
+        xyz="0 0.0345546529721542 1.38777878078145E-17"
         rpy="0 0 0" />
       <mass
@@ -161,8 +160,8 @@
       <inertia
         ixx="7.54150196205056E-06"
-        ixy="1.40155850818218E-21"
-        ixz="-8.27048938529183E-22"
+        ixy="1.39395083716622E-21"
+        ixz="-8.27180612553027E-22"
         iyy="5.85653067123054E-06"
-        iyz="-1.78257050125666E-21"
+        iyz="-1.76985419744977E-21"
         izz="7.09027556219276E-06" />
     </inertial>
@@ -192,5 +191,5 @@
   </link>
   <joint
-    name="Cont2.1Loca"
+    name="Cont2_1Loca"
     type="continuous">
     <origin
@@ -245,5 +244,5 @@
   </link>
   <joint
-    name="Cont2.2Llanta"
+    name="Cont2_2Llanta"
     type="continuous">
     <origin
@@ -267,9 +266,9 @@
       <inertia
         ixx="7.54150196205055E-06"
-        ixy="3.09430207591605E-21"
-        ixz="2.11758236813575E-22"
+        ixy="3.0363079599354E-21"
+        ixz="2.64697796016969E-22"
         iyy="5.85653067123052E-06"
-        iyz="4.4410066045179E-22"
-        izz="7.09027556219274E-06" />
+        iyz="4.10688840129326E-22"
+        izz="7.09027556219275E-06" />
     </inertial>
     <visual>
@@ -298,5 +297,5 @@
   </link>
   <joint
-    name="Cont3.1Loca"
+    name="Cont3_1Loca"
     type="continuous">
     <origin
@@ -351,5 +350,5 @@
   </link>
   <joint
-    name="Cont3.2Llanta"
+    name="Cont3_2Llanta"
     type="continuous">
     <origin
@@ -404,5 +403,5 @@
   </link>
   <joint
-    name="Cont4.1Lidar"
+    name="Cont4_1Lidar"
     type="fixed">
     <origin
@@ -413,6 +412,4 @@
     <child
       link="Lidar" />
-    <axis
-      xyz="0 1 0" />
   </joint>
   <link
@@ -420,14 +417,14 @@
     <inertial>
       <origin
-        xyz="-0.00218640113558175 0.0383778465870377 -0.00515828443968223"
-        rpy="0 0 0" />
-      <mass
-        value="0.080717320175421" />
+        xyz="-0.00218640113558179 0.0383778465870386 -0.00515828443968225"
+        rpy="0 0 0" />
+      <mass
+        value="0.0807173201754209" />
       <inertia
         ixx="2.37796512993044E-05"
-        ixy="8.55530391588442E-07"
-        ixz="-2.49698267928059E-07"
+        ixy="8.55530391588438E-07"
+        ixz="-2.49698267928064E-07"
         iyy="1.83589770932125E-05"
-        iyz="-4.19202714077007E-06"
+        iyz="-4.19202714077008E-06"
         izz="2.27836705307719E-05" />
     </inertial>
@@ -458,5 +455,5 @@
   <joint
     name="Rev1Cam"
-    type="continuous">
+    type="revolute">
     <origin
       xyz="0.001 0.0505 1.745"
@@ -469,6 +466,6 @@
       xyz="0 1 0" />
     <limit
-      lower="0.5236"
-      upper="-0.5236"
+      lower="-0.5236"
+      upper="0.5236"
       effort="0"
       velocity="0" />
@@ -484,8 +481,8 @@
       <inertia
         ixx="2.60101323603901E-05"
-        ixy="-1.98669220487654E-07"
+        ixy="-1.98669220487655E-07"
         ixz="-5.07308429498082E-06"
         iyy="4.1839084740969E-05"
-        iyz="3.16753039765723E-07"
+        iyz="3.16753039765726E-07"
         izz="3.84670102617887E-05" />
     </inertial>
@@ -516,8 +513,8 @@
   <joint
     name="Rev2Cam"
-    type="continuous">
+    type="revolute">
     <origin
       xyz="0 0.05 0"
-      rpy="-0.12119923501911 -0.000974083686339191 -0.0160540649488372" />
+      rpy="-0.1212 -0.00097408 -0.016054" />
     <parent
       link="RevCam1" />
@@ -525,8 +522,8 @@
       link="RevCam2" />
     <axis
-      xyz="0.991299708192299 0 0.131624042400552" />
+      xyz="0.9913 0 0.13162" />
     <limit
-      lower="0.5236"
-      upper="-0.5236"
+      lower="-0.5236"
+      upper="0.5236"
       effort="0"
       velocity="0" />
@@ -536,14 +533,14 @@
     <inertial>
       <origin
-        xyz="2.70839394232595E-06 0.0154840832193527 0.0423792552563691"
-        rpy="0 0 0" />
-      <mass
-        value="0.152258268041015" />
-      <inertia
-        ixx="2.28182703915157E-05"
-        ixy="-2.5626085953302E-09"
-        ixz="-6.38822957916521E-09"
-        iyy="0.000372324879577432"
-        iyz="-3.15065570916892E-08"
+        xyz="2.70839394232334E-06 0.0154840832193527 0.0423792552563695"
+        rpy="0 0 0" />
+      <mass
+        value="0.152258268041012" />
+      <inertia
+        ixx="2.28182703915153E-05"
+        ixy="-2.56260859534036E-09"
+        ixz="-6.38822957916651E-09"
+        iyy="0.000372324879577431"
+        iyz="-3.15065570917248E-08"
         izz="0.000374741837893712" />
     </inertial>
@@ -576,6 +573,6 @@
     type="fixed">
     <origin
-      xyz="-0.00321508643507233 -0.0539823818454634 0.0300733117769173"
-      rpy="1.4793695539324 0.132007098338006 3.14159265358979" />
+      xyz="-0.0032151 -0.053982 0.030073"
+      rpy="1.4794 0.13201 3.1416" />
     <parent
       link="RevCam2" />
@@ -585,3 +582,91 @@
       xyz="0 0 0" />
   </joint>
+  <link
+    name="BaseBrazo">
+    <inertial>
+      <origin
+        xyz="-3.80554962542412E-17 -6.93889390390723E-17 -4.9999999999939E-05"
+        rpy="0 0 0" />
+      <mass
+        value="0.00121022002997899" />
+      <inertia
+        ixx="1.17272637070328E-06"
+        ixy="2.74649812761777E-23"
+        ixz="-1.57772181044193E-28"
+        iyy="1.17272637070328E-06"
+        iyz="-6.31088724176813E-28"
+        izz="2.34545072437318E-06" />
+    </inertial>
+    <visual>
+      <origin
+        xyz="0 0 0"
+        rpy="0 0 0" />
+      <geometry>
+        <mesh
+          filename="package://robot_description/meshes/Dashgo/BaseBrazo.STL" />
+      </geometry>
+      <material
+        name="">
+        <color
+          rgba="0.792156862745098 0.819607843137255 0.933333333333333 1" />
+      </material>
+    </visual>
+    <collision>
+      <origin
+        xyz="0 0 0"
+        rpy="0 0 0" />
+      <geometry>
+        <mesh
+          filename="package://robot_description/meshes/Dashgo/BaseBrazo.STL" />
+      </geometry>
+    </collision>
+  </link>
+  <joint
+    name="Fix6Bra"
+    type="fixed">
+    <origin
+      xyz="0.0005 0.043 0.4581"
+      rpy="0 0 0" />
+    <parent
+      link="Base" />
+    <child
+      link="BaseBrazo" />
+    <axis
+      xyz="0 0 0" />
+  </joint>
+  <!-- XARM -->
+  <xacro:arg name="prefix" default=""/>
+  <xacro:arg name="ros_namespace" default="xarm"/>
+  <xacro:arg name="limited" default="false"/>
+  <xacro:arg name="effort_control" default="false"/>
+  <xacro:arg name="velocity_control" default="false"/>
+  <xacro:arg name="add_other_geometry" default="false"/>
+  <xacro:arg name="geometry_type" default="box"/>
+  <xacro:arg name="geometry_mass" default="0.1"/>
+  <xacro:arg name="geometry_height" default="0.1"/>
+  <xacro:arg name="geometry_radius" default="0.1"/>
+  <xacro:arg name="geometry_length" default="0.1"/>
+  <xacro:arg name="geometry_width" default="0.1"/>
+  <xacro:arg name="geometry_mesh_filename" default=""/>
+  <xacro:arg name="geometry_mesh_origin_xyz" default="0 0 0"/>
+  <xacro:arg name="geometry_mesh_origin_rpy" default="0 0 0"/>
+  <xacro:arg name="geometry_mesh_tcp_xyz" default="0 0 0"/>
+  <xacro:arg name="geometry_mesh_tcp_rpy" default="0 0 0"/>
+  <xacro:arg name="add_realsense_d435i" default="false"/>
+  <!-- load xarm5 robot -->
+  <xacro:include filename="$(find xarm_description)/urdf/xarm5_robot_macro.xacro" />
+  <xacro:xarm5_robot prefix="$(arg prefix)" namespace="$(arg ros_namespace)" limited="$(arg limited)"
+    effort_control="$(arg effort_control)" velocity_control="$(arg velocity_control)"
+    rs_d435i="$(arg add_realsense_d435i)"
+    attach_to="BaseBrazo"
+    add_other_geometry="$(arg add_other_geometry)"
+    geometry_type="$(arg geometry_type)" geometry_mass="$(arg geometry_mass)"
+    geometry_height="$(arg geometry_height)" geometry_radius="$(arg geometry_radius)"
+    geometry_length="$(arg geometry_length)" geometry_width="$(arg geometry_width)"
+    geometry_mesh_filename="$(arg geometry_mesh_filename)"
+    geometry_mesh_origin_xyz="$(arg geometry_mesh_origin_xyz)" geometry_mesh_origin_rpy="$(arg geometry_mesh_origin_rpy)"
+    geometry_mesh_tcp_xyz="$(arg geometry_mesh_tcp_xyz)" geometry_mesh_tcp_rpy="$(arg geometry_mesh_tcp_rpy)" />
+  <!-- load gripper -->
+  <xacro:include filename="$(find robot_description)/urdf/gripper/gripper.urdf.xacro" />
+  <xacro:load_gripper attach_to="$(arg prefix)link_eef" xyz="0 0 0.003" rpy="0 0 0" />
 </robot>
