Commit message: moveit_config + controllers DASHGO

File: catkin_home/src/robot_description/urdf/dashgo.urdf.xacro (robot description, xacro)
@@ -4,19 +4,71 @@
      For more information, please see http://wiki.ros.org/sw_urdf_exporter -->
 <robot xmlns:xacro="http://ros.org/wiki/xacro" name="dashgo">
+  <virtual_joint child_link="internal_odom" name="world_joint" parent_frame="odom" type="planar" />
+  <!-- ############################BASE_MOVEMENT############################## -->
+  <link name="internal_odom" />
+  <joint name="internal_odom_joint" type="fixed">
+      <origin rpy="0 0 0" xyz="0 0 0" />
+      <parent link="internal_odom" />
+      <child link="internal_odom_inertia" />
+  </joint>
+  <link name="internal_odom_inertia">
+      <inertial>
+          <mass value="0.10" />
+          <!--  assume as square, hence inertia = (1/12) * m * (a^2 + b^2)  -->
+          <inertia ixx="0.000729" ixy="0" ixz="0" iyy="0.000729" iyz="0" izz="0.000729" />
+      </inertial>
+  </link>
+  <joint name="odom_y" type="prismatic">
+      <axis xyz="0 1 0" />
+      <parent link="internal_odom_inertia" />
+      <child link="odom_yx_link" />
+      <limit effort="1" lower="0" upper="0" velocity="0.4" />
+      <dynamics damping="0.7" friction="2" />
+  </joint>
+  <link name="odom_yx_link">
+      <inertial>
+          <mass value="0.10" />
+          <!--  assume as square, hence inertia = (1/12) * m * (a^2 + b^2)  -->
+          <inertia ixx="0.000729" ixy="0" ixz="0" iyy="0.000729" iyz="0" izz="0.000729" />
+      </inertial>
+  </link>
+  <joint name="odom_x" type="prismatic">
+      <axis xyz="1 0 0" />
+      <parent link="odom_yx_link" />
+      <child link="odom_xr_link" />
+      <limit effort="1" lower="-10" upper="10" velocity="0.4" />
+      <dynamics damping="0.7" friction="2" />
+  </joint>
+  <link name="odom_xr_link">
+      <inertial>
+          <mass value="0.10" />
+          <!--  assume as square, hence inertia = (1/12) * m * (a^2 + b^2)  -->
+          <inertia ixx="0.000729" ixy="0" ixz="0" iyy="0.000729" iyz="0" izz="0.000729" />
+      </inertial>
+  </link>
+  <joint name="odom_r" type="revolute">
+      <axis xyz="0 0 1" />
+      <parent link="odom_xr_link" />
+      <child link="base_link" />
+      <limit effort="1" lower="-6.2832" upper="6.2832" velocity="0.4" />
+      <dynamics damping="0.7" friction="2" />
+  </joint>
+  <!-- ########################################################################### -->
+  <link name="base_link"></link>
   <link
     name="Base">
     <inertial>
       <origin
-        xyz="7.28752940389763E-05 0.0569098315439798 0.259207232289335"
-        rpy="0 0 0" />
-      <mass
-        value="5.92220977742572" />
-      <inertia
-        ixx="0.134189556605473"
-        ixy="-2.49642917566465E-05"
-        ixz="7.32459015245289E-10"
-        iyy="0.135866070097009"
-        iyz="0.000122787889238699"
-        izz="0.0791062934791391" />
+        xyz="0.00112427313846248 0.0541261508672339 0.24050906361582"
+        rpy="0 0 0" />
+      <mass
+        value="5.93374358050292" />
+      <inertia
+        ixx="0.102381643014475"
+        ixy="-2.49686782363747E-05"
+        ixz="7.32458903286202E-10"
+        iyy="0.103854959010774"
+        iyz="0.000125261050360604"
+        izz="0.0793094023514086" />
     </inertial>
     <visual>
@@ -44,9 +96,14 @@
     </collision>
   </link>
+  <joint name="base_joint" type="fixed">
+    <origin xyz="0 0 0" rpy="0 0 0"/>
+    <parent link="base_link"/>
+    <child link="Base"/>
+  </joint>
   <link
     name="Llanta1">
     <inertial>
       <origin
-        xyz="5.39845945723982E-15 1.04291575375726E-14 0.019999999999994"
+        xyz="3.88578058618805E-16 6.52256026967279E-16 0.0200000000000003"
         rpy="0 0 0" />
       <mass
@@ -54,8 +111,8 @@
       <inertia
         ixx="0.000631308353030454"
-        ixy="6.14301607074545E-41"
+        ixy="-1.64320882748444E-36"
         ixz="1.72050413075699E-18"
         iyy="0.000631308353030454"
-        iyz="-1.33885585873066E-36"
+        iyz="-1.04568558444466E-36"
         izz="0.00112157176228534" />
     </inertial>
@@ -85,9 +142,9 @@
   </link>
   <joint
-    name="Cont1_1Llanta"
+    name="Llanta1Cont"
     type="continuous">
     <origin
-      xyz="0.146 0.1155 0.0375"
-      rpy="1.5708 0 1.5708" />
+      xyz="0.145999999999999 0.1155 0.0375"
+      rpy="1.5707963267949 0 1.5707963267949" />
     <parent
       link="Base" />
@@ -138,9 +195,9 @@
   </link>
   <joint
-    name="Cont1_2Llanta"
+    name="Llanta2Cont"
     type="continuous">
     <origin
       xyz="-0.146 0.1155 0.0375"
-      rpy="1.5708 0.020949 1.5708" />
+      rpy="1.5707963267949 0.0209487637131551 1.5707963267949" />
     <parent
       link="Base" />
@@ -154,5 +211,5 @@
     <inertial>
       <origin
-        xyz="0 0.0345546529721542 1.38777878078145E-17"
+        xyz="0 0.0345546529721542 -2.77555756156289E-17"
         rpy="0 0 0" />
       <mass
@@ -160,8 +217,8 @@
       <inertia
         ixx="7.54150196205056E-06"
-        ixy="1.39395083716622E-21"
-        ixz="-8.27180612553027E-22"
+        ixy="1.16160786447369E-21"
+        ixz="-8.76254817321673E-22"
         iyy="5.85653067123054E-06"
-        iyz="-1.76985419744977E-21"
+        iyz="-1.79120955050736E-21"
         izz="7.09027556219276E-06" />
     </inertial>
@@ -191,8 +248,8 @@
   </link>
   <joint
-    name="Cont2_1Loca"
+    name="Loca1Cont"
     type="continuous">
     <origin
-      xyz="-0.09 -0.0720000000000001 0"
+      xyz="-0.09 -0.072 0"
       rpy="1.5707963267949 0 0" />
     <parent
@@ -207,14 +264,14 @@
     <inertial>
       <origin
-        xyz="-2.77555756156289E-17 -0.00741632050454702 0"
-        rpy="0 0 0" />
-      <mass
-        value="0.0694291976443344" />
+        xyz="1.38777878078145E-17 -0.00741632050454701 1.38777878078145E-17"
+        rpy="0 0 0" />
+      <mass
+        value="0.0694291976443345" />
       <inertia
         ixx="3.17985725211052E-05"
-        ixy="-5.2134949516848E-38"
-        ixz="0"
+        ixy="-5.21349495168481E-38"
+        ixz="3.52930394689292E-22"
         iyy="1.95153903045283E-05"
-        iyz="7.67877008722871E-41"
+        iyz="7.67877008722515E-41"
         izz="1.95153903045283E-05" />
     </inertial>
@@ -244,5 +301,5 @@
   </link>
   <joint
-    name="Cont2_2Llanta"
+    name="LlantaLoca1Cont"
     type="continuous">
     <origin
@@ -260,15 +317,15 @@
     <inertial>
       <origin
-        xyz="-4.16333634234434E-17 0.0345546529721542 5.55111512312578E-17"
+        xyz="1.38777878078145E-17 0.0345546529721542 2.77555756156289E-17"
         rpy="0 0 0" />
       <mass
         value="0.0167352759899297" />
       <inertia
-        ixx="7.54150196205055E-06"
-        ixy="3.0363079599354E-21"
-        ixz="2.64697796016969E-22"
-        iyy="5.85653067123052E-06"
-        iyz="4.10688840129326E-22"
-        izz="7.09027556219275E-06" />
+        ixx="7.54150196205057E-06"
+        ixy="-2.55901620932607E-21"
+        ixz="3.17637355220363E-22"
+        iyy="5.85653067123054E-06"
+        iyz="2.07178253258396E-21"
+        izz="7.09027556219276E-06" />
     </inertial>
     <visual>
@@ -297,9 +354,9 @@
   </link>
   <joint
-    name="Cont3_1Loca"
+    name="Loca2Cont"
     type="continuous">
     <origin
       xyz="0.09 -0.072 0"
-      rpy="1.5707963267949 0 0.132004559319761" />
+      rpy="1.5707963267949 0 0.119243381039157" />
     <parent
       link="Base" />
@@ -313,5 +370,5 @@
     <inertial>
       <origin
-        xyz="-1.72084568816899E-15 -0.00469061857919632 -0.00574455456677565"
+        xyz="0 -0.00469061857919597 -0.00574455456677592"
         rpy="0 0 0" />
       <mass
@@ -319,9 +376,9 @@
       <inertia
         ixx="3.17985725211052E-05"
-        ixy="1.6940658945086E-21"
-        ixz="-2.22346148654254E-21"
+        ixy="-8.78796682776337E-21"
+        ixz="8.470329472543E-22"
         iyy="1.95153903045283E-05"
-        iyz="2.5410988417629E-21"
-        izz="1.95153903045283E-05" />
+        iyz="-1.6940658945086E-21"
+        izz="1.95153903045284E-05" />
     </inertial>
     <visual>
@@ -350,5 +407,5 @@
   </link>
   <joint
-    name="Cont3_2Llanta"
+    name="LlantaLoca2Cont"
     type="continuous">
     <origin
@@ -403,5 +460,5 @@
   </link>
   <joint
-    name="Cont4_1Lidar"
+    name="Lidar1Cont"
     type="fixed">
     <origin
@@ -417,15 +474,15 @@
     <inertial>
       <origin
-        xyz="-0.00218640113558179 0.0383778465870386 -0.00515828443968225"
-        rpy="0 0 0" />
-      <mass
-        value="0.0807173201754209" />
-      <inertia
-        ixx="2.37796512993044E-05"
-        ixy="8.55530391588438E-07"
-        ixz="-2.49698267928064E-07"
-        iyy="1.83589770932125E-05"
-        iyz="-4.19202714077008E-06"
-        izz="2.27836705307719E-05" />
+        xyz="-0.00218640113558178 0.0383778465870379 -0.00515828443968216"
+        rpy="0 0 0" />
+      <mass
+        value="0.0807173201754215" />
+      <inertia
+        ixx="2.37796512993046E-05"
+        ixy="8.55530391588451E-07"
+        ixz="-2.49698267928072E-07"
+        iyy="1.83589770932126E-05"
+        iyz="-4.19202714077016E-06"
+        izz="2.27836705307722E-05" />
     </inertial>
     <visual>
@@ -454,8 +511,8 @@
   </link>
   <joint
-    name="Rev1Cam"
+    name="Cam1Rev1"
     type="revolute">
     <origin
-      xyz="0.001 0.0505 1.745"
+      xyz="0.001 0.0505 1.545"
       rpy="1.5708 0 0.034703" />
     <parent
@@ -475,15 +532,15 @@
     <inertial>
       <origin
-        xyz="-0.0039179304343604 -0.0102932368661917 0.0320850186207662"
-        rpy="0 0 0" />
-      <mass
-        value="0.0649807233686397" />
-      <inertia
-        ixx="2.60101323603901E-05"
-        ixy="-1.98669220487655E-07"
-        ixz="-5.07308429498082E-06"
-        iyy="4.1839084740969E-05"
-        iyz="3.16753039765726E-07"
-        izz="3.84670102617887E-05" />
+        xyz="-0.00391793043436037 -0.0102932368661919 0.0320850186207662"
+        rpy="0 0 0" />
+      <mass
+        value="0.0649807233686399" />
+      <inertia
+        ixx="2.601013236039E-05"
+        ixy="-1.98669220487697E-07"
+        ixz="-5.07308429498073E-06"
+        iyy="4.18390847409689E-05"
+        iyz="3.16753039765753E-07"
+        izz="3.84670102617888E-05" />
     </inertial>
     <visual>
@@ -512,9 +569,9 @@
   </link>
   <joint
-    name="Rev2Cam"
+    name="Cam1Rev2"
     type="revolute">
     <origin
       xyz="0 0.05 0"
-      rpy="-0.1212 -0.00097408 -0.016054" />
+      rpy="0.0 0.0 0.0" />
     <parent
       link="RevCam1" />
@@ -530,26 +587,26 @@
   </joint>
   <link
-    name="Cam">
-    <inertial>
-      <origin
-        xyz="2.70839394232334E-06 0.0154840832193527 0.0423792552563695"
-        rpy="0 0 0" />
-      <mass
-        value="0.152258268041012" />
-      <inertia
-        ixx="2.28182703915153E-05"
-        ixy="-2.56260859534036E-09"
-        ixz="-6.38822957916651E-09"
-        iyy="0.000372324879577431"
-        iyz="-3.15065570917248E-08"
-        izz="0.000374741837893712" />
-    </inertial>
-    <visual>
-      <origin
-        xyz="0 0 0"
-        rpy="0 0 0" />
-      <geometry>
-        <mesh
-          filename="package://robot_description/meshes/Dashgo/Cam.STL" />
+    name="Cam1">
+    <inertial>
+      <origin
+        xyz="0.0 0.0 0.0"
+        rpy="0 0 0" />
+      <mass
+        value="0.152258268245259" />
+      <inertia
+        ixx="2.28182702795267E-05"
+        ixy="-2.56241481012795E-09"
+        ixz="-6.38770400261561E-09"
+        iyy="0.000372324880916607"
+        iyz="-3.15065555476608E-08"
+        izz="0.000374741839243315" />
+    </inertial>
+    <visual>
+      <origin
+        xyz="-0.02 0 -0.035"
+        rpy="3.1416 3.1416 1.57" />
+      <geometry>
+        <mesh
+          filename="package://robot_description/meshes/Dashgo/Cam1.STL" />
       </geometry>
       <material
@@ -565,18 +622,18 @@
       <geometry>
         <mesh
-          filename="package://robot_description/meshes/Dashgo/Cam.STL" />
-      </geometry>
-    </collision>
-  </link>
-  <joint
-    name="Fix1Cam"
+          filename="package://robot_description/meshes/Dashgo/Cam1.STL" />
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
File: catkin_home/src/robot_description/urdf/gripper/gripper.urdf.xacro (robot description, xacro)
@@ -52,4 +52,11 @@
       </collision>
     </link>
+    <link name="end_effector_link">
+    </link>
+    <joint name="end_effector_joint" type="fixed">
+      <parent link="Base_Gripper" />
+      <child link="end_effector_link" />
+      <origin xyz="0 0 0.165" rpy="0 0 0" />
+    </joint>
     <link
       name="Servo1">
@@ -97,5 +104,6 @@
       <origin
         xyz="0 0.035167 0.088595"
-        rpy="0 -0.36888 -1.5708" />
+        rpy="0 -0.01 -1.5708" />
+        <!-- 0.35 -->
       <parent
         link="Base_Gripper" />
@@ -105,6 +113,6 @@
         xyz="0 1 0" />
       <limit
-        lower="-0.349066"
-        upper="0.349066"
+        lower="-0.39"
+        upper="0.02"
         effort="0"
         velocity="0" />
@@ -208,5 +216,5 @@
       <origin
         xyz="0 -0.034832 0.088595"
-        rpy="0 -0.12482 -1.5708" />
+        rpy="0 -0.02 -1.5708" />
       <parent
         link="Base_Gripper" />
@@ -216,8 +224,12 @@
         xyz="0 1 0" />
       <limit
-        lower="-0.349066"
-        upper="0.349066"
+        lower="-0.02"
+        upper="0.39"
         effort="0"
         velocity="0" />
+      <mimic
+        joint="Rev1Servo"
+        multiplier="-1"
+        offset="0" />
     </joint>
     <link
