Commit message: update urdf, new camera

File: catkin_home/src/robot_description/urdf/dashgo.urdf.xacro (robot description, xacro)
@@ -56,44 +56,4 @@
   <!-- ########################################################################### -->
   <link name="base_link"></link>
-  <link
-    name="Base">
-    <inertial>
-      <origin
-        xyz="0.00112427313846248 0.0541261508672339 0.24050906361582"
-        rpy="0 0 0" />
-      <mass
-        value="5.93374358050292" />
-      <inertia
-        ixx="0.102381643014475"
-        ixy="-2.49686782363747E-05"
-        ixz="7.32458903286202E-10"
-        iyy="0.103854959010774"
-        iyz="0.000125261050360604"
-        izz="0.0793094023514086" />
-    </inertial>
-    <visual>
-      <origin
-        xyz="0 0 0"
-        rpy="0 0 0" />
-      <geometry>
-        <mesh
-          filename="package://robot_description/meshes/Dashgo/Base.STL" />
-      </geometry>
-      <material
-        name="">
-        <color
-          rgba="0.792156862745098 0.819607843137255 0.933333333333333 1" />
-      </material>
-    </visual>
-    <collision>
-      <origin
-        xyz="0 0 0"
-        rpy="0 0 0" />
-      <geometry>
-        <mesh
-          filename="package://robot_description/meshes/Dashgo/Base.STL" />
-      </geometry>
-    </collision>
-  </link>
   <joint name="base_joint" type="fixed">
     <origin xyz="0 0 0" rpy="0 0 0"/>
@@ -101,9 +61,47 @@
     <child link="Base"/>
   </joint>
-  <link
-    name="Llanta1">
-    <inertial>
-      <origin
-        xyz="3.88578058618805E-16 6.52256026967279E-16 0.0200000000000003"
+  <link name="Base">
+    <inertial>
+      <origin
+        xyz="-0.0421641375528847 0.0262460783517876 0.278949374295985"
+        rpy="0 0 0" />
+      <mass
+        value="26.7355250620724" />
+      <inertia
+        ixx="0.418467609556011"
+        ixy="0.0235787657447133"
+        ixz="8.3665476036404E-06"
+        iyy="0.302793463787765"
+        iyz="0.000125414849304393"
+        izz="0.482705153704045" />
+    </inertial>
+    <visual>
+      <origin
+        xyz="0 0 0"
+        rpy="0 0 0" />
+      <geometry>
+        <mesh
+          filename="package://robot_description/meshes/Dashgo/Base.STL" />
+      </geometry>
+      <material
+        name="">
+        <color
+          rgba="0.792156862745098 0.819607843137255 0.933333333333333 1" />
+      </material>
+    </visual>
+    <collision>
+      <origin
+        xyz="0 0 0"
+        rpy="0 0 0" />
+      <geometry>
+        <mesh
+          filename="package://robot_description/meshes/Dashgo/Base.STL" />
+      </geometry>
+    </collision>
+  </link>
+  <link name="Llanta1">
+    <inertial>
+      <origin
+        xyz="4.02455846426619E-16 6.59194920871187E-16 0.0200000000000003"
         rpy="0 0 0" />
       <mass
@@ -114,5 +112,5 @@
         ixz="1.72050413075699E-18"
         iyy="0.000631308353030454"
-        iyz="-1.04568558444466E-36"
+        iyz="-1.31827511759964E-36"
         izz="0.00112157176228534" />
     </inertial>
@@ -141,10 +139,9 @@
     </collision>
   </link>
-  <joint
-    name="Llanta1Cont"
+  <joint name="Llanta1Cont"
     type="continuous">
     <origin
-      xyz="0.145999999999999 0.1155 0.0375"
-      rpy="1.5707963267949 0 1.5707963267949" />
+      xyz="0.146 0.1155 0.0375"
+      rpy="1.5708 0 1.5708" />
     <parent
       link="Base" />
@@ -154,6 +151,5 @@
       xyz="0 0 1" />
   </joint>
-  <link
-    name="Llanta2">
+  <link name="Llanta2">
     <inertial>
       <origin
@@ -194,10 +190,9 @@
     </collision>
   </link>
-  <joint
-    name="Llanta2Cont"
+  <joint name="Llanta2Cont"
     type="continuous">
     <origin
       xyz="-0.146 0.1155 0.0375"
-      rpy="1.5707963267949 0.0209487637131551 1.5707963267949" />
+      rpy="1.5708 0.020949 1.5708" />
     <parent
       link="Base" />
@@ -207,6 +202,5 @@
       xyz="0 0 1" />
   </joint>
-  <link
-    name="Loca1">
+  <link name="Loca1">
     <inertial>
       <origin
@@ -217,8 +211,8 @@
       <inertia
         ixx="7.54150196205056E-06"
-        ixy="1.16160786447369E-21"
-        ixz="-8.76254817321673E-22"
+        ixy="1.29419148906084E-21"
+        ixz="-8.52898332671465E-22"
         iyy="5.85653067123054E-06"
-        iyz="-1.79120955050736E-21"
+        iyz="-1.78257050125666E-21"
         izz="7.09027556219276E-06" />
     </inertial>
@@ -247,10 +241,9 @@
     </collision>
   </link>
-  <joint
-    name="Loca1Cont"
+  <joint name="Loca1Cont"
     type="continuous">
     <origin
       xyz="-0.09 -0.072 0"
-      rpy="1.5707963267949 0 0" />
+      rpy="1.5708 0 0" />
     <parent
       link="Base" />
@@ -260,6 +253,5 @@
       xyz="0 1 0" />
   </joint>
-  <link
-    name="LlantaLoca1">
+  <link name="LlantaLoca1">
     <inertial>
       <origin
@@ -267,5 +259,5 @@
         rpy="0 0 0" />
       <mass
-        value="0.0694291976443345" />
+        value="0.0694291976443344" />
       <inertia
         ixx="3.17985725211052E-05"
@@ -300,6 +292,5 @@
     </collision>
   </link>
-  <joint
-    name="LlantaLoca1Cont"
+  <joint name="LlantaLoca1Cont"
     type="continuous">
     <origin
@@ -313,9 +304,8 @@
       xyz="1 0 0" />
   </joint>
-  <link
-    name="Loca2">
-    <inertial>
-      <origin
-        xyz="1.38777878078145E-17 0.0345546529721542 2.77555756156289E-17"
+  <link name="Loca2">
+    <inertial>
+      <origin
+        xyz="0 0.0345546529721542 2.77555756156289E-17"
         rpy="0 0 0" />
       <mass
@@ -323,8 +313,8 @@
       <inertia
         ixx="7.54150196205057E-06"
-        ixy="-2.55901620932607E-21"
+        ixy="-2.82359729101002E-21"
         ixz="3.17637355220363E-22"
         iyy="5.85653067123054E-06"
-        iyz="2.07178253258396E-21"
+        iyz="2.05773707188381E-21"
         izz="7.09027556219276E-06" />
     </inertial>
@@ -353,10 +343,9 @@
     </collision>
   </link>
-  <joint
-    name="Loca2Cont"
+  <joint name="Loca2Cont"
     type="continuous">
     <origin
       xyz="0.09 -0.072 0"
-      rpy="1.5707963267949 0 0.119243381039157" />
+      rpy="1.5708 0 0.11924" />
     <parent
       link="Base" />
@@ -366,6 +355,5 @@
       xyz="0 1 0" />
   </joint>
-  <link
-    name="LlantaLoca2">
+  <link name="LlantaLoca2">
     <inertial>
       <origin
@@ -376,6 +364,6 @@
       <inertia
         ixx="3.17985725211052E-05"
-        ixy="-8.78796682776337E-21"
-        ixz="8.470329472543E-22"
+        ixy="-8.15269211732264E-21"
+        ixz="4.2351647362715E-22"
         iyy="1.95153903045283E-05"
         iyz="-1.6940658945086E-21"
@@ -406,10 +394,9 @@
     </collision>
   </link>
-  <joint
-    name="LlantaLoca2Cont"
+  <joint name="LlantaLoca2Cont"
     type="continuous">
     <origin
       xyz="0 0.01 0"
-      rpy="-0.886055251315474 0 0" />
+      rpy="-0.88606 0 0" />
     <parent
       link="Loca2" />
@@ -419,6 +406,5 @@
       xyz="1 0 0" />
   </joint>
-  <link
-    name="Lidar">
+  <link name="Lidar">
     <inertial>
       <origin
@@ -459,30 +445,30 @@
     </collision>
   </link>
-  <joint
-    name="Lidar1Cont"
-    type="fixed">
+  <joint name="Lidar1Cont"
+    type="continuous">
     <origin
       xyz="0 -0.11 0.12"
-      rpy="1.5707963267949 0 0" />
+      rpy="1.5708 0 0" />
     <parent
       link="Base" />
     <child
       link="Lidar" />
-  </joint>
-  <link
-    name="RevCam1">
-    <inertial>
-      <origin
-        xyz="-0.00218640113558178 0.0383778465870379 -0.00515828443968216"
-        rpy="0 0 0" />
-      <mass
-        value="0.0807173201754215" />
-      <inertia
-        ixx="2.37796512993046E-05"
-        ixy="8.55530391588451E-07"
-        ixz="-2.49698267928072E-07"
-        iyy="1.83589770932126E-05"
-        iyz="-4.19202714077016E-06"
-        izz="2.27836705307722E-05" />
+    <axis
+      xyz="0 1 0" />
+  </joint>
+  <link name="RevCam1">
+    <inertial>
+      <origin
+        xyz="-0.00218640043520604 0.0373778462346743 0.0578417163847615"
+        rpy="0 0 0" />
+      <mass
+        value="0.0807173231195892" />
+      <inertia
+        ixx="2.37796509107372E-05"
+        ixy="8.55528572510069E-07"
+        ixz="-2.49699440783422E-07"
+        iyy="1.83589761907289E-05"
+        iyz="-4.19202686542368E-06"
+        izz="2.27836700405391E-05" />
     </inertial>
     <visual>
@@ -510,10 +496,9 @@
     </collision>
   </link>
-  <joint
-    name="Cam1Rev1"
+  <joint name="Cam1Rev1"
     type="revolute">
     <origin
-      xyz="0.001 0.0505 1.545"
-      rpy="1.5708 0 0.034703" />
+      xyz="-0.16729 0.098455 1.546"
+      rpy="1.5708 0.0 0.13201" />
     <parent
       link="Base" />
@@ -523,24 +508,23 @@
       xyz="0 1 0" />
     <limit
-      lower="-0.5236"
-      upper="0.5236"
+      lower="-0.54"
+      upper="0.54"
       effort="0"
       velocity="0" />
   </joint>
-  <link
-    name="RevCam2">
-    <inertial>
-      <origin
-        xyz="-0.00391793043436037 -0.0102932368661919 0.0320850186207662"
-        rpy="0 0 0" />
-      <mass
-        value="0.0649807233686399" />
-      <inertia
-        ixx="2.601013236039E-05"
-        ixy="-1.98669220487697E-07"
-        ixz="-5.07308429498073E-06"
-        iyy="4.18390847409689E-05"
-        iyz="3.16753039765753E-07"
-        izz="3.84670102617888E-05" />
+  <link name="RevCam2">
+    <inertial>
+      <origin
+        xyz="0.00149250457233677 -0.00361361108108715 0.0165031514881021"
+        rpy="0 0 0" />
+      <mass
+        value="0.0702746066702973" />
+      <inertia
+        ixx="3.32748236022629E-05"
+        ixy="5.65176745386308E-06"
+        ixz="-4.55903201425305E-06"
+        iyy="4.5252809651764E-05"
+        iyz="4.8432689106791E-06"
+        izz="4.86199055260646E-05" />
     </inertial>
     <visual>
@@ -568,10 +552,9 @@
     </collision>
   </link>
-  <joint
-    name="Cam1Rev2"
+  <joint name="Cam1Rev2"
     type="revolute">
     <origin
-      xyz="0 0.05 0"
-      rpy="0.0 0.0 0.0" />
+      xyz="-0.0021558 0.0036505 0.085266"
+      rpy="-0.08 -0.13856 0.0010948" />
     <parent
       link="RevCam1" />
@@ -579,31 +562,30 @@
       link="RevCam2" />
     <axis
-      xyz="0.9913 0 0.13162" />
+      xyz="1 0 0" />
     <limit
-      lower="-0.5236"
-      upper="0.5236"
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