Commit message: grasping v1.0

File: catkin_home/src/robot_description/urdf/dashgo.urdf.xacro (robot description, xacro)
@@ -23,5 +23,5 @@
       <parent link="internal_odom_inertia" />
       <child link="odom_yx_link" />
-      <limit effort="1" lower="0" upper="0" velocity="0.4" />
+      <limit effort="1" lower="0.0" upper="0.0" velocity="0.08" />
       <dynamics damping="0.7" friction="2" />
   </joint>
@@ -37,5 +37,5 @@
       <parent link="odom_yx_link" />
       <child link="odom_xr_link" />
-      <limit effort="1" lower="-10" upper="10" velocity="0.4" />
+      <limit effort="1" lower="-1.0" upper="1.0" velocity="0.08" />
       <dynamics damping="0.7" friction="2" />
   </joint>
@@ -51,5 +51,5 @@
       <parent link="odom_xr_link" />
       <child link="base_link" />
-      <limit effort="1" lower="-6.2832" upper="6.2832" velocity="0.4" />
+      <limit effort="1" lower="0" upper="0" velocity="0.18" />
       <dynamics damping="0.7" friction="2" />
   </joint>
@@ -57,5 +57,5 @@
   <link name="base_link"></link>
   <joint name="base_joint" type="fixed">
-    <origin xyz="0 0 0" rpy="0 0 0"/>
+    <origin xyz="0 0 0" rpy="0 0 1.57"/>
     <parent link="base_link"/>
     <child link="Base"/>
@@ -96,5 +96,5 @@
       <geometry>
         <mesh
-          filename="package://robot_description/meshes/Dashgo/Base.STL" />
+          filename="package://robot_description/meshes/Dashgo/Base_Collisions.STL" />
       </geometry>
     </collision>
@@ -496,4 +496,40 @@
     </collision>
   </link>
+  <!-- <joint name="Cam1X"
+    type="prismatic">
+    <origin
+      xyz="-0.16729 0.098455 1.546"
+      rpy="1.5708 0.0 0.13201" />
+    <parent
+      link="Base" />
+    <child
+      link="RevCam1" />
+    <axis
+      xyz="0 1 0" />
+    <limit
+      lower="-0.54"
+      upper="0.54"
+      effort="0"
+      velocity="0" />
+  <joint name="cam_y" type="prismatic">
+      <axis xyz="0 1 0" />
+      <parent link="cam" />
+      <child link="cam_yx_link" />
+      <limit effort="1" lower="0.0" upper="0.0" velocity="0.08" />
+      <dynamics damping="0.7" friction="2" />
+  </joint>
+  <link name="cam_yx_link">
+      <inertial>
+          <mass value="0.10" />
+          <inertia ixx="0.000729" ixy="0" ixz="0" iyy="0.000729" iyz="0" izz="0.000729" />
+      </inertial>
+  </link>
+  <joint name="cam_x" type="prismatic">
+      <axis xyz="1 0 0" />
+      <parent link="cam_y_link" />
+      <child link="cam_x_link" />
+      <limit effort="1" lower="-1.0" upper="1.0" velocity="0.08" />
+      <dynamics damping="0.7" friction="2" />
+  </joint> -->
   <joint name="Cam1Rev1"
     type="revolute">
@@ -863,4 +899,6 @@
   <!-- load gripper -->
   <xacro:include filename="$(find robot_description)/urdf/gripper/gripper.urdf.xacro" />
-  <xacro:load_gripper attach_to="$(arg prefix)link_eef" xyz="0 0 0.003" rpy="0 0 1.57" />
+  <xacro:include filename="$(find robot_description)/urdf/gripper/gripperP.urdf.xacro" />
+  <!-- <xacro:load_gripper attach_to="$(arg prefix)link_eef" xyz="0 0 0.003" rpy="0 0 1.57" /> -->
+  <xacro:load_gripperP attach_to="$(arg prefix)link_eef" xyz="0 0 0.003" rpy="0 0 1.57" />
 </robot>

File: catkin_home/src/robot_description/urdf/gripper/gripperP.urdf.xacro (robot description, xacro)
@@ -4,5 +4,5 @@
      For more information, please see http://wiki.ros.org/sw_urdf_exporter -->
 <robot xmlns:xacro="http://ros.org/wiki/xacro" name="Gripper">
-  <xacro:macro name="load_gripper" params="attach_to:='' xyz:='0 0 0' rpy:='0 0 0'">
+  <xacro:macro name="load_gripperP" params="attach_to:='' xyz:='0 0 0' rpy:='0 0 0'">
     <xacro:unless value="${attach_to == ''}">
       <joint name="gripper_fix" type="fixed">
@@ -16,37 +16,37 @@
       <inertial>
         <origin
-          xyz="-0.0060074 0.00022945 0.055534"
-          rpy="0 0 0" />
-        <mass
-          value="0.25675" />
-        <inertia
-          ixx="0.00029732"
-          ixy="5.577E-07"
-          ixz="6.8196E-06"
-          iyy="0.0001154"
-          iyz="-6.3991E-07"
-          izz="0.00028425" />
-      </inertial>
-      <visual>
-        <origin
-          xyz="0 0 0"
-          rpy="0 0 0" />
-        <geometry>
-          <mesh
-            filename="package://robot_description/meshes/Gripper/Base.STL" />
-        </geometry>
-        <material
-          name="">
-          <color
-            rgba="0.79216 0.81961 0.93333 1" />
-        </material>
-      </visual>
-      <collision>
-        <origin
-          xyz="0 0 0"
-          rpy="0 0 0" />
-        <geometry>
-          <mesh
-            filename="package://robot_description/meshes/Gripper/Base.STL" />
+          xyz="0.0235336388798847 -0.000229446948367704 0.0267925511331642"
+          rpy="0 0 0" />
+        <mass
+          value="0.256752989485429" />
+        <inertia
+          ixx="0.000284254820291498"
+          ixy="6.39914341640259E-07"
+          ixz="6.8196058010128E-06"
+          iyy="0.000115396784193605"
+          iyz="-5.5770176736161E-07"
+          izz="0.000297324024700765" />
+      </inertial>
+      <visual>
+        <origin
+          xyz="0 0 0"
+          rpy="0 0 0" />
+        <geometry>
+          <mesh
+            filename="package://robot_description/meshes/GripperP/BaseGri.STL" />
+        </geometry>
+        <material
+          name="">
+          <color
+            rgba="0.792156862745098 0.819607843137255 0.933333333333333 1" />
+        </material>
+      </visual>
+      <collision>
+        <origin
+          xyz="0 0 0"
+          rpy="0 0 0" />
+        <geometry>
+          <mesh
+            filename="package://robot_description/meshes/GripperP/BaseGri.STL" />
         </geometry>
       </collision>
@@ -57,5 +57,5 @@
       <parent link="Base_Gripper" />
       <child link="end_effector_link" />
-      <origin xyz="0 0 0.165" rpy="0 -1.57 0" />
+      <origin xyz="0.156 0 0.04" rpy="0 0 0" />
     </joint>
     <link
@@ -63,37 +63,37 @@
       <inertial>
         <origin
-          xyz="-4.50497350326651E-08 0.00440252858837619 0.0186297249994029"
-          rpy="0 0 0" />
-        <mass
-          value="0.0250047254852256" />
-        <inertia
-          ixx="1.36408467918995E-05"
-          ixy="1.57759886426113E-19"
-          ixz="-1.71524171818996E-19"
-          iyy="3.54946158391808E-06"
-          iyz="-1.80956359903929E-06"
-          izz="1.22463749616553E-05" />
-      </inertial>
-      <visual>
-        <origin
-          xyz="0 0 0"
-          rpy="0 0 0" />
-        <geometry>
-          <mesh
-            filename="package://robot_description/meshes/Gripper/Servo1.STL" />
-        </geometry>
-        <material
-          name="">
-          <color
-            rgba="0.792156862745098 0.819607843137255 0.933333333333333 1" />
-        </material>
-      </visual>
-      <collision>
-        <origin
-          xyz="0 0 0"
-          rpy="0 0 0" />
-        <geometry>
-          <mesh
-            filename="package://robot_description/meshes/Gripper/Servo1.STL" />
+          xyz="0.0186297249994027 -4.50497350604206E-08 -0.0319399514116179"
+          rpy="0 0 0" />
+        <mass
+          value="0.0250047254852252" />
+        <inertia
+          ixx="1.22463749616552E-05"
+          ixy="-1.64997983105085E-19"
+          ixz="-1.80956359903934E-06"
+          iyy="1.36408467918994E-05"
+          iyz="1.59449099201962E-19"
+          izz="3.54946158391805E-06" />
+      </inertial>
+      <visual>
+        <origin
+          xyz="0 0 0"
+          rpy="0 0 0" />
+        <geometry>
+          <mesh
+            filename="package://robot_description/meshes/GripperP/Servo1.STL" />
+        </geometry>
+        <material
+          name="">
+          <color
+            rgba="0.792156862745098 0.819607843137255 0.933333333333333 1" />
+        </material>
+      </visual>
+      <collision>
+        <origin
+          xyz="0 0 0"
+          rpy="0 0 0" />
+        <geometry>
+          <mesh
+            filename="package://robot_description/meshes/GripperP/Servo1.STL" />
         </geometry>
       </collision>
@@ -103,7 +103,6 @@
       type="revolute">
       <origin
-        xyz="0 0.035167 0.088595"
-        rpy="0 -0.01 -1.5708" />
-        <!-- 0.35 -->
+        xyz="0.056595 0.034832 0.069142"
+        rpy="0 0 0" />
       <parent
         link="Base_Gripper" />
@@ -111,119 +110,119 @@
         link="Servo1" />
       <axis
-        xyz="0 1 0" />
+        xyz="0 0 1" />
+      <limit
+        lower="-0.02"
+        upper="0.39"
+        effort="0"
+        velocity="0" />
+    </joint>
+    <link
+      name="Dedo1">
+      <inertial>
+        <origin
+          xyz="-0.0339571348134267 -9.21108600088205E-08 0.148247426657738"
+          rpy="0 0 0" />
+        <mass
+          value="0.0622996894008648" />
+        <inertia
+          ixx="0.000123327723316811"
+          ixy="-1.34450244791909E-10"
+          ixz="-5.84363068828124E-06"
+          iyy="0.000126724002658958"
+          iyz="1.56255677980962E-10"
+          izz="1.60491252999105E-05" />
+      </inertial>
+      <visual>
+        <origin
+          xyz="0 0 0"
+          rpy="0 0 0" />
+        <geometry>
+          <mesh
+            filename="package://robot_description/meshes/GripperP/Dedo1.STL" />
+        </geometry>
+        <material
+          name="">
+          <color
+            rgba="0.792156862745098 0.819607843137255 0.933333333333333 1" />
+        </material>
+      </visual>
+      <collision>
+        <origin
+          xyz="0 0 0"
+          rpy="0 0 0" />
+        <geometry>
+          <mesh
+            filename="package://robot_description/meshes/GripperP/Dedo1.STL" />
+        </geometry>
+      </collision>
+    </link>
+    <joint
+      name="Fix1Dedo"
+      type="fixed">
+      <origin
+        xyz="-0.0685 -0.035 -0.0342"
+        rpy="-1.5708 0 -1.5708" />
+      <parent
+        link="Servo1" />
+      <child
+        link="Dedo1" />
+      <axis
+        xyz="0 0 0" />
+    </joint>
+    <link
+      name="Servo2">
+      <inertial>
+        <origin
+          xyz="0.0186297249994028 -4.50497350534818E-08 -0.0319399514116179"
+          rpy="0 0 0" />
+        <mass
+          value="0.0250047254852252" />
+        <inertia
+          ixx="1.22463749616552E-05"
+          ixy="-1.65063023348749E-19"
+          ixz="-1.80956359903934E-06"
+          iyy="1.36408467918994E-05"
+          iyz="1.57491079497996E-19"
+          izz="3.54946158391805E-06" />
+      </inertial>
+      <visual>
+        <origin
+          xyz="0 0 0"
+          rpy="0 0 0" />
+        <geometry>
+          <mesh
+            filename="package://robot_description/meshes/GripperP/Servo2.STL" />
+        </geometry>
+        <material
+          name="">
+          <color
+            rgba="0.792156862745098 0.819607843137255 0.933333333333333 1" />
+        </material>
+      </visual>
+      <collision>
+        <origin
+          xyz="0 0 0"
+          rpy="0 0 0" />
+        <geometry>
+          <mesh
+            filename="package://robot_description/meshes/GripperP/Servo2.STL" />
+        </geometry>
+      </collision>
+    </link>
+    <joint
+      name="Rev2Servo"
+      type="revolute">
+      <origin
+        xyz="0.056595 -0.035167 0.069142"
+        rpy="0 0 0" />
+      <parent
+        link="Base_Gripper" />
+      <child
+        link="Servo2" />
+      <axis
+        xyz="0 0 1" />
       <limit
         lower="-0.39"
         upper="0.02"
-        effort="0"
-        velocity="0" />
-    </joint>
-    <link
-      name="Dedo1">
-      <inertial>
-        <origin
-          xyz="-0.0339572900023838 -9.3618305648923E-08 0.148246675379403"
-          rpy="0 0 0" />
-        <mass
-          value="0.0622990489702351" />
-        <inertia
-          ixx="0.000123328183626577"
-          ixy="-1.22881098411723E-10"
-          ixz="-5.84361445598599E-06"
-          iyy="0.000126724273269253"
-          iyz="1.57270956526926E-10"
-          izz="1.60489416583839E-05" />
-      </inertial>
-      <visual>
-        <origin
-          xyz="0 0 0"
-          rpy="0 0 0" />
-        <geometry>
-          <mesh
-            filename="package://robot_description/meshes/Gripper/Dedo1.STL" />
-        </geometry>
-        <material
-          name="">
-          <color
-            rgba="0.792156862745098 0.819607843137255 0.933333333333333 1" />
-        </material>
-      </visual>
-      <collision>
-        <origin
-          xyz="0 0 0"
-          rpy="0 0 0" />
-        <geometry>
-          <mesh
-            filename="package://robot_description/meshes/Gripper/Dedo1.STL" />
-        </geometry>
-      </collision>
-    </link>
-    <joint
-      name="Fix1Dedo"
-      type="fixed">
-      <origin
-        xyz="0.035 0.0021425 -0.0685"
-        rpy="0 0 0" />
-      <parent
-        link="Servo1" />
-      <child
-        link="Dedo1" />
-      <axis
-        xyz="0 0 0" />
-    </joint>
-    <link
-      name="Servo2">
-      <inertial>
-        <origin
-          xyz="-4.50497350118484E-08 0.00440252858837639 0.0186297249994028"
-          rpy="0 0 0" />
-        <mass
-          value="0.0250047254852253" />
-        <inertia
-          ixx="1.36408467918995E-05"
-          ixy="1.66044927441445E-19"
-          ixz="-1.7205356741103E-19"
-          iyy="3.54946158391805E-06"
-          iyz="-1.80956359903932E-06"
-          izz="1.22463749616553E-05" />
-      </inertial>
-      <visual>
-        <origin
-          xyz="0 0 0"
-          rpy="0 0 0" />
-        <geometry>
-          <mesh
-            filename="package://robot_description/meshes/Gripper/Servo2.STL" />
-        </geometry>
-        <material
-          name="">
-          <color
-            rgba="0.792156862745098 0.819607843137255 0.933333333333333 1" />
-        </material>
-      </visual>
-      <collision>
-        <origin
-          xyz="0 0 0"
-          rpy="0 0 0" />
-        <geometry>
-          <mesh
-            filename="package://robot_description/meshes/Gripper/Servo2.STL" />
-        </geometry>
-      </collision>
-    </link>
-    <joint
-      name="Rev2Servo"
-      type="revolute">
-      <origin
-        xyz="0 -0.034832 0.088595"
-        rpy="0 -0.02 -1.5708" />
-      <parent
-        link="Base_Gripper" />
-      <child
-        link="Servo2" />
-      <axis
-        xyz="0 1 0" />
-      <limit
-        lower="-0.02"
-        upper="0.39"
         effort="0"
         velocity="0" />
@@ -237,37 +236,37 @@
       <inertial>
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