Commit message: update cam urdf

File: catkin_home/src/robot_description/urdf/dashgo.urdf.xacro (robot description, xacro)
@@ -457,203 +457,4 @@
       xyz="0 1 0" />
   </joint>
-  <link name="RevCam1">
-    <inertial>
-      <origin
-        xyz="-0.00218640043520604 0.0373778462346743 0.0578417163847615"
-        rpy="0 0 0" />
-      <mass
-        value="0.0807173231195892" />
-      <inertia
-        ixx="2.37796509107372E-05"
-        ixy="8.55528572510069E-07"
-        ixz="-2.49699440783422E-07"
-        iyy="1.83589761907289E-05"
-        iyz="-4.19202686542368E-06"
-        izz="2.27836700405391E-05" />
-    </inertial>
-    <visual>
-      <origin
-        xyz="0 0 0"
-        rpy="0 0 0" />
-      <geometry>
-        <mesh
-          filename="package://robot_description/meshes/Dashgo/RevCam1.STL" />
-      </geometry>
-      <material
-        name="">
-        <color
-          rgba="0.792156862745098 0.819607843137255 0.933333333333333 1" />
-      </material>
-    </visual>
-    <collision>
-      <origin
-        xyz="0 0 0"
-        rpy="0 0 0" />
-      <geometry>
-        <mesh
-          filename="package://robot_description/meshes/Dashgo/RevCam1.STL" />
-      </geometry>
-    </collision>
-  </link>
-  <!-- <joint name="Cam1X"
-    type="prismatic">
-    <origin
-      xyz="-0.16729 0.098455 1.546"
-      rpy="1.5708 0.0 0.13201" />
-    <parent
-      link="Base" />
-    <child
-      link="RevCam1" />
-    <axis
-      xyz="0 1 0" />
-    <limit
-      lower="-0.54"
-      upper="0.54"
-      effort="0"
-      velocity="0" />
-  <joint name="cam_y" type="prismatic">
-      <axis xyz="0 1 0" />
-      <parent link="cam" />
-      <child link="cam_yx_link" />
-      <limit effort="1" lower="0.0" upper="0.0" velocity="0.08" />
-      <dynamics damping="0.7" friction="2" />
-  </joint>
-  <link name="cam_yx_link">
-      <inertial>
-          <mass value="0.10" />
-          <inertia ixx="0.000729" ixy="0" ixz="0" iyy="0.000729" iyz="0" izz="0.000729" />
-      </inertial>
-  </link>
-  <joint name="cam_x" type="prismatic">
-      <axis xyz="1 0 0" />
-      <parent link="cam_y_link" />
-      <child link="cam_x_link" />
-      <limit effort="1" lower="-1.0" upper="1.0" velocity="0.08" />
-      <dynamics damping="0.7" friction="2" />
-  </joint> -->
-  <joint name="Cam1Rev1"
-    type="revolute">
-    <origin
-      xyz="-0.16729 0.098455 1.546"
-      rpy="1.5708 0.0 0.13201" />
-    <parent
-      link="Base" />
-    <child
-      link="RevCam1" />
-    <axis
-      xyz="0 1 0" />
-    <limit
-      lower="-0.54"
-      upper="0.54"
-      effort="0"
-      velocity="0" />
-  </joint>
-  <link name="RevCam2">
-    <inertial>
-      <origin
-        xyz="0.00149250457233677 -0.00361361108108715 0.0165031514881021"
-        rpy="0 0 0" />
-      <mass
-        value="0.0702746066702973" />
-      <inertia
-        ixx="3.32748236022629E-05"
-        ixy="5.65176745386308E-06"
-        ixz="-4.55903201425305E-06"
-        iyy="4.5252809651764E-05"
-        iyz="4.8432689106791E-06"
-        izz="4.86199055260646E-05" />
-    </inertial>
-    <visual>
-      <origin
-        xyz="0 0 0"
-        rpy="0 0 0" />
-      <geometry>
-        <mesh
-          filename="package://robot_description/meshes/Dashgo/RevCam2.STL" />
-      </geometry>
-      <material
-        name="">
-        <color
-          rgba="0.792156862745098 0.819607843137255 0.933333333333333 1" />
-      </material>
-    </visual>
-    <collision>
-      <origin
-        xyz="0 0 0"
-        rpy="0 0 0" />
-      <geometry>
-        <mesh
-          filename="package://robot_description/meshes/Dashgo/RevCam2.STL" />
-      </geometry>
-    </collision>
-  </link>
-  <joint name="Cam1Rev2"
-    type="revolute">
-    <origin
-      xyz="-0.0021558 0.0036505 0.085266"
-      rpy="-0.08 -0.13856 0.0010948" />
-    <parent
-      link="RevCam1" />
-    <child
-      link="RevCam2" />
-    <axis
-      xyz="1 0 0" />
-    <limit
-      lower="-0.54"
-      upper="0.54"
-      effort="0"
-      velocity="0" />
-  </joint>
-  <link name="Cam1">
-    <inertial>
-      <origin
-        xyz="-0.0161158990750312 -2.71397957091191E-06 8.43511749604176E-06"
-        rpy="0 0 0" />
-      <mass
-        value="0.152258301511643" />
-      <inertia
-        ixx="0.00037232470424964"
-        ixy="2.49919563850586E-09"
-        ixz="-3.15602915288441E-08"
-        iyy="2.28180071550079E-05"
-        iyz="6.18457007379358E-09"
-        izz="0.000374741909994746" />
-    </inertial>
-    <visual>
-      <origin
-        xyz="0 0 0"
-        rpy="0 0 0" />
-      <geometry>
-        <mesh
-          filename="package://robot_description/meshes/Dashgo/Cam1.STL" />
-      </geometry>
-      <material
-        name="">
-        <color
-          rgba="0.792156862745098 0.819607843137255 0.933333333333333 1" />
-      </material>
-    </visual>
-    <collision>
-      <origin
-        xyz="0 0 0"
-        rpy="0 0 0" />
-      <geometry>
-        <mesh
-          filename="package://robot_description/meshes/Dashgo/Cam1.STL" />
-      </geometry>
-    </collision>
-  </link>
-  <joint name="Cam1Fix"
-    type="fixed">
-    <origin
-      xyz="0.0012272 -0.035179 0.037568"
-      rpy="-0.0081734 -0.62147 -1.566" />
-    <parent
-      link="RevCam2" />
-    <child
-      link="Cam1" />
-    <axis
-      xyz="0 0 0" />
-  </joint>
   <link name="BaseBrazo">
     <inertial>
@@ -704,162 +505,4 @@
     <child
       link="BaseBrazo" />
-    <axis
-      xyz="0 0 0" />
-  </joint>
-  <link name="Cam2Rev">
-    <inertial>
-      <origin
-        xyz="0.00682983624522909 -0.000385587206922666 -0.0349999920861893"
-        rpy="0 0 0" />
-      <mass
-        value="0.0348111598620482" />
-      <inertia
-        ixx="2.55962147675482E-05"
-        ixy="-2.5718115731198E-08"
-        ixz="-1.41168757122553E-12"
-        iyy="2.69229988150616E-05"
-        iyz="-3.22321270093433E-12"
-        izz="1.54258242876257E-05" />
-    </inertial>
-    <visual>
-      <origin
-        xyz="0 0 0"
-        rpy="0 0 0" />
-      <geometry>
-        <mesh
-          filename="package://robot_description/meshes/Dashgo/Cam2Rev.STL" />
-      </geometry>
-      <material
-        name="">
-        <color
-          rgba="0.792156862745098 0.819607843137255 0.933333333333333 1" />
-      </material>
-    </visual>
-    <collision>
-      <origin
-        xyz="0 0 0"
-        rpy="0 0 0" />
-      <geometry>
-        <mesh
-          filename="package://robot_description/meshes/Dashgo/Cam2Rev.STL" />
-      </geometry>
-    </collision>
-  </link>
-  <joint name="Cam2Rev"
-    type="revolute">
-    <origin
-      xyz="-0.0475 -0.16539 0.50877"
-      rpy="-1.5708 1.1309 -1.5708" />
-    <parent
-      link="Base" />
-    <child
-      link="Cam2Rev" />
-    <axis
-      xyz="0 0 1" />
-    <limit
-      lower="-0.5236"
-      upper="0.5236"
-      effort="0"
-      velocity="0" />
-  </joint>
-  <link name="Cam2">
-    <inertial>
-      <origin
-        xyz="-0.0161159159322545 -2.67749700753883E-06 8.41275410029541E-06"
-        rpy="0 0 0" />
-      <mass
-        value="0.152258232607803" />
-      <inertia
-        ixx="0.000372324819517498"
-        ixy="2.56638565002235E-09"
-        ixz="-3.15448631037864E-08"
-        iyy="2.28182500829627E-05"
-        iyz="6.19441632492445E-09"
-        izz="0.000374741789457093" />
-    </inertial>
-    <visual>
-      <origin
-        xyz="0 0 0"
-        rpy="0 0 0" />
-      <geometry>
-        <mesh
-          filename="package://robot_description/meshes/Dashgo/Cam2.STL" />
-      </geometry>
-      <material
-        name="">
-        <color
-          rgba="0.792156862745098 0.819607843137255 0.933333333333333 1" />
-      </material>
-    </visual>
-    <collision>
-      <origin
-        xyz="0 0 0"
-        rpy="0 0 0" />
-      <geometry>
-        <mesh
-          filename="package://robot_description/meshes/Dashgo/Cam2.STL" />
-      </geometry>
-    </collision>
-  </link>
-  <joint name="Cam2Fixed"
-    type="fixed">
-    <origin
-      xyz="0.034026 0.0014743 -0.035"
-      rpy="1.5708 0 0.032661" />
-    <parent
-      link="Cam2Rev" />
-    <child
-      link="Cam2" />
-    <axis
-      xyz="0 0 0" />
-  </joint>
-  <link name="Cam3">
-    <inertial>
-      <origin
-        xyz="-0.0161158990646986 -2.71398471196616E-06 8.43515159343333E-06"
-        rpy="0 0 0" />
-      <mass
-        value="0.15225830141293" />
-      <inertia
-        ixx="0.000372324703580476"
-        ixy="2.49921630269361E-09"
-        ixz="-3.15603379522398E-08"
-        iyy="2.28180071728585E-05"
-        iyz="6.18490198100671E-09"
-        izz="0.000374741909293992" />
-    </inertial>
-    <visual>
-      <origin
-        xyz="0 0 0"
-        rpy="0 0 0" />
-      <geometry>
-        <mesh
-          filename="package://robot_description/meshes/Dashgo/Cam3.STL" />
-      </geometry>
-      <material
-        name="">
-        <color
-          rgba="0.792156862745098 0.819607843137255 0.933333333333333 1" />
-      </material>
-    </visual>
-    <collision>
-      <origin
-        xyz="0 0 0"
-        rpy="0 0 0" />
-      <geometry>
-        <mesh
-          filename="package://robot_description/meshes/Dashgo/Cam3.STL" />
-      </geometry>
-    </collision>
-  </link>
-  <joint name="Cam3Fix"
-    type="fixed">
-    <origin
-      xyz="-0.159 0.063143 1.5387"
-      rpy="0 0.7854 -1.5708" />
-    <parent
-      link="Base" />
-    <child
-      link="Cam3" />
     <axis
       xyz="0 0 0" />
@@ -902,3 +545,61 @@
   <!-- <xacro:load_gripper attach_to="$(arg prefix)link_eef" xyz="0 0 0.003" rpy="0 0 1.57" /> -->
   <xacro:load_gripperP attach_to="$(arg prefix)link_eef" xyz="0 0 0.003" rpy="0 0 1.57" />
+  <!-- Cameras -->
+  <!-- <link name="Cam3">
+    <inertial>
+      <origin
+        xyz="-0.0161158990646986 -2.71398471196616E-06 8.43515159343333E-06"
+        rpy="0 0 0" />
+      <mass
+        value="0.15225830141293" />
+      <inertia
+        ixx="0.000372324703580476"
+        ixy="2.49921630269361E-09"
+        ixz="-3.15603379522398E-08"
+        iyy="2.28180071728585E-05"
+        iyz="6.18490198100671E-09"
+        izz="0.000374741909293992" />
+    </inertial>
+    <visual>
+      <origin
+        xyz="0 0 0"
+        rpy="0 0 0" />
+      <geometry>
+        <mesh
+          filename="package://robot_description/meshes/Dashgo/Cam3.STL" />
+      </geometry>
+      <material
+        name="">
+        <color
+          rgba="0.792156862745098 0.819607843137255 0.933333333333333 1" />
+      </material>
+    </visual>
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
Commit message: carry my luggage WIP, human analyzer

File: catkin_home/src/robot_description/urdf/dashgo.urdf.xacro (robot description, xacro)
@@ -545,61 +545,10 @@
   <!-- <xacro:load_gripper attach_to="$(arg prefix)link_eef" xyz="0 0 0.003" rpy="0 0 1.57" /> -->
   <xacro:load_gripperP attach_to="$(arg prefix)link_eef" xyz="0 0 0.003" rpy="0 0 1.57" />
-  <!-- Cameras -->
-  <!-- <link name="Cam3">
-    <inertial>
-      <origin
-        xyz="-0.0161158990646986 -2.71398471196616E-06 8.43515159343333E-06"
-        rpy="0 0 0" />
-      <mass
-        value="0.15225830141293" />
-      <inertia
-        ixx="0.000372324703580476"
-        ixy="2.49921630269361E-09"
-        ixz="-3.15603379522398E-08"
-        iyy="2.28180071728585E-05"
-        iyz="6.18490198100671E-09"
-        izz="0.000374741909293992" />
-    </inertial>
-    <visual>
-      <origin
-        xyz="0 0 0"
-        rpy="0 0 0" />
-      <geometry>
-        <mesh
-          filename="package://robot_description/meshes/Dashgo/Cam3.STL" />
-      </geometry>
-      <material
-        name="">
-        <color
-          rgba="0.792156862745098 0.819607843137255 0.933333333333333 1" />
-      </material>
-    </visual>
-    <collision>
-      <origin
-        xyz="0 0 0"
-        rpy="0 0 0" />
-      <geometry>
-        <mesh
-          filename="package://robot_description/meshes/Dashgo/Cam3.STL" />
-      </geometry>
-    </collision>
-  </link>
-  <joint name="Cam3Fix"
-    type="fixed">
-    <origin
-      xyz="-0.159 0.063143 1.5387"
-      rpy="0 0.7854 -1.5708" />
-    <parent
-      link="Base" />
-    <child
-      link="Cam3" />
-    <axis
-      xyz="0 0 0" />
-  </joint>
-   -->
   <xacro:include filename="$(find robot_description)/urdf/camera.urdf.xacro" />
   <!-- <xacro:load_camera name="Cam1" attach_to="Base" x="-0.159" y="0.063143" z="1.56" r_r="0.174533" r_p="0" r_y="-1.5708" />
   <xacro:load_camera name="Cam2" attach_to="Base" x="-0.085" y="-0.27" z="0.51" r_r="0.698132" r_p="0" r_y="-1.5708" /> -->
-  <xacro:load_camera name="Cam1" attach_to="Base" x="-0.159" y="-0.01" z="1.57" r_r="0.244533" r_p="0" r_y="-1.5708" />
-  <xacro:load_camera name="Cam2" attach_to="Base" x="-0.085" y="-0.27" z="0.48" r_r="0.538132" r_p="0" r_y="-1.5708" />
+  <xacro:load_camera name="Cam1" attach_to="Base" x="-0.25" y="-0.17" z="1.57" r_r="0.224533" r_p="0" r_y="-1.5708" />
+  <xacro:load_camera name="Cam2" attach_to="Base" x="-0.085" y="-0.24" z="0.48" r_r="0.538132" r_p="0" r_y="-1.5708" />
+  <!-- <xacro:load_camera name="Cam1" attach_to="base_link" x="0.02" y="0.0" z="1.57" r_r="0" r_p="0.224533" r_y="0" />
+  <xacro:load_camera name="Cam2" attach_to="base_link" x="0.185" y="0.2" z="0.48" r_r="0" r_p="0.538132" r_y="0" /> -->
 </robot>

Commit message: cary my luggage v1, remove base_controller

File: catkin_home/src/robot_description/urdf/dashgo.urdf.xacro (robot description, xacro)
@@ -4,55 +4,11 @@
      For more information, please see http://wiki.ros.org/sw_urdf_exporter -->
 <robot xmlns:xacro="http://ros.org/wiki/xacro" name="dashgo">
-  <virtual_joint child_link="internal_odom" name="world_joint" parent_frame="odom" type="planar" />
-  <!-- ############################BASE_MOVEMENT############################## -->
-  <link name="internal_odom" />
-  <joint name="internal_odom_joint" type="fixed">
-      <origin rpy="0 0 0" xyz="0 0 0" />
-      <parent link="internal_odom" />
-      <child link="internal_odom_inertia" />
-  </joint>
-  <link name="internal_odom_inertia">
-      <inertial>
-          <mass value="0.10" />
-          <!--  assume as square, hence inertia = (1/12) * m * (a^2 + b^2)  -->
-          <inertia ixx="0.000729" ixy="0" ixz="0" iyy="0.000729" iyz="0" izz="0.000729" />
-      </inertial>
-  </link>
-  <joint name="odom_y" type="prismatic">
-      <axis xyz="0 1 0" />
-      <parent link="internal_odom_inertia" />
-      <child link="odom_yx_link" />
-      <limit effort="1" lower="0.0" upper="0.0" velocity="0.08" />
-      <dynamics damping="0.7" friction="2" />
-  </joint>
-  <link name="odom_yx_link">
-      <inertial>
-          <mass value="0.10" />
-          <!--  assume as square, hence inertia = (1/12) * m * (a^2 + b^2)  -->
-          <inertia ixx="0.000729" ixy="0" ixz="0" iyy="0.000729" iyz="0" izz="0.000729" />
-      </inertial>
-  </link>
-  <joint name="odom_x" type="prismatic">
-      <axis xyz="1 0 0" />
-      <parent link="odom_yx_link" />
-      <child link="odom_xr_link" />
-      <limit effort="1" lower="-1.0" upper="1.0" velocity="0.08" />
-      <dynamics damping="0.7" friction="2" />
-  </joint>
-  <link name="odom_xr_link">
-      <inertial>
-          <mass value="0.10" />
-          <!--  assume as square, hence inertia = (1/12) * m * (a^2 + b^2)  -->
-          <inertia ixx="0.000729" ixy="0" ixz="0" iyy="0.000729" iyz="0" izz="0.000729" />
-      </inertial>
-  </link>
-  <joint name="odom_r" type="revolute">
-      <axis xyz="0 0 1" />
-      <parent link="odom_xr_link" />
-      <child link="base_link" />
-      <limit effort="1" lower="0" upper="0" velocity="0.18" />
-      <dynamics damping="0.7" friction="2" />
-  </joint>
-  <!-- ########################################################################### -->
+  <virtual_joint child_link="base_footprint" name="world_joint" parent_frame="odom" type="planar" />
+  <link name="base_footprint"></link>
+  <joint name="base_joint_1" type="fixed">
+    <origin xyz="0.11 0 0" rpy="0 0 0"/>
+    <parent link="base_footprint"/>
+    <child link="base_link"/>
+  </joint>
   <link name="base_link"></link>
   <joint name="base_joint" type="fixed">
@@ -544,5 +500,5 @@
   <xacro:include filename="$(find robot_description)/urdf/gripper/gripperP.urdf.xacro" />
   <!-- <xacro:load_gripper attach_to="$(arg prefix)link_eef" xyz="0 0 0.003" rpy="0 0 1.57" /> -->
-  <xacro:load_gripperP attach_to="$(arg prefix)link_eef" xyz="0 0 0.003" rpy="0 0 1.57" />
+  <xacro:load_gripper attach_to="$(arg prefix)link_eef" xyz="0 0 0.003" rpy="0 0 1.57" />
   <xacro:include filename="$(find robot_description)/urdf/camera.urdf.xacro" />
   <!-- <xacro:load_camera name="Cam1" attach_to="Base" x="-0.159" y="0.063143" z="1.56" r_r="0.174533" r_p="0" r_y="-1.5708" />
