Commit message: add gripper fake sf, remove unused robot_description pkg

File: catkin_home/src/robot_description/urdf/dashgo.urdf.xacro (robot description, xacro)
@@ -1,56 +1,42 @@
-<?xml version="1.0" encoding="utf-8"?>
-<!-- This URDF was automatically created by SolidWorks to URDF Exporter! Originally created by Stephen Brawner (brawner@gmail.com)
-     Commit Version: 1.6.0-4-g7f85cfe  Build Version: 1.6.7995.38578
-     For more information, please see http://wiki.ros.org/sw_urdf_exporter -->
+<?xml version='1.0' encoding='utf-8'?>
 <robot xmlns:xacro="http://ros.org/wiki/xacro" name="dashgo">
   <virtual_joint child_link="base_footprint" name="world_joint" parent_frame="odom" type="planar" />
-  <link name="base_footprint"></link>
-  <joint name="base_joint_1" type="fixed">
-    <origin xyz="0.11 0 0" rpy="0 0 0"/>
-    <parent link="base_footprint"/>
-    <child link="base_link"/>
-  </joint>
-  <link name="base_link"></link>
-  <joint name="base_joint" type="fixed">
-    <origin xyz="0 0 0" rpy="0 0 1.57"/>
-    <parent link="base_link"/>
-    <child link="Base"/>
+  <link name="base_footprint" />
+  <joint name="base_footprint_joint" type="fixed">
+    <origin xyz="0 0 0" rpy="0 0 0" />
+    <parent link="base_footprint" />
+    <child link="base_link" />
+  </joint>
+  <link name="base_link" />
+  <joint name="base_link_joint" type="fixed">
+    <origin xyz="0 0 0" rpy="0 0 0" />
+    <parent link="base_link" />
+    <child link="Base" />
+  </joint>
+  <link name="apriltag" />
+  <joint name="apriltag_joint" type="fixed">
+    <origin xyz="0.11625 0.03758 0" rpy="0 -1.57 3.1416" />
+    <parent link="link4" />
+    <child link="apriltag" />
   </joint>
   <link name="Base">
     <inertial>
-      <origin
-        xyz="-0.0421641375528847 0.0262460783517876 0.278949374295985"
-        rpy="0 0 0" />
-      <mass
-        value="26.7355250620724" />
-      <inertia
-        ixx="0.418467609556011"
-        ixy="0.0235787657447133"
-        ixz="8.3665476036404E-06"
-        iyy="0.302793463787765"
-        iyz="0.000125414849304393"
-        izz="0.482705153704045" />
-    </inertial>
-    <visual>
-      <origin
-        xyz="0 0 0"
-        rpy="0 0 0" />
-      <geometry>
-        <mesh
-          filename="package://robot_description/meshes/Dashgo/Base.STL" />
-      </geometry>
-      <material
-        name="">
-        <color
-          rgba="0.792156862745098 0.819607843137255 0.933333333333333 1" />
-      </material>
-    </visual>
-    <collision>
-      <origin
-        xyz="0 0 0"
-        rpy="0 0 0" />
-      <geometry>
-        <mesh
-          filename="package://robot_description/meshes/Dashgo/Base_Collisions.STL" />
+      <origin xyz="-0.0421641375528847 0.0262460783517876 0.278949374295985" rpy="0 0 0" />
+      <mass value="26.7355250620724" />
+      <inertia ixx="0.418467609556011" ixy="0.0235787657447133" ixz="8.3665476036404E-06" iyy="0.302793463787765" iyz="0.000125414849304393" izz="0.482705153704045" />
+    </inertial>
+    <visual>
+      <origin xyz="0 0 0" rpy="0 0 0" />
+      <geometry>
+        <mesh filename="package://robot_description/meshes/Dashgo/Base.STL" />
+      </geometry>
+      <material name="">
+        <color rgba="0.792156862745098 0.819607843137255 0.933333333333333 1" />
+      </material>
+    </visual>
+    <collision>
+      <origin xyz="0 0 0" rpy="0 0 0" />
+      <geometry>
+        <mesh filename="package://robot_description/meshes/Dashgo/Base_Collisions.STL" />
       </geometry>
     </collision>
@@ -58,453 +44,253 @@
   <link name="Llanta1">
     <inertial>
-      <origin
-        xyz="4.02455846426619E-16 6.59194920871187E-16 0.0200000000000003"
-        rpy="0 0 0" />
-      <mass
-        value="0.528918539158378" />
-      <inertia
-        ixx="0.000631308353030454"
-        ixy="-1.64320882748444E-36"
-        ixz="1.72050413075699E-18"
-        iyy="0.000631308353030454"
-        iyz="-1.31827511759964E-36"
-        izz="0.00112157176228534" />
-    </inertial>
-    <visual>
-      <origin
-        xyz="0 0 0"
-        rpy="0 0 0" />
-      <geometry>
-        <mesh
-          filename="package://robot_description/meshes/Dashgo/Llanta1.STL" />
-      </geometry>
-      <material
-        name="">
-        <color
-          rgba="0.792156862745098 0.819607843137255 0.933333333333333 1" />
-      </material>
-    </visual>
-    <collision>
-      <origin
-        xyz="0 0 0"
-        rpy="0 0 0" />
-      <geometry>
-        <mesh
-          filename="package://robot_description/meshes/Dashgo/Llanta1.STL" />
-      </geometry>
-    </collision>
-  </link>
-  <joint name="Llanta1Cont"
-    type="continuous">
-    <origin
-      xyz="0.146 0.1155 0.0375"
-      rpy="1.5708 0 1.5708" />
-    <parent
-      link="Base" />
-    <child
-      link="Llanta1" />
-    <axis
-      xyz="0 0 1" />
+      <origin xyz="4.02455846426619E-16 6.59194920871187E-16 0.0200000000000003" rpy="0 0 0" />
+      <mass value="0.528918539158378" />
+      <inertia ixx="0.000631308353030454" ixy="-1.64320882748444E-36" ixz="1.72050413075699E-18" iyy="0.000631308353030454" iyz="-1.31827511759964E-36" izz="0.00112157176228534" />
+    </inertial>
+    <visual>
+      <origin xyz="0 0 0" rpy="0 0 0" />
+      <geometry>
+        <mesh filename="package://robot_description/meshes/Dashgo/Llanta1.STL" />
+      </geometry>
+      <material name="">
+        <color rgba="0.792156862745098 0.819607843137255 0.933333333333333 1" />
+      </material>
+    </visual>
+    <collision>
+      <origin xyz="0 0 0" rpy="0 0 0" />
+      <geometry>
+        <mesh filename="package://robot_description/meshes/Dashgo/Llanta1.STL" />
+      </geometry>
+    </collision>
+  </link>
+  <joint name="Llanta1Cont" type="continuous">
+    <origin xyz="0.146 0.1155 0.0375" rpy="1.5708 0 1.5708" />
+    <parent link="Base" />
+    <child link="Llanta1" />
+    <axis xyz="0 0 1" />
   </joint>
   <link name="Llanta2">
     <inertial>
-      <origin
-        xyz="-1.38777878078145E-17 -1.11022302462516E-16 -0.02"
-        rpy="0 0 0" />
-      <mass
-        value="0.528918539158378" />
-      <inertia
-        ixx="0.000631308353030454"
-        ixy="-8.470329472543E-22"
-        ixz="-9.10263751530836E-20"
-        iyy="0.000631308353030454"
-        iyz="4.50857846912387E-20"
-        izz="0.00112157176228534" />
-    </inertial>
-    <visual>
-      <origin
-        xyz="0 0 0"
-        rpy="0 0 0" />
-      <geometry>
-        <mesh
-          filename="package://robot_description/meshes/Dashgo/Llanta2.STL" />
-      </geometry>
-      <material
-        name="">
-        <color
-          rgba="0.792156862745098 0.819607843137255 0.933333333333333 1" />
-      </material>
-    </visual>
-    <collision>
-      <origin
-        xyz="0 0 0"
-        rpy="0 0 0" />
-      <geometry>
-        <mesh
-          filename="package://robot_description/meshes/Dashgo/Llanta2.STL" />
-      </geometry>
-    </collision>
-  </link>
-  <joint name="Llanta2Cont"
-    type="continuous">
-    <origin
-      xyz="-0.146 0.1155 0.0375"
-      rpy="1.5708 0.020949 1.5708" />
-    <parent
-      link="Base" />
-    <child
-      link="Llanta2" />
-    <axis
-      xyz="0 0 1" />
+      <origin xyz="-1.38777878078145E-17 -1.11022302462516E-16 -0.02" rpy="0 0 0" />
+      <mass value="0.528918539158378" />
+      <inertia ixx="0.000631308353030454" ixy="-8.470329472543E-22" ixz="-9.10263751530836E-20" iyy="0.000631308353030454" iyz="4.50857846912387E-20" izz="0.00112157176228534" />
+    </inertial>
+    <visual>
+      <origin xyz="0 0 0" rpy="0 0 0" />
+      <geometry>
+        <mesh filename="package://robot_description/meshes/Dashgo/Llanta2.STL" />
+      </geometry>
+      <material name="">
+        <color rgba="0.792156862745098 0.819607843137255 0.933333333333333 1" />
+      </material>
+    </visual>
+    <collision>
+      <origin xyz="0 0 0" rpy="0 0 0" />
+      <geometry>
+        <mesh filename="package://robot_description/meshes/Dashgo/Llanta2.STL" />
+      </geometry>
+    </collision>
+  </link>
+  <joint name="Llanta2Cont" type="continuous">
+    <origin xyz="-0.146 0.1155 0.0375" rpy="1.5708 0.020949 1.5708" />
+    <parent link="Base" />
+    <child link="Llanta2" />
+    <axis xyz="0 0 1" />
   </joint>
   <link name="Loca1">
     <inertial>
-      <origin
-        xyz="0 0.0345546529721542 -2.77555756156289E-17"
-        rpy="0 0 0" />
-      <mass
-        value="0.0167352759899297" />
-      <inertia
-        ixx="7.54150196205056E-06"
-        ixy="1.29419148906084E-21"
-        ixz="-8.52898332671465E-22"
-        iyy="5.85653067123054E-06"
-        iyz="-1.78257050125666E-21"
-        izz="7.09027556219276E-06" />
-    </inertial>
-    <visual>
-      <origin
-        xyz="0 0 0"
-        rpy="0 0 0" />
-      <geometry>
-        <mesh
-          filename="package://robot_description/meshes/Dashgo/Loca1.STL" />
-      </geometry>
-      <material
-        name="">
-        <color
-          rgba="0.792156862745098 0.819607843137255 0.933333333333333 1" />
-      </material>
-    </visual>
-    <collision>
-      <origin
-        xyz="0 0 0"
-        rpy="0 0 0" />
-      <geometry>
-        <mesh
-          filename="package://robot_description/meshes/Dashgo/Loca1.STL" />
-      </geometry>
-    </collision>
-  </link>
-  <joint name="Loca1Cont"
-    type="continuous">
-    <origin
-      xyz="-0.09 -0.072 0"
-      rpy="1.5708 0 0" />
-    <parent
-      link="Base" />
-    <child
-      link="Loca1" />
-    <axis
-      xyz="0 1 0" />
+      <origin xyz="0 0.0345546529721542 -2.77555756156289E-17" rpy="0 0 0" />
+      <mass value="0.0167352759899297" />
+      <inertia ixx="7.54150196205056E-06" ixy="1.29419148906084E-21" ixz="-8.52898332671465E-22" iyy="5.85653067123054E-06" iyz="-1.78257050125666E-21" izz="7.09027556219276E-06" />
+    </inertial>
+    <visual>
+      <origin xyz="0 0 0" rpy="0 0 0" />
+      <geometry>
+        <mesh filename="package://robot_description/meshes/Dashgo/Loca1.STL" />
+      </geometry>
+      <material name="">
+        <color rgba="0.792156862745098 0.819607843137255 0.933333333333333 1" />
+      </material>
+    </visual>
+    <collision>
+      <origin xyz="0 0 0" rpy="0 0 0" />
+      <geometry>
+        <mesh filename="package://robot_description/meshes/Dashgo/Loca1.STL" />
+      </geometry>
+    </collision>
+  </link>
+  <joint name="Loca1Cont" type="continuous">
+    <origin xyz="-0.09 -0.072 0" rpy="1.5708 0 0" />
+    <parent link="Base" />
+    <child link="Loca1" />
+    <axis xyz="0 1 0" />
   </joint>
   <link name="LlantaLoca1">
     <inertial>
-      <origin
-        xyz="1.38777878078145E-17 -0.00741632050454701 1.38777878078145E-17"
-        rpy="0 0 0" />
-      <mass
-        value="0.0694291976443344" />
-      <inertia
-        ixx="3.17985725211052E-05"
-        ixy="-5.21349495168481E-38"
-        ixz="3.52930394689292E-22"
-        iyy="1.95153903045283E-05"
-        iyz="7.67877008722515E-41"
-        izz="1.95153903045283E-05" />
-    </inertial>
-    <visual>
-      <origin
-        xyz="0 0 0"
-        rpy="0 0 0" />
-      <geometry>
-        <mesh
-          filename="package://robot_description/meshes/Dashgo/LlantaLoca1.STL" />
-      </geometry>
-      <material
-        name="">
-        <color
-          rgba="0.792156862745098 0.819607843137255 0.933333333333333 1" />
-      </material>
-    </visual>
-    <collision>
-      <origin
-        xyz="0 0 0"
-        rpy="0 0 0" />
-      <geometry>
-        <mesh
-          filename="package://robot_description/meshes/Dashgo/LlantaLoca1.STL" />
-      </geometry>
-    </collision>
-  </link>
-  <joint name="LlantaLoca1Cont"
-    type="continuous">
-    <origin
-      xyz="0 0.01 0"
-      rpy="0 0 0" />
-    <parent
-      link="Loca1" />
-    <child
-      link="LlantaLoca1" />
-    <axis
-      xyz="1 0 0" />
+      <origin xyz="1.38777878078145E-17 -0.00741632050454701 1.38777878078145E-17" rpy="0 0 0" />
+      <mass value="0.0694291976443344" />
+      <inertia ixx="3.17985725211052E-05" ixy="-5.21349495168481E-38" ixz="3.52930394689292E-22" iyy="1.95153903045283E-05" iyz="7.67877008722515E-41" izz="1.95153903045283E-05" />
+    </inertial>
+    <visual>
+      <origin xyz="0 0 0" rpy="0 0 0" />
+      <geometry>
+        <mesh filename="package://robot_description/meshes/Dashgo/LlantaLoca1.STL" />
+      </geometry>
+      <material name="">
+        <color rgba="0.792156862745098 0.819607843137255 0.933333333333333 1" />
+      </material>
+    </visual>
+    <collision>
+      <origin xyz="0 0 0" rpy="0 0 0" />
+      <geometry>
+        <mesh filename="package://robot_description/meshes/Dashgo/LlantaLoca1.STL" />
+      </geometry>
+    </collision>
+  </link>
+  <joint name="LlantaLoca1Cont" type="continuous">
+    <origin xyz="0 0.01 0" rpy="0 0 0" />
+    <parent link="Loca1" />
+    <child link="LlantaLoca1" />
+    <axis xyz="1 0 0" />
   </joint>
   <link name="Loca2">
     <inertial>
-      <origin
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