Commit message: add gripper fake sf, remove unused robot_description pkg

File: catkin_home/src/robot_description/urdf/gripper/gripperFakeSF.urdf.xacro (robot description, xacro)
@@ -4,5 +4,5 @@
      For more information, please see http://wiki.ros.org/sw_urdf_exporter -->
 <robot xmlns:xacro="http://ros.org/wiki/xacro" name="Gripper">
-  <xacro:macro name="load_gripper" params="attach_to:='' xyz:='0 0 0' rpy:='0 0 0'">
+  <xacro:macro name="load_gripperFakeSF" params="attach_to:='' xyz:='0 0 0' rpy:='0 0 0'">
     <xacro:unless value="${attach_to == ''}">
       <joint name="gripper_fix" type="fixed">
@@ -12,41 +12,40 @@
       </joint>
     </xacro:unless>
-    <link
-      name="Base_Gripper">
-      <inertial>
-        <origin
-          xyz="-0.0060074 0.00022945 0.055534"
-          rpy="0 0 0" />
-        <mass
-          value="0.25675" />
-        <inertia
-          ixx="0.00029732"
-          ixy="5.577E-07"
-          ixz="6.8196E-06"
-          iyy="0.0001154"
-          iyz="-6.3991E-07"
-          izz="0.00028425" />
-      </inertial>
-      <visual>
-        <origin
-          xyz="0 0 0"
-          rpy="0 0 0" />
-        <geometry>
-          <mesh
-            filename="package://robot_description/meshes/Gripper/Base.STL" />
-        </geometry>
-        <material
-          name="">
-          <color
-            rgba="0.79216 0.81961 0.93333 1" />
-        </material>
-      </visual>
-      <collision>
-        <origin
-          xyz="0 0 0"
-          rpy="0 0 0" />
-        <geometry>
-          <mesh
-            filename="package://robot_description/meshes/Gripper/Base.STL" />
+    <link name="Base_Gripper">
+      <inertial>
+        <origin
+          xyz="-0.00600744878247479 0.000229447019284631 0.0275811003234641"
+          rpy="0 0 0" />
+        <mass
+          value="0.25675298967361" />
+        <inertia
+          ixx="0.000297324022723542"
+          ixy="5.57701217289319E-07"
+          ixz="6.8196059580779E-06"
+          iyy="0.000115396784513201"
+          iyz="-6.39913613193201E-07"
+          izz="0.000284254818153183" />
+      </inertial>
+      <visual>
+        <origin
+          xyz="0 0 0"
+          rpy="0 0 0" />
+        <geometry>
+          <mesh
+            filename="package://robot_description/meshes/GripperFakeSF/Base_Gripper.STL" />
+        </geometry>
+        <material
+          name="">
+          <color
+            rgba="0.792156862745098 0.819607843137255 0.933333333333333 1" />
+        </material>
+      </visual>
+      <collision>
+        <origin
+          xyz="0 0 0"
+          rpy="0 0 0" />
+        <geometry>
+          <mesh
+            filename="package://robot_description/meshes/GripperFakeSF/Base_Gripper.STL" />
         </geometry>
       </collision>
@@ -57,20 +56,19 @@
       <parent link="Base_Gripper" />
       <child link="end_effector_link" />
-      <origin xyz="0 0 0.165" rpy="0 -1.57 0" />
-    </joint>
-    <link
-      name="Servo1">
-      <inertial>
-        <origin
-          xyz="-4.50497350326651E-08 0.00440252858837619 0.0186297249994029"
-          rpy="0 0 0" />
-        <mass
-          value="0.0250047254852256" />
+      <origin xyz="0.0 -0.14 0" rpy="1.57 0 -1.57" />
+    </joint>
+    <link name="Servo1">
+      <inertial>
+        <origin
+          xyz="-4.50497350465429E-08 0.00440252858837645 0.0186297249994028"
+          rpy="0 0 0" />
+        <mass
+          value="0.0250047254852253" />
         <inertia
           ixx="1.36408467918995E-05"
-          ixy="1.57759886426113E-19"
-          ixz="-1.71524171818996E-19"
-          iyy="3.54946158391808E-06"
-          iyz="-1.80956359903929E-06"
+          ixy="1.57389452627317E-19"
+          ixz="-1.65284737063933E-19"
+          iyy="3.54946158391806E-06"
+          iyz="-1.80956359903934E-06"
           izz="1.22463749616553E-05" />
       </inertial>
@@ -81,29 +79,26 @@
         <geometry>
           <mesh
-            filename="package://robot_description/meshes/Gripper/Servo1.STL" />
-        </geometry>
-        <material
-          name="">
-          <color
-            rgba="0.792156862745098 0.819607843137255 0.933333333333333 1" />
-        </material>
-      </visual>
-      <collision>
-        <origin
-          xyz="0 0 0"
-          rpy="0 0 0" />
-        <geometry>
-          <mesh
-            filename="package://robot_description/meshes/Gripper/Servo1.STL" />
-        </geometry>
-      </collision>
-    </link>
-    <joint
-      name="Rev1Servo"
-      type="revolute">
-      <origin
-        xyz="0 0.035167 0.088595"
-        rpy="0 -0.01 -1.5708" />
-        <!-- 0.35 -->
+            filename="package://robot_description/meshes/GripperFakeSF/Servo1.STL" />
+        </geometry>
+        <material
+          name="">
+          <color
+            rgba="0.792156862745098 0.819607843137255 0.933333333333333 1" />
+        </material>
+      </visual>
+      <collision>
+        <origin
+          xyz="0 0 0"
+          rpy="0 0 0" />
+        <geometry>
+          <mesh
+            filename="package://robot_description/meshes/GripperFakeSF/Servo1.STL" />
+        </geometry>
+      </collision>
+    </link>
+    <joint name="Rev1Servo" type="revolute">
+      <origin
+        xyz="0 -0.048595 0.035167"
+        rpy="1.5708 1.5708 0" />
       <parent
         link="Base_Gripper" />
@@ -113,54 +108,51 @@
         xyz="0 1 0" />
       <limit
-        lower="-0.39"
-        upper="0.02"
+        lower="-0.5"
+        upper="0.5"
         effort="0"
         velocity="0" />
     </joint>
-    <link
-      name="Dedo1">
-      <inertial>
-        <origin
-          xyz="-0.0339572900023838 -9.3618305648923E-08 0.148246675379403"
-          rpy="0 0 0" />
-        <mass
-          value="0.0622990489702351" />
-        <inertia
-          ixx="0.000123328183626577"
-          ixy="-1.22881098411723E-10"
-          ixz="-5.84361445598599E-06"
-          iyy="0.000126724273269253"
-          iyz="1.57270956526926E-10"
-          izz="1.60489416583839E-05" />
-      </inertial>
-      <visual>
-        <origin
-          xyz="0 0 0"
-          rpy="0 0 0" />
-        <geometry>
-          <mesh
-            filename="package://robot_description/meshes/Gripper/Dedo1.STL" />
-        </geometry>
-        <material
-          name="">
-          <color
-            rgba="0.792156862745098 0.819607843137255 0.933333333333333 1" />
-        </material>
-      </visual>
-      <collision>
-        <origin
-          xyz="0 0 0"
-          rpy="0 0 0" />
-        <geometry>
-          <mesh
-            filename="package://robot_description/meshes/Gripper/Dedo1.STL" />
-        </geometry>
-      </collision>
-    </link>
-    <joint
-      name="Fix1Dedo"
-      type="fixed">
-      <origin
-        xyz="0.035 0.0021425 -0.0685"
+    <link name="Dedo1">
+      <inertial>
+        <origin
+          xyz="-0.0339571348134233 -9.21108558320401E-08 0.148247426657733"
+          rpy="0 0 0" />
+        <mass
+          value="0.0622996894009069" />
+        <inertia
+          ixx="0.000123327723316758"
+          ixy="-1.34450246244474E-10"
+          ixz="-5.84363068828583E-06"
+          iyy="0.00012672400265891"
+          iyz="1.56255674072228E-10"
+          izz="1.60491252999285E-05" />
+      </inertial>
+      <visual>
+        <origin
+          xyz="0 0 0"
+          rpy="0 0 0" />
+        <geometry>
+          <mesh
+            filename="package://robot_description/meshes/GripperFakeSF/Dedo1.STL" />
+        </geometry>
+        <material
+          name="">
+          <color
+            rgba="0.792156862745098 0.819607843137255 0.933333333333333 1" />
+        </material>
+      </visual>
+      <collision>
+        <origin
+          xyz="0 0 0"
+          rpy="0 0 0" />
+        <geometry>
+          <mesh
+            filename="package://robot_description/meshes/GripperFakeSF/Dedo1.STL" />
+        </geometry>
+      </collision>
+    </link>
+    <joint name="Fix1Dedo" type="fixed">
+      <origin
+        xyz="0.035 0.0021425 -0.0985"
         rpy="0 0 0" />
       <parent
@@ -171,9 +163,8 @@
         xyz="0 0 0" />
     </joint>
-    <link
-      name="Servo2">
-      <inertial>
-        <origin
-          xyz="-4.50497350118484E-08 0.00440252858837639 0.0186297249994028"
+    <link name="Servo2">
+      <inertial>
+        <origin
+          xyz="-4.50497350534818E-08 0.00440252858837659 0.0186297249994028"
           rpy="0 0 0" />
         <mass
@@ -181,8 +172,8 @@
         <inertia
           ixx="1.36408467918995E-05"
-          ixy="1.66044927441445E-19"
-          ixz="-1.7205356741103E-19"
+          ixy="1.57699642761219E-19"
+          ixz="-1.65780172575981E-19"
           iyy="3.54946158391805E-06"
-          iyz="-1.80956359903932E-06"
+          iyz="-1.80956359903934E-06"
           izz="1.22463749616553E-05" />
       </inertial>
@@ -193,28 +184,26 @@
         <geometry>
           <mesh
-            filename="package://robot_description/meshes/Gripper/Servo2.STL" />
-        </geometry>
-        <material
-          name="">
-          <color
-            rgba="0.792156862745098 0.819607843137255 0.933333333333333 1" />
-        </material>
-      </visual>
-      <collision>
-        <origin
-          xyz="0 0 0"
-          rpy="0 0 0" />
-        <geometry>
-          <mesh
-            filename="package://robot_description/meshes/Gripper/Servo2.STL" />
-        </geometry>
-      </collision>
-    </link>
-    <joint
-      name="Rev2Servo"
-      type="revolute">
-      <origin
-        xyz="0 -0.034832 0.088595"
-        rpy="0 -0.02 -1.5708" />
+            filename="package://robot_description/meshes/GripperFakeSF/Servo2.STL" />
+        </geometry>
+        <material
+          name="">
+          <color
+            rgba="0.792156862745098 0.819607843137255 0.933333333333333 1" />
+        </material>
+      </visual>
+      <collision>
+        <origin
+          xyz="0 0 0"
+          rpy="0 0 0" />
+        <geometry>
+          <mesh
+            filename="package://robot_description/meshes/GripperFakeSF/Servo2.STL" />
+        </geometry>
+      </collision>
+    </link>
+    <joint name="Rev2Servo" type="revolute">
+      <origin
+        xyz="0 -0.048595 -0.034832"
+        rpy="1.5708 1.5708 0" />
       <parent
         link="Base_Gripper" />
@@ -224,6 +213,6 @@
         xyz="0 1 0" />
       <limit
-        lower="-0.02"
-        upper="0.39"
+        lower="-0.5"
+        upper="0.5"
         effort="0"
         velocity="0" />
@@ -233,50 +222,47 @@
         offset="0" />
     </joint>
-    <link
-      name="Dedo2">
-      <inertial>
-        <origin
-          xyz="-0.0339571351919315 -9.20512037367108E-08 0.148247430105431"
-          rpy="0 0 0" />
-        <mass
-          value="0.0622996947963828" />
-        <inertia
-          ixx="0.000123327640391479"
-          ixy="-1.34548142614061E-10"
-          ixz="-5.84362978685844E-06"
-          iyy="0.000126723917872848"
-          iyz="1.53337647171162E-10"
-          izz="1.60491213480393E-05" />
-      </inertial>
-      <visual>
-        <origin
-          xyz="0 0 0"
-          rpy="0 0 0" />
-        <geometry>
-          <mesh
-            filename="package://robot_description/meshes/Gripper/Dedo2.STL" />
-        </geometry>
-        <material
-          name="">
-          <color
-            rgba="0.792156862745098 0.819607843137255 0.933333333333333 1" />
-        </material>
-      </visual>
-      <collision>
-        <origin
-          xyz="0 0 0"
-          rpy="0 0 0" />
-        <geometry>
-          <mesh
-            filename="package://robot_description/meshes/Gripper/Dedo2.STL" />
-        </geometry>
-      </collision>
-    </link>
-    <joint
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
File: catkin_home/src/robot_description/urdf/gripper/gripperP.urdf.xacro (robot description, xacro)
@@ -12,6 +12,5 @@
       </joint>
     </xacro:unless>
-    <link
-      name="Base_Gripper">
+    <link name="Base_Gripper">
       <inertial>
         <origin
@@ -59,6 +58,5 @@
       <origin xyz="0.156 0 0.04" rpy="0 0 0" />
     </joint>
-    <link
-      name="Servo1">
+    <link name="Servo1">
       <inertial>
         <origin
@@ -99,6 +97,5 @@
       </collision>
     </link>
-    <joint
-      name="Rev1Servo"
+    <joint name="Rev1Servo"
       type="revolute">
       <origin
@@ -117,6 +114,5 @@
         velocity="0" />
     </joint>
-    <link
-      name="Dedo1">
+    <link name="Dedo1">
       <inertial>
         <origin
@@ -157,6 +153,5 @@
       </collision>
     </link>
-    <joint
-      name="Fix1Dedo"
+    <joint name="Fix1Dedo"
       type="fixed">
       <origin
@@ -170,6 +165,5 @@
         xyz="0 0 0" />
     </joint>
-    <link
-      name="Servo2">
+    <link name="Servo2">
       <inertial>
         <origin
@@ -210,6 +204,5 @@
       </collision>
     </link>
-    <joint
-      name="Rev2Servo"
+    <joint name="Rev2Servo"
       type="revolute">
       <origin
@@ -232,6 +225,5 @@
         offset="0" />
     </joint>
-    <link
-      name="Dedo2">
+    <link name="Dedo2">
       <inertial>
         <origin
@@ -272,6 +264,5 @@
       </collision>
     </link>
-    <joint
-      name="Fix2Dedo"
+    <joint name="Fix2Dedo"
       type="fixed">
       <origin
