Commit message: change gripperSF stl

File: catkin_home/src/robot_description/urdf/dashgo.urdf.xacro (robot description, xacro)
@@ -16,6 +16,6 @@
   <link name="apriltag" />
   <joint name="apriltag_joint" type="fixed">
-    <origin xyz="0.11625 0.03758 0" rpy="0 -1.57 3.1416" />
-    <parent link="link4" />
+    <origin xyz="0 -0.0375 0.0375" rpy="0 -1.57 1.57" />
+    <parent link="link5" />
     <child link="apriltag" />
   </joint>
@@ -290,7 +290,7 @@
   <xacro:include filename="$(find robot_description)/urdf/gripper/gripperFakeSF.urdf.xacro" />
   <xacro:include filename="$(find robot_description)/urdf/gripper/gripperSF.urdf.xacro" />
-  <xacro:load_gripperFakeSF attach_to="$(arg prefix)link_eef" xyz="0 0 0.003" rpy="-1.57 0 1.57" />
+  <xacro:load_gripperSF attach_to="$(arg prefix)link_eef" xyz="0 0 0.007" rpy="-1.57 0 1.57" />
   <xacro:include filename="$(find robot_description)/urdf/camera.urdf.xacro" />
-  <xacro:load_camera name="Cam1" attach_to="Base" x="-0.14733609953780444" y="-0.013216790422497737" z="1.5898169001977585" r_p="0.008378069114521033" r_r="0.7682487395321386" r_y="-1.6006887457492875" />
+  <xacro:load_camera name="Cam1" attach_to="Base" x="-0.1480668895189948" y="0.017240912957425025" z="1.5750724926280606" r_p="0.029148540802230845" r_r="0.8826864963968823" r_y="-1.5168108174976027" />
   <xacro:load_camera name="Cam2" attach_to="Base" x="-0.085" y="-0.24" z="0.48" r_r="0.538132" r_p="0" r_y="-1.5708" />
 </robot>

File: catkin_home/src/robot_description/urdf/gripper/gripperSF.urdf.xacro (robot description, xacro)
@@ -15,27 +15,28 @@
     </link>
     <joint name="end_effector_joint" type="fixed">
-      <parent link="Base_Gripper" />
-      <child link="end_effector_link" />
-      <origin xyz="0.0 -0.14 0" rpy="1.57 0 -1.57" />
+        <parent link="Base_Gripper" />
+        <child link="end_effector_link" />
+        <origin xyz="0.0 -0.125 0" rpy="1.57 0 -1.57" />
     </joint>
-    <link name="Base_Gripper">
+    <link
+      name="Base_Gripper">
       <inertial>
         <origin
-          xyz="-0.00600744878247479 0.000229447019284631 0.0275811003234641"
+          xyz="4.21738922031144E-18 2.00787620612413E-18 0.0378144840174591"
           rpy="0 0 0" />
         <mass
-          value="0.25675298967361" />
+          value="0.516607789353608" />
         <inertia
-          ixx="0.000297324022723542"
-          ixy="5.57701217289319E-07"
-          ixz="6.8196059580779E-06"
-          iyy="0.000115396784513201"
-          iyz="-6.39913613193201E-07"
-          izz="0.000284254818153183" />
+          ixx="0.000831389945414142"
+          ixy="-2.21787801740781E-20"
+          ixz="1.66219465220325E-20"
+          iyy="0.000443816179175048"
+          iyz="3.05902948293233E-21"
+          izz="0.000681097815743884" />
       </inertial>
       <visual>
         <origin
           xyz="0 0 0"
-          rpy="0 0 0" />
+          rpy="1.57 0 0" />
         <geometry>
           <mesh
@@ -57,224 +58,231 @@
         </geometry>
       </collision>
-    </link>
-    <link name="Servo1">
-      <inertial>
-        <origin
-          xyz="-4.50497350465429E-08 0.00440252858837645 0.0186297249994028"
-          rpy="0 0 0" />
-        <mass
-          value="0.0250047254852253" />
-        <inertia
-          ixx="1.36408467918995E-05"
-          ixy="1.57389452627317E-19"
-          ixz="-1.65284737063933E-19"
-          iyy="3.54946158391806E-06"
-          iyz="-1.80956359903934E-06"
-          izz="1.22463749616553E-05" />
-      </inertial>
-      <visual>
-        <origin
-          xyz="0 0 0"
-          rpy="0 0 0" />
-        <geometry>
-          <mesh
-            filename="package://robot_description/meshes/GripperSF/Servo1.STL" />
-        </geometry>
-        <material
-          name="">
-          <color
-            rgba="0.792156862745098 0.819607843137255 0.933333333333333 1" />
-        </material>
-      </visual>
-      <collision>
-        <origin
-          xyz="0 0 0"
-          rpy="0 0 0" />
-        <geometry>
-          <mesh
-            filename="package://robot_description/meshes/GripperSF/Servo1.STL" />
-        </geometry>
-      </collision>
-    </link>
-    <joint name="Rev1Servo" type="revolute">
-      <origin
-        xyz="0 -0.048595 0.035167"
-        rpy="1.5708 1.5708 0" />
-      <parent
-        link="Base_Gripper" />
-      <child
-        link="Servo1" />
-      <axis
-        xyz="0 1 0" />
-      <limit
-        lower="-0.5"
-        upper="0.5"
-        effort="0"
-        velocity="0" />
-    </joint>
-    <link name="Dedo1">
-      <inertial>
-        <origin
-          xyz="-0.0339571348134233 -9.21108558320401E-08 0.148247426657733"
-          rpy="0 0 0" />
-        <mass
-          value="0.0622996894009069" />
-        <inertia
-          ixx="0.000123327723316758"
-          ixy="-1.34450246244474E-10"
-          ixz="-5.84363068828583E-06"
-          iyy="0.00012672400265891"
-          iyz="1.56255674072228E-10"
-          izz="1.60491252999285E-05" />
-      </inertial>
-      <visual>
-        <origin
-          xyz="0 0 0"
-          rpy="0 0 0" />
-        <geometry>
-          <mesh
-            filename="package://robot_description/meshes/GripperSF/Dedo1.STL" />
-        </geometry>
-        <material
-          name="">
-          <color
-            rgba="0.792156862745098 0.819607843137255 0.933333333333333 1" />
-        </material>
-      </visual>
-      <collision>
-        <origin
-          xyz="0 0 0"
-          rpy="0 0 0" />
-        <geometry>
-          <mesh
-            filename="package://robot_description/meshes/GripperSF/Dedo1.STL" />
-        </geometry>
-      </collision>
-    </link>
-    <joint name="Fix1Dedo" type="fixed">
-      <origin
-        xyz="0.035 0.0021425 -0.0985"
-        rpy="0 0 0" />
-      <parent
-        link="Servo1" />
-      <child
-        link="Dedo1" />
-      <axis
-        xyz="0 0 0" />
-    </joint>
-    <link name="Servo2">
-      <inertial>
-        <origin
-          xyz="-4.50497350534818E-08 0.00440252858837659 0.0186297249994028"
-          rpy="0 0 0" />
-        <mass
-          value="0.0250047254852253" />
-        <inertia
-          ixx="1.36408467918995E-05"
-          ixy="1.57699642761219E-19"
-          ixz="-1.65780172575981E-19"
-          iyy="3.54946158391805E-06"
-          iyz="-1.80956359903934E-06"
-          izz="1.22463749616553E-05" />
-      </inertial>
-      <visual>
-        <origin
-          xyz="0 0 0"
-          rpy="0 0 0" />
-        <geometry>
-          <mesh
-            filename="package://robot_description/meshes/GripperSF/Servo2.STL" />
-        </geometry>
-        <material
-          name="">
-          <color
-            rgba="0.792156862745098 0.819607843137255 0.933333333333333 1" />
-        </material>
-      </visual>
-      <collision>
-        <origin
-          xyz="0 0 0"
-          rpy="0 0 0" />
-        <geometry>
-          <mesh
-            filename="package://robot_description/meshes/GripperSF/Servo2.STL" />
-        </geometry>
-      </collision>
-    </link>
-    <joint name="Rev2Servo" type="revolute">
-      <origin
-        xyz="0 -0.048595 -0.034832"
-        rpy="1.5708 1.5708 0" />
-      <parent
-        link="Base_Gripper" />
-      <child
-        link="Servo2" />
-      <axis
-        xyz="0 1 0" />
-      <limit
-        lower="-0.5"
-        upper="0.5"
-        effort="0"
-        velocity="0" />
-      <mimic
-        joint="Rev1Servo"
-        multiplier="-1"
-        offset="0" />
-    </joint>
-    <link name="Dedo2">
-      <inertial>
-        <origin
-          xyz="-0.0339566917270822 -9.21107859009999E-08 0.148247426657711"
-          rpy="0 0 0" />
-        <mass
-          value="0.0622996894008418" />
-        <inertia
-          ixx="0.000123327723316674"
-          ixy="-1.34450244755006E-10"
-          ixz="-5.84363068828243E-06"
-          iyy="0.000126724002658815"
-          iyz="1.56255677499792E-10"
-          izz="1.60491252999025E-05" />
-      </inertial>
-      <visual>
-        <origin
-          xyz="0 0 0"
-          rpy="0 0 0" />
-        <geometry>
-          <mesh
-            filename="package://robot_description/meshes/GripperSF/Dedo2.STL" />
-        </geometry>
-        <material
-          name="">
-          <color
-            rgba="0.792156862745098 0.819607843137255 0.933333333333333 1" />
-        </material>
-      </visual>
-      <collision>
-        <origin
-          xyz="0 0 0"
-          rpy="0 0 0" />
-        <geometry>
-          <mesh
-            filename="package://robot_description/meshes/GripperSF/Dedo2.STL" />
-        </geometry>
-      </collision>
-    </link>
-    <joint name="Fix2Dedo" type="fixed">
-      <origin
-        xyz="-0.035 0.0021425 -0.0985"
-        rpy="0 0 3.1416" />
-      <parent
-        link="Servo2" />
-      <child
-        link="Dedo2" />
-      <axis
-        xyz="0 0 0" />
-      <limit
-        lower="0"
-        upper="0"
-        effort="0"
-        velocity="0" />
-    </joint>
+  </link>
+  <link
+    name="Servo1">
+    <inertial>
+      <origin
+        xyz="2.08166817117217E-17 0.00765209400201583 0.002"
+        rpy="0 0 0" />
+      <mass
+        value="0.00340320788790707" />
+      <inertia
+        ixx="3.64324463782157E-07"
+        ixy="-7.27918939046664E-23"
+        ixz="-2.27911008833175E-24"
+        iyy="1.72972745084653E-07"
+        iyz="3.50518784550926E-24"
+        izz="5.28221987832391E-07" />
+    </inertial>
+    <visual>
+      <origin
+        xyz="0 0 0"
+        rpy="0 0 0" />
+      <geometry>
+        <mesh
+          filename="package://robot_description/meshes/GripperSF/Servo1.STL" />
+      </geometry>
+      <material
+        name="">
+        <color
+          rgba="0.792156862745098 0.819607843137255 0.933333333333333 1" />
+      </material>
+    </visual>
+    <collision>
+      <origin
+        xyz="0 0 0"
+        rpy="0 0 0" />
+      <geometry>
+        <mesh
+          filename="package://robot_description/meshes/GripperSF/Servo1.STL" />
+      </geometry>
+    </collision>
+  </link>
+  <joint
+    name="Rev1Servo"
+    type="revolute">
+    <origin
+      xyz="0.025 -0.085 0.0125"
+      rpy="1.5708 -0.7854 1.5708" />
+    <parent
+      link="Base_Gripper" />
+    <child
+      link="Servo1" />
+    <axis
+      xyz="0 0 1" />
+    <limit
+      lower="-0.52"
+      upper="0.52"
+      effort="0"
+      velocity="0" />
+  </joint>
+  <link
+    name="Dedo1">
+    <inertial>
+      <origin
+        xyz="0.025 0.0194950722582391 0.0215202503489297"
+        rpy="0 0 0" />
+      <mass
+        value="0.0481456303681194" />
+      <inertia
+        ixx="1.85056890508066E-05"
+        ixy="6.4090118340269E-22"
+        ixz="1.49782108916524E-21"
+        iyy="2.29959536609367E-05"
+        iyz="-7.07475784630465E-06"
+        izz="1.55704147099196E-05" />
+    </inertial>
+    <visual>
+      <origin
+        xyz="0 0 0"
+        rpy="3.14 0 0" />
+      <geometry>
+        <mesh
+          filename="package://robot_description/meshes/GripperSF/Dedo1.STL" />
+      </geometry>
+      <material
+        name="">
+        <color
+          rgba="0.792156862745098 0.819607843137255 0.933333333333333 1" />
+      </material>
+    </visual>
+    <collision>
+      <origin
+        xyz="0 0 0"
+        rpy="0 0 0" />
+      <geometry>
+        <mesh
+          filename="package://robot_description/meshes/GripperSF/Dedo1.STL" />
+      </geometry>
+    </collision>
+  </link>
+  <joint
+    name="Fix1Dedo"
+    type="fixed">
+    <origin
+      xyz="0 0.025 -0.046"
+      rpy="3.1416 -1.5708 0" />
+    <parent
+      link="Servo1" />
+    <child
+      link="Dedo1" />
+    <axis
+      xyz="0 0 0" />
+  </joint>
+  <link
+    name="Servo2">
+    <inertial>
+      <origin
+        xyz="-6.93889390390723E-18 0.00765209400201584 0.00200000000000001"
+        rpy="0 0 0" />
+      <mass
+        value="0.00340320788790707" />
+      <inertia
+        ixx="3.64324463782157E-07"
+        ixy="1.45583787809333E-22"
+        ixz="4.15267079728299E-24"
+        iyy="1.72972745084653E-07"
+        iyz="3.30065685426304E-24"
+        izz="5.28221987832391E-07" />
+    </inertial>
+    <visual>
+      <origin
+        xyz="0 0 0"
+        rpy="0 0 0" />
+      <geometry>
+        <mesh
+          filename="package://robot_description/meshes/GripperSF/Servo2.STL" />
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
Commit message: Xarm 6 update

File: catkin_home/src/robot_description/urdf/dashgo.urdf.xacro (robot description, xacro)
@@ -16,6 +16,6 @@
   <link name="apriltag" />
   <joint name="apriltag_joint" type="fixed">
-    <origin xyz="0 -0.0375 0.0375" rpy="0 -1.57 1.57" />
-    <parent link="link5" />
+    <origin xyz="0.03 -0.035 0" rpy="1.57 3.14 1.57" />
+    <parent link="Base_Gripper" />
     <child link="apriltag" />
   </joint>
@@ -284,13 +284,13 @@
   <xacro:arg name="geometry_mesh_tcp_rpy" default="0 0 0" />
   <xacro:arg name="add_realsense_d435i" default="false" />
-  <xacro:include filename="$(find xarm_description)/urdf/xarm5_robot_macro.xacro" />
-  <xacro:xarm5_robot prefix="$(arg prefix)" namespace="$(arg ros_namespace)" limited="$(arg limited)" effort_control="$(arg effort_control)" velocity_control="$(arg velocity_control)" rs_d435i="$(arg add_realsense_d435i)" attach_to="BaseBrazo" add_other_geometry="$(arg add_other_geometry)" geometry_type="$(arg geometry_type)" geometry_mass="$(arg geometry_mass)" geometry_height="$(arg geometry_height)" geometry_radius="$(arg geometry_radius)" geometry_length="$(arg geometry_length)" geometry_width="$(arg geometry_width)" geometry_mesh_filename="$(arg geometry_mesh_filename)" geometry_mesh_origin_xyz="$(arg geometry_mesh_origin_xyz)" geometry_mesh_origin_rpy="$(arg geometry_mesh_origin_rpy)" geometry_mesh_tcp_xyz="$(arg geometry_mesh_tcp_xyz)" geometry_mesh_tcp_rpy="$(arg geometry_mesh_tcp_rpy)" />
+  <xacro:include filename="$(find xarm_description)/urdf/xarm6_robot_macro.xacro" />
+  <xacro:xarm6_robot prefix="$(arg prefix)" namespace="$(arg ros_namespace)" limited="$(arg limited)" effort_control="$(arg effort_control)" velocity_control="$(arg velocity_control)" rs_d435i="$(arg add_realsense_d435i)" attach_to="BaseBrazo" add_other_geometry="$(arg add_other_geometry)" geometry_type="$(arg geometry_type)" geometry_mass="$(arg geometry_mass)" geometry_height="$(arg geometry_height)" geometry_radius="$(arg geometry_radius)" geometry_length="$(arg geometry_length)" geometry_width="$(arg geometry_width)" geometry_mesh_filename="$(arg geometry_mesh_filename)" geometry_mesh_origin_xyz="$(arg geometry_mesh_origin_xyz)" geometry_mesh_origin_rpy="$(arg geometry_mesh_origin_rpy)" geometry_mesh_tcp_xyz="$(arg geometry_mesh_tcp_xyz)" geometry_mesh_tcp_rpy="$(arg geometry_mesh_tcp_rpy)" />
   <xacro:include filename="$(find robot_description)/urdf/gripper/gripper.urdf.xacro" />
   <xacro:include filename="$(find robot_description)/urdf/gripper/gripperP.urdf.xacro" />
   <xacro:include filename="$(find robot_description)/urdf/gripper/gripperFakeSF.urdf.xacro" />
   <xacro:include filename="$(find robot_description)/urdf/gripper/gripperSF.urdf.xacro" />
-  <xacro:load_gripperSF attach_to="$(arg prefix)link_eef" xyz="0 0 0.007" rpy="-1.57 0 1.57" />
+  <xacro:load_gripperSF attach_to="$(arg prefix)link_eef" xyz="0 0 0.007" rpy="-1.57 0 2.3554" />
   <xacro:include filename="$(find robot_description)/urdf/camera.urdf.xacro" />
-  <xacro:load_camera name="Cam1" attach_to="Base" x="-0.1480668895189948" y="0.017240912957425025" z="1.5750724926280606" r_p="0.029148540802230845" r_r="0.8826864963968823" r_y="-1.5168108174976027" />
+  <xacro:load_camera name="Cam1" attach_to="Base" x="-0.1489890924003532" y="0.012537554524483352" z="1.576021669791469" r_p="-0.023918715399906476" r_r="0.7386447939707235" r_y="-1.5125889208048597" />
   <xacro:load_camera name="Cam2" attach_to="Base" x="-0.085" y="-0.24" z="0.48" r_r="0.538132" r_p="0" r_y="-1.5708" />
 </robot>

Commit message: Gripper on camera. Calibration not tested

File: catkin_home/src/robot_description/urdf/dashgo.urdf.xacro (robot description, xacro)
@@ -16,6 +16,6 @@
   <link name="apriltag" />
   <joint name="apriltag_joint" type="fixed">
-    <origin xyz="0.03 -0.035 0" rpy="1.57 3.14 1.57" />
-    <parent link="Base_Gripper" />
+    <origin xyz="0.06 0 0.06" rpy="3.14 -1.57 0" />
+    <parent link="BaseBrazo" />
     <child link="apriltag" />
   </joint>
@@ -292,5 +292,5 @@
   <xacro:load_gripperSF attach_to="$(arg prefix)link_eef" xyz="0 0 0.007" rpy="-1.57 0 2.3554" />
   <xacro:include filename="$(find robot_description)/urdf/camera.urdf.xacro" />
-  <xacro:load_camera name="Cam1" attach_to="Base" x="-0.1489890924003532" y="0.012537554524483352" z="1.576021669791469" r_p="-0.023918715399906476" r_r="0.7386447939707235" r_y="-1.5125889208048597" />
+  <xacro:load_camera name="Cam1" attach_to="Base_Gripper" x="0.05" y="0" z="-0.05" r_p="0" r_r="0" r_y="0" />
   <xacro:load_camera name="Cam2" attach_to="Base" x="-0.085" y="-0.24" z="0.48" r_r="0.538132" r_p="0" r_y="-1.5708" />
 </robot>

Commit message: No column v1.

File: catkin_home/src/robot_description/urdf/dashgo.urdf.xacro (robot description, xacro)
@@ -36,7 +36,7 @@
     </visual>
     <collision>
-      <origin xyz="0 0 0" rpy="0 0 0" />
-      <geometry>
-        <mesh filename="package://robot_description/meshes/Dashgo/Base_Collisions.STL" />
+      <origin xyz="-.235 -.2371 0" rpy="0 0 0" />
+      <geometry>
+        <mesh filename="package://robot_description/meshes/Dashgo/Base_Collisions_CamGripper.STL" />
       </geometry>
     </collision>

Commit message: Arm action server & URDF update

File: catkin_home/src/robot_description/urdf/dashgo.urdf.xacro (robot description, xacro)
@@ -29,14 +29,14 @@
       <origin xyz="0 0 0" rpy="0 0 0" />
       <geometry>
-        <mesh filename="package://robot_description/meshes/Dashgo/Base.STL" />
-      </geometry>
-      <material name="">
-        <color rgba="0.792156862745098 0.819607843137255 0.933333333333333 1" />
-      </material>
-    </visual>
-    <collision>
-      <origin xyz="0 0 0" rpy="0 0 0" />
-      <geometry>
-        <mesh filename="package://robot_description/meshes/Dashgo/Base_Collisions.STL" />
+        <mesh filename="package://robot_description/meshes/Dashgo/BaseSinPalo.stl" />
+      </geometry>
+      <material name="">
+        <color rgba="0.792156862745098 0.819607843137255 0.933333333333333 1" />
+      </material>
+    </visual>
+    <collision>
+      <origin xyz="0 0 0" rpy="0 0 0" />
+      <geometry>
+        <mesh filename="package://robot_description/meshes/Dashgo/BaseCollisionsSinPalo.stl" />
       </geometry>
     </collision>

Commit message: Cam gripper urdf updated

File: catkin_home/src/robot_description/urdf/dashgo.urdf.xacro (robot description, xacro)
@@ -16,6 +16,6 @@
   <link name="apriltag" />
   <joint name="apriltag_joint" type="fixed">
-    <origin xyz="0.03 -0.035 0" rpy="1.57 3.14 1.57" />
-    <parent link="Base_Gripper" />
+    <origin xyz="0.06 0 0.06" rpy="3.14 -1.57 0" />
+    <parent link="BaseBrazo" />
     <child link="apriltag" />
   </joint>
@@ -292,5 +292,5 @@
   <xacro:load_gripperSF attach_to="$(arg prefix)link_eef" xyz="0 0 0.007" rpy="-1.57 0 2.3554" />
   <xacro:include filename="$(find robot_description)/urdf/camera.urdf.xacro" />
-  <xacro:load_camera name="Cam1" attach_to="Base" x="-0.1489890924003532" y="0.012537554524483352" z="1.576021669791469" r_p="-0.023918715399906476" r_r="0.7386447939707235" r_y="-1.5125889208048597" />
+  <xacro:load_camera name="Cam1" attach_to="Base_Gripper" x="0.07" y="-0.05" z="0.0" r_p="-0.785398" r_r="1.5707" r_y="0.0" />
   <xacro:load_camera name="Cam2" attach_to="Base" x="-0.085" y="-0.24" z="0.48" r_r="0.538132" r_p="0" r_y="-1.5708" />
 </robot>

Commit message: Dashgo urdf updated (testing missing)

File: catkin_home/src/robot_description/urdf/dashgo.urdf.xacro (robot description, xacro)
@@ -29,14 +29,14 @@
       <origin xyz="0 0 0" rpy="0 0 0" />
       <geometry>
-        <mesh filename="package://robot_description/meshes/Dashgo/BaseSinPalo.stl" />
-      </geometry>
-      <material name="">
-        <color rgba="0.792156862745098 0.819607843137255 0.933333333333333 1" />
-      </material>
-    </visual>
-    <collision>
-      <origin xyz="0 0 0" rpy="0 0 0" />
-      <geometry>
-        <mesh filename="package://robot_description/meshes/Dashgo/BaseCollisionsSinPalo.stl" />
+        <mesh filename="package://robot_description/meshes/Dashgo/dashgo_cubierta.stl" />
+      </geometry>
+      <material name="">
+        <color rgba="0.792156862745098 0.819607843137255 0.933333333333333 1" />
+      </material>
+    </visual>
+    <collision>
+      <origin xyz="0 0 0" rpy="0 0 0" />
+      <geometry>
+        <mesh filename="package://robot_description/meshes/Dashgo/dashgo_cubierta_collisions.stl" />
       </geometry>
     </collision>

Commit message: URDF Base updated

File: catkin_home/src/robot_description/urdf/dashgo.urdf.xacro (robot description, xacro)
@@ -38,5 +38,5 @@
       <origin xyz="0 0 0" rpy="0 0 0" />
       <geometry>
-        <mesh filename="package://robot_description/meshes/Dashgo/dashgo_cubierta_collisions.stl" />
+        <mesh filename="package://robot_description/meshes/Dashgo/dashgo_cubierta_colliders.stl" />
       </geometry>
     </collision>
