Commit message: changes to tiago files

File: docker/noetic/tiago_files/tiago.srdf.xacro (robot description, xacro)
@@ -26,4 +26,6 @@
     <!--CHAINS: When a chain is specified, all the links along the chain (including endpoints) are included in the group. Additionally, all the joints that are parents to included links are also included. This means that joints along the chain and the parent joint of the base link are included in the group-->
     <!--SUBGROUPS: Groups can also be formed by referencing to already defined group names-->
+    <!--VIRTUAL JOINT: Purpose: this element defines a virtual joint between a robot link and an external frame of reference (considered fixed with respect to the robot)-->
+    <virtual_joint name="world_joint" type="planar" parent_frame="odom" child_link="internal_odom"/>
 <xacro:if value="${has_arm}">
     <group name="arm">
@@ -48,4 +50,13 @@
         <joint name="arm_tool_joint" />
     </group>
+    <group name="base">
+        <joint name="odom_x"/>
+        <joint name="odom_y"/>
+        <joint name="odom_r"/>
+    </group>
+    <group name="whole_body">
+        <group name="base"/>
+        <group name="arm_torso"/>
+    </group>
     <xacro:include filename="$(find tiago_moveit_config)/config/srdf/end_effectors/${end_effector}.srdf.xacro" />
     <xacro:define_end_effector arm="arm" name="${end_effector_name}"/>

Commit message: add head planning group to srdf - Tiago

File: docker/noetic/tiago_files/tiago.srdf.xacro (robot description, xacro)
@@ -55,4 +55,8 @@
         <joint name="odom_r"/>
     </group>
+    <group name="head">
+        <joint name="head_1_joint"/>
+        <joint name="head_2_joint"/>
+    </group>
     <group name="whole_body">
         <group name="base"/>

Commit message: pick v1.0 with Tiago

File: docker/noetic/tiago_files/tiago.srdf.xacro (robot description, xacro)
@@ -38,4 +38,5 @@
         <joint name="arm_7_joint" />
         <joint name="arm_tool_joint" />
+        <joint name="end_effector_joint" />
     </group>
     <group name="arm_torso">
@@ -49,4 +50,5 @@
         <joint name="arm_7_joint" />
         <joint name="arm_tool_joint" />
+        <joint name="end_effector_joint" />
     </group>
     <group name="base">
